File: Hardware/PS-AmperesPCB.kicad_pcb (KiCad board)
At the start: 2 copper layers, 80.6 x 94.4 mm, 164 parts, among them IC1 SN74AHC1G32DBVR, IC2 INA241A4IDR, IC3 AMC1350DWVR, IC4 TLV9002QDRQ1, IC5 LM76202QPWPRQ1, J1 PeripheralCAN, J2 PeripheralCAN, J3 SWD, J4 Conn_01x02_Pin, J5 USB4120-03-C, J6 Scrut Conn, SW1 RST, SW2 BOOT, SW3 Scrut Select, U1 LT1963AEST-3.3#TRPBF, U2 TPS5405DR, U3 TPS2115ADRBR, U4 LT1963AEST-3.3#TRPBF, U5 STM32L431CBTx, U6 TCAN337, U7 CDSOT23-T24CAN, U8 CP2102N-A02-GQFN24, U9 REF35125QDBVR, Y1 8M

Commit message: slightly cooked
Parts:
- removed C44: 7.5uF, Capacitor_SMD:C_0603_1608Metric_Pad1.08x0.95mm_HandSolder
- removed IC4: TLV9002QDRQ1, Parts:TLV9002QDRQ1
- removed SW3: Scrut Select, Parts:CAS220TB
- added C55: 0.1uF, Capacitor_SMD:C_0603_1608Metric_Pad1.08x0.95mm_HandSolder, F.Cu at (214.3, 75.1)
- added D19: VBUS, LED_SMD:LED_0603_1608Metric_Pad1.05x0.95mm_HandSolder, F.Cu at (232.7, 75.2)
- added F2: 3568, Fuse:Fuseholder_Blade_Mini_Keystone_3568, F.Cu at (216.0, 66.0)
- added R24: 768, Resistor_SMD:R_0603_1608Metric_Pad0.98x0.95mm_HandSolder, F.Cu at (232.7, 77.7)
- added R40: 0, Resistor_SMD:R_0603_1608Metric_Pad0.98x0.95mm_HandSolder, F.Cu at (214.3, 77.6)
- added R41: 10k, Resistor_SMD:R_0603_1608Metric_Pad0.98x0.95mm_HandSolder, F.Cu at (232.7, 82.2)
- added R42: 10k, Resistor_SMD:R_0603_1608Metric_Pad0.98x0.95mm_HandSolder, F.Cu at (233.9, 64.8)
- added R43: 10k, Resistor_SMD:R_0603_1608Metric_Pad0.98x0.95mm_HandSolder, F.Cu at (214.3, 80.1)
- added R45: 24.9k, Resistor_SMD:R_0603_1608Metric_Pad0.98x0.95mm_HandSolder, F.Cu at (214.3, 82.6)
- added SW4: Scrut Select, Parts:SW_CJS-1200TA, F.Cu at (220.0, 83.2)
- added TP20: Out-, TestPoint:TestPoint_Pad_1.0x1.0mm, F.Cu at (226.0, 83.0)
- added U10: TLV9002QDRQ1, Package_SO:SOIC-8_3.9x4.9mm_P1.27mm, F.Cu at (220.7, 77.2)
- C41: value 1uF -> 68nF
- C49: value 0.1uF -> 68nF
- J5: value USB4120-03-C -> USB4105-GF-A; footprint Parts:USB412003C -> UTSVT_Connectors:USB_C_Receptacle_GCT_USB4105-xx-A_16P_TopMnt_Horizontal
- R25: value 8.2k -> 0
- R26: value 3.3k -> 24.9k
- R27: value 4.3k -> 10k
- R28: value 34k -> 47k
- R29: value 51 -> 50
- TP1: value TP_Current -> I_OUT
- TP15, TP8, TP9: footprint TestPoint:TestPoint_Pad_1.0x1.0mm -> TestPoint:TestPoint_Pad_1.5x1.5mm
- TP17, TP18, TP19: footprint TestPoint:TestPoint_Keystone_5005-5009_Compact -> TestPoint:TestPoint_Pad_1.0x1.0mm
- moved J5 56.7 mm to (217.6, 94.3), turned to 0 degrees
Connections:
- net Net-(IC1-A) renamed /MCU/Boot_SW
- C41 pad 1: Net-(IC4-IN1-) -> Net-(U10A--)
- C49 pad 1: +3.3V -> Net-(U10A-+)
- IC2 pad 1: /Current Sense/INPUT- -> GND HV
- IC3 pad 6: GND -> /Current Sense/OUT-
- J1 pad 1: +24V_Ext -> +24V_In
- J2 pad 1: +24V_Ext -> +24V_In
- R25 pad 1: Net-(C44-Pad1) -> /Current Sense/SHUNT-
- R25 pad 2: /Current Sense/OUT1 -> GND HV
- R26 pad 1: /Current Sense/OUT+ -> Net-(U10A--)
- R26 pad 2: Net-(C44-Pad1) -> /Current Sense/OUT1
- R27 pad 1: Net-(C44-Pad1) -> /Current Sense/OUT-
- R27 pad 2: Net-(IC4-IN1-) -> Net-(U10A--)
- U5 pad 17: /MCU/Boot_GPIO -> unconnected-(U5-PA7-Pad17)
- U8 pad 14: unconnected-(U8-~{TXT}/GPIO.0-Pad14) -> /MCU/Boot_GPIO
Routing:
- net GND HV: track 0.00 -> 7.14 mm
- net /Current Sense/INPUT-: track 7.14 -> 0.00 mm
- net Net-(C44-Pad1): track 6.82 -> 0.00 mm
- net (no net): track 0.00 -> 6.82 mm
- net Net-(U10A--): track 0.00 -> 5.23 mm
- net Net-(IC4-IN1-): track 5.23 -> 0.00 mm
- net Net-(U10A-+): track 0.00 -> 2.68 mm, vias 0 -> 1
- net +3.3V: track 111.2 -> 108.6 mm, vias 27 -> 26

Commit message: started layout not really but kind of
Parts:
- removed R41: 10k, Resistor_SMD:R_0603_1608Metric_Pad0.98x0.95mm_HandSolder
- moved SW4 62.9 mm to (167.0, 49.4), turned to -45 degrees
- moved D13 54.0 mm to (221.3, 102.9)
- moved C32 54.0 mm to (220.2, 95.4)
- moved C33 54.0 mm to (218.2, 95.1)
- moved C34 54.0 mm to (219.4, 98.4)
- moved C35 54.0 mm to (220.2, 91.4)
- moved C36 54.0 mm to (218.2, 91.6)
- moved D14 54.0 mm to (214.4, 97.5)
- moved R19 54.0 mm to (219.1, 92.0)
- moved R20 54.0 mm to (219.1, 96.3)
- moved R21 54.0 mm to (219.1, 94.1)
- moved R22 54.0 mm to (214.4, 106.8)
- moved R23 54.0 mm to (214.4, 100.5)
- moved U8 54.0 mm to (214.5, 92.5)
- moved R42 36.7 mm to (207.8, 90.6)
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Routing:
- net /MCU/Boot_GPIO: track 22.1 -> 0.00 mm, vias 2 -> 0
- net /Current Sense/OUT1: track 13.5 -> 1.13 mm
- net /Current Sense/OUT+: track 11.9 -> 0.00 mm, vias 1 -> 0
- net +24V_Ext: track 9.85 -> 0.00 mm, vias 1 -> 0
- net /Current Sense/INPUT+: track 7.10 -> 0.00 mm
- net (no net): track 6.82 -> 0.00 mm
- net /USB/D+: track 11.1 -> 4.27 mm
- net GND HV: track 7.14 -> 1.43 mm
- net /Current Sense/SENSE+: track 16.6 -> 11.3 mm, vias 1 -> 0
- net /MCU/ADC1_IN16: track 117.5 -> 113.8 mm
- net /USB/VBUS_IN: track 9.06 -> 5.60 mm, vias 5 -> 3
- net Net-(U10A-+): track 2.68 -> 0.00 mm, vias 1 -> 0
- net /USB/CC1: track 2.38 -> 0.00 mm, vias 1 -> 0
- net /USB/CC2: track 2.30 -> 0.00 mm, vias 1 -> 0
- net /USB/D-: track 14.0 -> 12.2 mm
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
Commit message: layout stuff
Parts:
- C23, C24, C26, C32, C33, C35, C36, FB1, FB2, R22, R23: moved to F.Cu
- TP1: footprint TestPoint:TestPoint_Keystone_5005-5009_Compact -> Connector_PinHeader_2.54mm:PinHeader_1x01_P2.54mm_Vertical
- TP15, TP8, TP9: footprint TestPoint:TestPoint_Pad_1.5x1.5mm -> UTSVT_Special:TestPoint_HEX_3mmID
- moved J2 240.6 mm to (366.0, 90.8), turned to 0 degrees
- moved TP10 122.2 mm to (246.8, 47.3)
- moved TP12 122.2 mm to (246.8, 51.3)
- moved TP16 122.2 mm to (246.8, 55.3)
- moved TP9 122.2 mm to (246.8, 59.1), turned to -90 degrees
- moved TP11 122.2 mm to (241.7, 47.2)
- moved TP13 122.2 mm to (241.7, 55.2)
- moved TP14 122.2 mm to (241.7, 51.3)
- moved TP4 122.2 mm to (241.7, 59.2)
- moved TP1 107.5 mm to (105.3, 140.6)
- moved TP18 107.5 mm to (99.2, 140.6)
- moved U10 84.6 mm to (138.8, 98.0), turned to -90 degrees
- moved R45 84.0 mm to (132.0, 99.4), turned to -90 degrees
- moved C55 84.0 mm to (131.7, 90.5), turned to -90 degrees
- moved R43 82.1 mm to (133.6, 95.4), turned to 90 degrees
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Connections:
- D14 pad 2: /USB/D+ -> /USB/D-
- D14 pad 3: /USB/D- -> /USB/D+
Routing:
- net /MCU/ADC1_IN16: track 113.8 -> 3.61 mm, vias 2 -> 0
- net +3.3V: track 106.9 -> 21.5 mm, vias 26 -> 0
- net /CAN_LOW: track 87.5 -> 2.25 mm, vias 3 -> 0
- net /CAN_HIGH: track 84.3 -> 0.00 mm, vias 3 -> 0
- net /Current Sense/SHUNT+: track 46.6 -> 0.00 mm, vias 2 -> 0
- net /Current Sense/SHUNT-: track 43.2 -> 0.00 mm, vias 2 -> 0
- net /Current Sense/Scrut_Out: track 41.2 -> 0.02 mm, vias 2 -> 0
- net /Current Sense/Scrut-: track 42.2 -> 1.56 mm, vias 1 -> 0
- net +5V_VBUS: track 38.8 -> 0.00 mm, vias 7 -> 0
- net /Current Sense/Scrut+: track 35.6 -> 0.00 mm, vias 2 -> 0
- net /Current Sense/I_OUT: track 31.5 -> 0.81 mm
- net GND: track 58.7 -> 29.4 mm, vias 94 -> 1
- net +1V25: track 28.6 -> 3.92 mm, vias 4 -> 0
- net /MCU/USART1_RX: track 20.3 -> 0.00 mm, vias 2 -> 0
- net /MCU/SWCLK: track 20.2 -> 0.00 mm
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- removed copper zone on F.Cu, net +24V
- removed copper zone on F.Cu, net +24V_Ext
- removed copper zone on F.Cu, net +3.3V
- removed copper zone on B.Cu, net +5V_BUCK
- removed copper zone on B.Cu, net +5V_VBUS
- removed copper zone on B.Cu, net /USB/VBUS_IN
Other:
- board text added: "Michael Adeluyi | Amperes RevB | December 2025"
- board text removed: "Michael Adeluyi - Amperes RevB - October 2025"
