File: Hardware/PS-AmperesPCB.kicad_pcb (KiCad board)
At the start: 2 copper layers, 80.6 x 94.4 mm, 172 parts, among them IC1 SN74AHC1G32DBVR, IC2 INA241A4IDR, IC3 AMC1350DWVR, IC5 LM76202QPWPRQ1, J1 PeripheralCAN, J2 PeripheralCAN, J3 SWD, J4 Conn_01x02_Pin, J5 USB4105-GF-A, J6 Scrut Conn, SW1 RST, SW2 BOOT, SW4 Scrut Select, U1 LT1963AEST-3.3#TRPBF, U10 TLV9002QDRQ1, U2 TPS5405DR, U3 TPS2115ADRBR, U4 LT1963AEST-3.3#TRPBF, U5 STM32L431CBTx, U6 TCAN337, U7 CDSOT23-T24CAN, U8 CP2102N-A02-GQFN24, U9 REF35125QDBVR, Y1 8M

Commit message: post review council sch changes: shielded connectors, removed SHDN resistor, diode OR for boot, standardized resistors
Parts:
- moved J2 166.7 mm to (201.6, 63.4)
- moved FB2 34.7 mm to (140.5, 111.9), turned to -90 degrees
- moved C24 30.0 mm to (138.9, 111.9), turned to 90 degrees
- moved C23 29.1 mm to (137.3, 111.9), turned to 90 degrees
- moved C26 28.3 mm to (135.7, 111.9), turned to 90 degrees
- moved FB1 27.7 mm to (134.1, 111.9), turned to 90 degrees
Routing:
- net /MCU/NRST: track 10.7 -> 4.58 mm

Commit message: starting routing i think
Parts:
- removed J1, J2: PeripheralCAN, UTSVT_Connectors:Molex_Nano-Fit_105309-xx04_1x04_P2.50mm_Vertical
- removed R42: 10k, Resistor_SMD:R_0603_1608Metric_Pad0.98x0.95mm_HandSolder
- added D21: 1N5819HW, Diode_SMD:D_SOD-123, F.Cu at (159.7, 120.9)
- added D22: 1N5819HW, Diode_SMD:D_SOD-123, F.Cu at (164.8, 120.9)
- added J7: Nanofit 1x05, Connector_Molex:Molex_Nano-Fit_105309-xx05_1x05_P2.50mm_Vertical, F.Cu at (154.3, 60.8)
- added J8: Nanofit 1x05, Connector_Molex:Molex_Nano-Fit_105309-xx05_1x05_P2.50mm_Vertical, F.Cu at (172.1, 60.8)
- 250 uOhm Shunt: renamed from R39
- R24, R5: value 768 -> 1k
- moved TP16 118.7 mm to (131.2, 82.1)
- moved TP10 118.7 mm to (131.2, 74.0)
- moved TP12 118.4 mm to (131.2, 76.7)
- moved TP11 116.2 mm to (128.6, 74.0)
- moved TP14 115.9 mm to (128.6, 76.7)
- moved TP13 113.1 mm to (131.2, 79.4)
- moved TP9 107.5 mm to (146.7, 98.2), turned to 90 degrees
- moved TP4 98.9 mm to (150.9, 98.4), turned to 90 degrees
- moved TP20 85.8 mm to (125.6, 96.9)
- moved TP2 85.5 mm to (176.9, 77.7)
- moved TP19 66.6 mm to (125.7, 109.0)
- moved TP3 57.2 mm to (166.7, 98.4)
- moved D1 56.5 mm to (169.8, 99.1), turned to 180 degrees
- moved R1 56.3 mm to (169.8, 97.5)
- moved TP18 55.2 mm to (125.6, 92.1)
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Connections:
- IC5 pad 7: /Power/PowerProtection/SHDN -> unconnected-(IC5-~{SHDN}-Pad7)
- R34 pad 1: +3.3V -> /MCU/Boot_GPIO
- R34 pad 2: /Power/PowerProtection/SHDN -> GND
- U5 pad 17: unconnected-(U5-PA7-Pad17) -> /MCU/MCU_Boot_GPIO
- U8 pad 14: /MCU/Boot_GPIO -> /MCU/USB_Boot_GPIO
Routing:
- net +3.3V: track 21.5 -> 6.18 mm
- net GND: track 29.4 -> 17.4 mm, vias 1 -> 0
- net /MCU/LED_DISCHARGE: track 9.78 -> 0.00 mm
- net /CAN/CAN1_TX: track 9.59 -> 0.00 mm
- net /CAN/CAN1_RX: track 8.42 -> 0.00 mm
- net /MCU/BOOT0: track 8.41 -> 0.00 mm
- net /MCU/LED_CHARGE: track 7.08 -> 0.00 mm
- net /Current Sense/I_OUT: track 0.81 -> 7.76 mm
- net /Power/ROSC: track 5.49 -> 0.00 mm
- net Net-(U2-BOOT): track 4.43 -> 0.00 mm
- net /Power/PowerProtection/SHDN: track 4.13 -> 0.00 mm
- net /MCU/LED_FAULT: track 4.07 -> 0.00 mm
- net +24V: track 3.71 -> 0.00 mm
- net /MCU/LED_HB: track 3.71 -> 0.00 mm
- net +5V_BUCK: track 3.48 -> 0.00 mm
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- removed copper zone on B.Cu, net (none)
- removed copper zone on B.Cu, net +3.3V
- removed copper zone on B.Cu, net +3.3V HV
- removed copper zone on F.Cu, net +3.3V HV
- removed copper zone on B.Cu, net +5V HV
- removed copper zone on F.Cu, net +5V HV
- removed copper zone on F.Cu, net +5V_BUCK
- removed copper zone on B.Cu, net /Power/PowerProtection/RTN
- removed copper zone on B.Cu, net GND
- removed copper zone on F.Cu, net GND
- removed copper zone on F.Cu, net GND HV
- removed copper zone on F.Cu, net Net-(D6-K)
Other:
- board size 80.6 x 94.4 mm -> 278.1 x 94.4 mm
- board text added: "+ -"
- board text added: "5-3.3V LDO (HV)"
- board text added: "5-3.3V LDO (LV)"
- board text added: "EXT"
- board text added: "GND|CAN_L|CAN_H|24V|SHIELD"
- board text added: "Michael Adeluyi Amperes RevB December 2025"
- board text added: "RX"
- board text added: "SWD|GND|CLK|3v3"
- board text added: "TX"
- board text added: "Termination"
- board text added: "USR"
- board text removed: "5-3.3V LDO"
- board text removed: "<->"
- board text removed: "Michael Adeluyi | Amperes RevB | December 2025"
- board text removed: "Status"
- board text removed: "Term"

Commit message: almost done with routing
Parts:
- added F1: Fuse, Parts:FUSC3216X125N, F.Cu at (164.0, 80.2)
- added TP21: 5V_HV, TestPoint:TestPoint_Pad_1.0x1.0mm, F.Cu at (154.8, 93.7)
- R39: renamed from 250 uOhm Shunt
- moved TP19 59.1 mm to (165.7, 65.6)
- moved TP14 15.9 mm to (125.0, 92.2)
- moved TP16 15.2 mm to (125.0, 96.0)
- moved TP12 13.2 mm to (125.0, 88.4)
- moved TP18 13.1 mm to (125.4, 105.2)
- moved TP17 12.5 mm to (125.0, 99.8)
- moved TP20 12.2 mm to (125.4, 109.1)
- moved TP1 9.24 mm to (132.3, 108.8)
- moved TP11 7.62 mm to (131.0, 81.2)
- moved TP13 6.54 mm to (131.0, 72.9), turned to 0 degrees
- moved D2 5.24 mm to (153.7, 98.8), turned to 180 degrees
- moved C1 4.10 mm to (160.0, 74.1), turned to 90 degrees
- moved C2 3.87 mm to (160.0, 78.0), turned to -90 degrees
- moved D3 3.81 mm to (134.9, 121.2)
- moved TP10 3.64 mm to (131.0, 77.6)
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Connections:
- C1 pad 1: +24V -> Net-(PS1-+VIN)
- C2 pad 1: +24V -> Net-(PS1-+VIN)
- D14 pad 2: /USB/D- -> /USB/D+
- D14 pad 3: /USB/D+ -> /USB/D-
- PS1 pad 2: +24V -> Net-(PS1-+VIN)
Routing:
- net /MCU/ADC1_IN16: track 3.61 -> 91.1 mm, vias 0 -> 2
- net /CAN_HIGH: track 0.00 -> 78.4 mm, vias 0 -> 3
- net /CAN_LOW: track 2.25 -> 79.6 mm, vias 0 -> 2
- net +5V_VBUS: track 0.00 -> 56.1 mm, vias 0 -> 3
- net +3.3V: track 6.18 -> 51.4 mm, vias 0 -> 22
- net /Current Sense/SENSE+: track 0.00 -> 32.1 mm, vias 0 -> 3
- net /MCU/MCU_Boot_GPIO: track 0.00 -> 29.2 mm, vias 0 -> 2
- net /MCU/USART1_TX: track 0.00 -> 27.7 mm, vias 0 -> 2
- net /MCU/USART1_RX: track 0.00 -> 27.6 mm, vias 0 -> 2
- net +3.3V HV: track 6.76 -> 31.9 mm, vias 0 -> 7
- net GND: track 17.4 -> 42.3 mm, vias 0 -> 2
- net +5V_BUCK: track 0.00 -> 24.5 mm, vias 0 -> 2
- net /Current Sense/SHUNT+: track 0.00 -> 23.3 mm
- net /Current Sense/I_OUT: track 7.76 -> 28.0 mm, vias 0 -> 2
- net /ShieldGND: track 0.00 -> 20.1 mm
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- added copper zone on F.Cu, net +24V
- added copper zone on F.Cu, net +24V_Ext
- added copper zone on B.Cu, net +24V_In
- added copper zone on B.Cu, net +3.3V
- added copper zone on F.Cu, net +3.3V
- added copper zone on B.Cu, net +3.3V HV
- added copper zone on B.Cu, net +5V HV
- added copper zone on F.Cu, net +5V HV
- added copper zone on F.Cu, net +5V_BUCK
- added copper zone on B.Cu, net /Power/PowerProtection/RTN
- added copper zone on F.Cu, net /USB/VBUS_IN
- added copper zone on F.Cu, net GND
- added copper zone on F.Cu, net GND HV
- added copper zone on F.Cu, net Net-(D6-K)
- added copper zone on F.Cu, net Net-(PS1-+VIN)
Other:
- board size 278.1 x 94.4 mm -> 168.9 x 94.4 mm
- board text added: "5V HV"
- board text added: "5V MUX"
- board text added: "Buck Fuse"
- board text added: "Current"
- board text added: "HV"
- board text added: "I_OUT"
- board text added: "LV"
- board text added: "Out-"
- board text added: "PP IMON"
- board text added: "Scrut_out"
- board text removed: "5-3.3V LDO (HV)"
- board text removed: "Current Signal"

Commit message: wow
Parts:
- moved TP13 24.5 mm to (142.4, 94.6)
- moved TP17 19.3 mm to (141.3, 89.4)
- moved TP16 19.2 mm to (141.3, 85.9)
- moved TP14 17.9 mm to (141.8, 98.5)
- moved TP12 15.7 mm to (137.0, 98.5)
- moved TP1 9.15 mm to (140.1, 104.0)
- moved TP20 6.43 mm to (131.8, 108.6)
- moved C46 5.64 mm to (136.8, 92.1), turned to 180 degrees
- moved R26 4.75 mm to (125.0, 100.9)
- moved R45 4.75 mm to (125.0, 97.0)
- moved C47 4.75 mm to (125.9, 94.0)
- moved C48 4.75 mm to (125.9, 92.3)
- moved D16 4.75 mm to (133.9, 103.9)
- moved IC3 4.75 mm to (131.6, 87.9)
- moved R27 4.75 mm to (131.2, 93.2)
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Routing:
- net /Current Sense/Scrut-: track 8.54 -> 45.0 mm, vias 0 -> 2
- net /Current Sense/Scrut+: track 8.93 -> 43.0 mm, vias 0 -> 2
- net /Current Sense/Scrut_Out: track 7.51 -> 30.6 mm, vias 0 -> 2
- net /Current Sense/OUT+: track 5.49 -> 24.7 mm, vias 0 -> 2
- net /Current Sense/SENSE+: track 32.1 -> 15.2 mm, vias 3 -> 0
- net /Current Sense/OUT-: track 7.45 -> 23.6 mm, vias 0 -> 2
- net +24V: track 2.59 -> 15.3 mm, vias 0 -> 2
- net /Current Sense/SHUNT-: track 17.7 -> 29.2 mm, vias 0 -> 2
- net +3.3V HV: track 31.9 -> 23.2 mm
- net /Current Sense/SHUNT+: track 23.3 -> 31.6 mm, vias 0 -> 2
- net +1V25: track 18.2 -> 22.2 mm
- net /Current Sense/I_OUT: track 28.0 -> 30.4 mm
- net +3.3V: track 51.4 -> 49.5 mm, vias 22 -> 21
- net /MCU/ADC1_IN16: track 91.1 -> 89.6 mm
- added copper zone on F.Cu, net +3.3V HV
Other:
- board text added: "3V3 LDO"
- board text added: "Current Signal"
- board text added: "HV Buck Fuse"
- board text removed: "5-3.3V LDO (LV)"
- board text removed: "Buck Fuse"
- board text removed: "CAN High"
- board text removed: "CAN Low"
- board text removed: "Current"
- board text removed: "IMON"
- board text removed: "I_Out"
- board text removed: "Scrut_Out"
