File: hardware/PS-HVCarrier.kicad_sch (KiCad schematic)
At the start: 0 parts

Commit message: quote on quote version control
Parts:
- added J2: IMD_Conn, symbol Connector_Generic:Conn_01x08
- added J3: LEM CAB 500-C, LHRS_Connectors:Molex_Nano-Fit_105309-xx05_1x05_P2.50mm_Vertical, symbol lhrs_connectors:CAN_NANO_01x05
- added R6: 0, symbol Device:R
- added R8: 2.1k, symbol Device:R
Connections:
- new net: J3.5 (SHIELD), R6.2
- new net +12V: J3.1 (12V)
- new net +24V: J2.2 (Pin_2)
- new net GND: J2.1 (Pin_1), J2.3 (Pin_3), J3.4 (GND), R6.1, R8.1
- new net IMD_CAN_H: J2.5 (Pin_5)
- new net IMD_CAN_L: J2.6 (Pin_6)
- new net IMD_OKHS: J2.8 (Pin_8), R8.2
- new net LEM_CAN_H: J3.2 (CAN_H)
- new net LEM_CAN_L: J3.3 (CAN_L)
Other:
- added sheet 100PinMCU (100PinMCU.kicad_sch)
- added sheet Current_Sense (Current_Sense.kicad_sch)
- added sheet IMD_CAN_Transceiver (CAN_Transceiver.kicad_sch)
- added sheet Other_CAN_Transceiver (CAN_Transceiver2.0.kicad_sch)
- added sheet Power (Power.kicad_sch)
- added sheet Voltage_Sense (Voltage_Sense.kicad_sch)
