File: hardware/5VBuck_HV.kicad_sch (KiCad schematic)
At the start: 12 parts, among them U1 LMR51635XDDCR

Commit message: labeled + stm32 cube layout
Parts:
- gave numbers to parts that had none: 4
- renumbered C1 to C42, C2 to C43, C3 to C44, C4 to C45, L1 to L3, R1 to R33, R2 to R34, U1 to U6
Changed lines of the file:
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@@
 		(on_board yes)
 		(dnp no)
-		(property "Reference" "L1"
+		(property "Reference" "L3"
 			(at 106.68 48.514 90)
 			(effects
@@
 			(project "5VBuck"
 				(path "/2365a867-6254-4a7c-9718-f325e0bbac5c/904fa10a-747c-46cf-90d1-33d76069dc5d/4a0a5c1f-90e2-4192-9baf-b7e6fdd68fc2"
-					(reference "L1")
+					(reference "L3")
 					(unit 1)
 				)
@@
 		(dnp no)
 		(fields_autoplaced yes)
-		(property "Reference" "R2"
+		(property "Reference" "R34"
 			(at 170.18 49.5299 0)
 			(effects
@@
 			(project "5VBuck"
 				(path "/2365a867-6254-4a7c-9718-f325e0bbac5c/904fa10a-747c-46cf-90d1-33d76069dc5d/4a0a5c1f-90e2-4192-9baf-b7e6fdd68fc2"
-					(reference "R2")
+					(reference "R34")
 					(unit 1)
 				)
@@
 		(dnp no)
 		(fields_autoplaced yes)
-		(property "Reference" "C1"
+		(property "Reference" "C42"
 			(at 40.64 45.7262 0)
 			(effects
@@
 			(project "5VBuck"
 				(path "/2365a867-6254-4a7c-9718-f325e0bbac5c/904fa10a-747c-46cf-90d1-33d76069dc5d/4a0a5c1f-90e2-4192-9baf-b7e6fdd68fc2"
-					(reference "C1")
+					(reference "C42")
 					(unit 1)
 				)
@@
 		(on_board yes)
 		(dnp no)
-		(property "Reference" "TP?"
+		(property "Reference" "TP21"
 			(at 184.15 80.5179 0)
 			(effects
@@
 			(project "5VBuck"
 				(path "/2365a867-6254-4a7c-9718-f325e0bbac5c/904fa10a-747c-46cf-90d1-33d76069dc5d/4a0a5c1f-90e2-4192-9baf-b7e6fdd68fc2"
-					(reference "TP?")
+					(reference "TP21")
 					(unit 1)
 				)
@@
 		(on_board yes)
 		(dnp no)
-		(property "Reference" "C2"
+		(property "Reference" "C43"
 			(at 100.838 40.64 0)
 			(effects
@@
 			(project "5VBuck"
 				(path "/2365a867-6254-4a7c-9718-f325e0bbac5c/904fa10a-747c-46cf-90d1-33d76069dc5d/4a0a5c1f-90e2-4192-9baf-b7e6fdd68fc2"
-					(reference "C2")
+					(reference "C43")
 					(unit 1)
 				)
@@
 		(dnp no)
 		(fields_autoplaced yes)
-		(property "Reference" "U1"
+		(property "Reference" "U6"
 			(at 73.66 31.75 0)
 			(effects
@@
 			(project "5VBuck"
 				(path "/2365a867-6254-4a7c-9718-f325e0bbac5c/904fa10a-747c-46cf-90d1-33d76069dc5d/4a0a5c1f-90e2-4192-9baf-b7e6fdd68fc2"
-					(reference "U1")
+					(reference "U6")
 					(unit 1)
 				)
@@
 		(on_board yes)
 		(dnp no)
-		(property "Reference" "TP?"
+		(property "Reference" "TP19"
 			(at 171.45 80.5179 0)
 			(effects
@@
 			(project "5VBuck"
 				(path "/2365a867-6254-4a7c-9718-f325e0bbac5c/904fa10a-747c-46cf-90d1-33d76069dc5d/4a0a5c1f-90e2-4192-9baf-b7e6fdd68fc2"
-					(reference "TP?")
+					(reference "TP19")
 					(unit 1)
 				)
@@
 		(dnp no)
 		(fields_autoplaced yes)
-		(property "Reference" "#FLG01"
+		(property "Reference" "#FLG09"
 			(at 93.98 40.005 0)
 			(effects
@@
 			(project "5VBuck"
 				(path "/2365a867-6254-4a7c-9718-f325e0bbac5c/904fa10a-747c-46cf-90d1-33d76069dc5d/4a0a5c1f-90e2-4192-9baf-b7e6fdd68fc2"
-					(reference "#FLG01")
+					(reference "#FLG09")
 					(unit 1)
 				)
@@
 		(on_board yes)
 		(dnp no)
-		(property "Reference" "TP?"
+		(property "Reference" "TP22"
 			(at 184.15 93.2179 0)
 			(effects
@@
 			(project "5VBuck"
 				(path "/2365a867-6254-4a7c-9718-f325e0bbac5c/904fa10a-747c-46cf-90d1-33d76069dc5d/4a0a5c1f-90e2-4192-9baf-b7e6fdd68fc2"
-					(reference "TP?")
+					(reference "TP22")
 					(unit 1)
 				)
@@
 		(dnp no)
 		(fields_autoplaced yes)
-		(property "Reference" "C4"
+		(property "Reference" "C45"
 			(at 129.54 49.5362 0)
 			(effects
@@
 			(project "5VBuck"
 				(path "/2365a867-6254-4a7c-9718-f325e0bbac5c/904fa10a-747c-46cf-90d1-33d76069dc5d/4a0a5c1f-90e2-4192-9baf-b7e6fdd68fc2"
-					(reference "C4")
+					(reference "C45")
 					(unit 1)
 				)
@@
 		(on_board yes)
 		(dnp no)
-		(property "Reference" "#FLG02"
+		(property "Reference" "#FLG010"
 			(at 93.98 45.085 0)
 			(effects
@@
 			(project "5VBuck"
 				(path "/2365a867-6254-4a7c-9718-f325e0bbac5c/904fa10a-747c-46cf-90d1-33d76069dc5d/4a0a5c1f-90e2-4192-9baf-b7e6fdd68fc2"
-					(reference "#FLG02")
+					(reference "#FLG010")
 					(unit 1)
 				)
@@
 		(dnp no)
 		(fields_autoplaced yes)
-		(property "Reference" "R1"
+		(property "Reference" "R33"
 			(at 170.18 41.9099 0)
 			(effects
@@
 			(project "5VBuck"
 				(path "/2365a867-6254-4a7c-9718-f325e0bbac5c/904fa10a-747c-46cf-90d1-33d76069dc5d/4a0a5c1f-90e2-4192-9baf-b7e6fdd68fc2"
-					(reference "R1")
+					(reference "R33")
 					(unit 1)
 				)
@@
 		(dnp no)
 		(fields_autoplaced yes)
-		(property "Reference" "C3"
+		(property "Reference" "C44"
 			(at 118.11 49.5362 0)
 			(effects
@@
 			(project "5VBuck"
 				(path "/2365a867-6254-4a7c-9718-f325e0bbac5c/904fa10a-747c-46cf-90d1-33d76069dc5d/4a0a5c1f-90e2-4192-9baf-b7e6fdd68fc2"
-					(reference "C3")
+					(reference "C44")
 					(unit 1)
 				)
@@
 		(on_board yes)
 		(dnp no)
-		(property "Reference" "TP?"
+		(property "Reference" "TP20"
 			(at 171.45 93.2179 0)
 			(effects
@@
 			(project "5VBuck"
 				(path "/2365a867-6254-4a7c-9718-f325e0bbac5c/904fa10a-747c-46cf-90d1-33d76069dc5d/4a0a5c1f-90e2-4192-9baf-b7e6fdd68fc2"
-					(reference "TP?")
-					(unit 1)
-				)
+					(reference "TP20")
+					(unit 1)
+				)

Commit message: added debug led
Parts:
- renumbered R33 to R40, R34 to R41, TP19 to TP20, TP20 to TP21, TP21 to TP22, TP22 to TP23, U6 to U7
Changed lines of the file:
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@@
 		(dnp no)
 		(fields_autoplaced yes)
-		(property "Reference" "R34"
+		(property "Reference" "R41"
 			(at 170.18 49.5299 0)
 			(effects
@@
 			(project "5VBuck"
 				(path "/2365a867-6254-4a7c-9718-f325e0bbac5c/904fa10a-747c-46cf-90d1-33d76069dc5d/4a0a5c1f-90e2-4192-9baf-b7e6fdd68fc2"
-					(reference "R34")
+					(reference "R41")
 					(unit 1)
 				)
@@
 		(on_board yes)
 		(dnp no)
-		(property "Reference" "TP21"
+		(property "Reference" "TP22"
 			(at 184.15 80.5179 0)
 			(effects
@@
 			(project "5VBuck"
 				(path "/2365a867-6254-4a7c-9718-f325e0bbac5c/904fa10a-747c-46cf-90d1-33d76069dc5d/4a0a5c1f-90e2-4192-9baf-b7e6fdd68fc2"
-					(reference "TP21")
+					(reference "TP22")
 					(unit 1)
 				)
@@
 		(dnp no)
 		(fields_autoplaced yes)
-		(property "Reference" "U6"
+		(property "Reference" "U7"
 			(at 73.66 31.75 0)
 			(effects
@@
 			(project "5VBuck"
 				(path "/2365a867-6254-4a7c-9718-f325e0bbac5c/904fa10a-747c-46cf-90d1-33d76069dc5d/4a0a5c1f-90e2-4192-9baf-b7e6fdd68fc2"
-					(reference "U6")
+					(reference "U7")
 					(unit 1)
 				)
@@
 		(on_board yes)
 		(dnp no)
-		(property "Reference" "TP19"
+		(property "Reference" "TP20"
 			(at 171.45 80.5179 0)
 			(effects
@@
 			(project "5VBuck"
 				(path "/2365a867-6254-4a7c-9718-f325e0bbac5c/904fa10a-747c-46cf-90d1-33d76069dc5d/4a0a5c1f-90e2-4192-9baf-b7e6fdd68fc2"
-					(reference "TP19")
+					(reference "TP20")
 					(unit 1)
 				)
@@
 		(on_board yes)
 		(dnp no)
-		(property "Reference" "TP22"
+		(property "Reference" "TP23"
 			(at 184.15 93.2179 0)
 			(effects
@@
 			(project "5VBuck"
 				(path "/2365a867-6254-4a7c-9718-f325e0bbac5c/904fa10a-747c-46cf-90d1-33d76069dc5d/4a0a5c1f-90e2-4192-9baf-b7e6fdd68fc2"
-					(reference "TP22")
+					(reference "TP23")
 					(unit 1)
 				)
@@
 		(dnp no)
 		(fields_autoplaced yes)
-		(property "Reference" "R33"
+		(property "Reference" "R40"
 			(at 170.18 41.9099 0)
 			(effects
@@
 			(project "5VBuck"
 				(path "/2365a867-6254-4a7c-9718-f325e0bbac5c/904fa10a-747c-46cf-90d1-33d76069dc5d/4a0a5c1f-90e2-4192-9baf-b7e6fdd68fc2"
-					(reference "R33")
+					(reference "R40")
 					(unit 1)
 				)
@@
 		(on_board yes)
 		(dnp no)
-		(property "Reference" "TP20"
+		(property "Reference" "TP21"
 			(at 171.45 93.2179 0)
 			(effects
@@
 			(project "5VBuck"
 				(path "/2365a867-6254-4a7c-9718-f325e0bbac5c/904fa10a-747c-46cf-90d1-33d76069dc5d/4a0a5c1f-90e2-4192-9baf-b7e6fdd68fc2"
-					(reference "TP20")
-					(unit 1)
-				)
+					(reference "TP21")
+					(unit 1)
+				)
