File: hardware/AMC1311.kicad_sch (KiCad schematic)
At the start: 39 parts, among them U11 AMC1311QDWVRQ1, U12 AMC1311QDWVRQ1, U13 AMC1311QDWVRQ1

Commit message: labeled + stm32 cube layout
Parts:
- renumbered C63 to C75, C64 to C76, C65 to C77, C66 to C78, C67 to C79, C68 to C80, C69 to C81, C70 to C82, C71 to C83, C72 to C84, C73 to C85, C74 to C86, C75 to C87, C76 to C88, C77 to C89, C78 to C90, C79 to C91, C80 to C92

Commit message: added debug led
Parts:
- renumbered R56 to R63, R57 to R64, R58 to R65, R59 to R66, R60 to R67, R61 to R68, R62 to R69, R63 to R70, R64 to R71, R65 to R72, R66 to R73, R67 to R74, R68 to R75, R69 to R76, R70 to R77, R71 to R78, R72 to R79, R73 to R80, U11 to U12, U12 to U13, U13 to U14
