File: hardware/12VBuck.kicad_sch (KiCad schematic)
At the start: 12 parts, among them U3 LMR51635XDDCR

Commit message: labeled + stm32 cube layout
Parts:
- renumbered C12 to C10, C9 to C11, C10 to C12, C11 to C9, L3 to L1, R1 to R6, R4 to R7, TP9 to TP11, TP10 to TP12, TP11 to TP13, TP12 to TP14, U3 to U1
Changed lines of the file:
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@@
 		(dnp no)
 		(fields_autoplaced yes)
-		(property "Reference" "C9"
+		(property "Reference" "C11"
 			(at 172.72 88.9062 0)
 			(effects
@@
 			(project "PS-Buck"
 				(path "/2365a867-6254-4a7c-9718-f325e0bbac5c/904fa10a-747c-46cf-90d1-33d76069dc5d/3d7c722a-11ca-4e65-b53b-d133826eeb8d"
-					(reference "C9")
+					(reference "C11")
 					(unit 1)
 				)
@@
 		(dnp no)
 		(fields_autoplaced yes)
-		(property "Reference" "#FLG013"
+		(property "Reference" "#FLG02"
 			(at 149.86 79.375 0)
 			(effects
@@
 			(project "PS-Buck"
 				(path "/2365a867-6254-4a7c-9718-f325e0bbac5c/904fa10a-747c-46cf-90d1-33d76069dc5d/3d7c722a-11ca-4e65-b53b-d133826eeb8d"
-					(reference "#FLG013")
+					(reference "#FLG02")
 					(unit 1)
 				)
@@
 		(dnp no)
 		(fields_autoplaced yes)
-		(property "Reference" "C11"
+		(property "Reference" "C9"
 			(at 96.52 85.0962 0)
 			(effects
@@
 			(project "PS-Buck"
 				(path "/2365a867-6254-4a7c-9718-f325e0bbac5c/904fa10a-747c-46cf-90d1-33d76069dc5d/3d7c722a-11ca-4e65-b53b-d133826eeb8d"
-					(reference "C11")
+					(reference "C9")
 					(unit 1)
 				)
@@
 		(on_board yes)
 		(dnp no)
-		(property "Reference" "TP9"
+		(property "Reference" "TP11"
 			(at 229.87 123.6979 0)
 			(effects
@@
 			(project "PowerPath"
 				(path "/2365a867-6254-4a7c-9718-f325e0bbac5c/904fa10a-747c-46cf-90d1-33d76069dc5d/3d7c722a-11ca-4e65-b53b-d133826eeb8d"
-					(reference "TP9")
+					(reference "TP11")
 					(unit 1)
 				)
@@
 		(on_board yes)
 		(dnp no)
-		(property "Reference" "L3"
+		(property "Reference" "L1"
 			(at 161.29 87.884 90)
 			(effects
@@
 			(project "PS-Buck"
 				(path "/2365a867-6254-4a7c-9718-f325e0bbac5c/904fa10a-747c-46cf-90d1-33d76069dc5d/3d7c722a-11ca-4e65-b53b-d133826eeb8d"
-					(reference "L3")
+					(reference "L1")
 					(unit 1)
 				)
@@
 		(on_board yes)
 		(dnp no)
-		(property "Reference" "TP11"
+		(property "Reference" "TP13"
 			(at 242.57 123.6979 0)
 			(effects
@@
 			(project "PowerPath"
 				(path "/2365a867-6254-4a7c-9718-f325e0bbac5c/904fa10a-747c-46cf-90d1-33d76069dc5d/3d7c722a-11ca-4e65-b53b-d133826eeb8d"
-					(reference "TP11")
+					(reference "TP13")
 					(unit 1)
 				)
@@
 		(on_board yes)
 		(dnp no)
-		(property "Reference" "TP10"
+		(property "Reference" "TP12"
 			(at 229.87 136.3979 0)
 			(effects
@@
 			(project "PowerPath"
 				(path "/2365a867-6254-4a7c-9718-f325e0bbac5c/904fa10a-747c-46cf-90d1-33d76069dc5d/3d7c722a-11ca-4e65-b53b-d133826eeb8d"
-					(reference "TP10")
+					(reference "TP12")
 					(unit 1)
 				)
@@
 		(dnp no)
 		(fields_autoplaced yes)
-		(property "Reference" "U3"
+		(property "Reference" "U1"
 			(at 129.54 71.12 0)
 			(effects
@@
 			(project "PS-Buck"
 				(path "/2365a867-6254-4a7c-9718-f325e0bbac5c/904fa10a-747c-46cf-90d1-33d76069dc5d/3d7c722a-11ca-4e65-b53b-d133826eeb8d"
-					(reference "U3")
+					(reference "U1")
 					(unit 1)
 				)
@@
 		(on_board yes)
 		(dnp no)
-		(property "Reference" "TP12"
+		(property "Reference" "TP14"
 			(at 242.57 136.3979 0)
 			(effects
@@
 			(project "PowerPath"
 				(path "/2365a867-6254-4a7c-9718-f325e0bbac5c/904fa10a-747c-46cf-90d1-33d76069dc5d/3d7c722a-11ca-4e65-b53b-d133826eeb8d"
-					(reference "TP12")
+					(reference "TP14")
 					(unit 1)
 				)
@@
 		(dnp no)
 		(fields_autoplaced yes)
-		(property "Reference" "C10"
+		(property "Reference" "C12"
 			(at 184.15 88.9062 0)
 			(effects
@@
 			(project "PS-Buck"
 				(path "/2365a867-6254-4a7c-9718-f325e0bbac5c/904fa10a-747c-46cf-90d1-33d76069dc5d/3d7c722a-11ca-4e65-b53b-d133826eeb8d"
-					(reference "C10")
+					(reference "C12")
 					(unit 1)
 				)
@@
 		(dnp no)
 		(fields_autoplaced yes)
-		(property "Reference" "#FLG015"
+		(property "Reference" "#FLG04"
 			(at 181.61 84.455 0)
 			(effects
@@
 			(project "PS-Buck"
 				(path "/2365a867-6254-4a7c-9718-f325e0bbac5c/904fa10a-747c-46cf-90d1-33d76069dc5d/3d7c722a-11ca-4e65-b53b-d133826eeb8d"
-					(reference "#FLG015")
+					(reference "#FLG04")
 					(unit 1)
 				)
@@
 		(dnp no)
 		(fields_autoplaced yes)
-		(property "Reference" "#FLG011"
+		(property "Reference" "#FLG01"
 			(at 88.9 79.375 0)
 			(effects
@@
 			(project "PS-Buck"
 				(path "/2365a867-6254-4a7c-9718-f325e0bbac5c/904fa10a-747c-46cf-90d1-33d76069dc5d/3d7c722a-11ca-4e65-b53b-d133826eeb8d"
-					(reference "#FLG011")
+					(reference "#FLG01")
 					(unit 1)
 				)
@@
 		(on_board yes)
 		(dnp no)
-		(property "Reference" "C12"
+		(property "Reference" "C10"
 			(at 156.718 80.01 0)
 			(effects
@@
 			(project "PS-Buck"
 				(path "/2365a867-6254-4a7c-9718-f325e0bbac5c/904fa10a-747c-46cf-90d1-33d76069dc5d/3d7c722a-11ca-4e65-b53b-d133826eeb8d"
-					(reference "C12")
+					(reference "C10")
 					(unit 1)
 				)
@@
 		(on_board yes)
 		(dnp no)
-		(property "Reference" "#FLG014"
+		(property "Reference" "#FLG03"
 			(at 149.86 84.455 0)
 			(effects
@@
 			(project "PS-Buck"
 				(path "/2365a867-6254-4a7c-9718-f325e0bbac5c/904fa10a-747c-46cf-90d1-33d76069dc5d/3d7c722a-11ca-4e65-b53b-d133826eeb8d"
-					(reference "#FLG014")
+					(reference "#FLG03")
 					(unit 1)
 				)
@@
 		(dnp no)
 		(fields_autoplaced yes)
-		(property "Reference" "R1"
+		(property "Reference" "R6"
 			(at 227.33 85.0899 0)
 			(effects
@@
 			(project "PS-Buck"
 				(path "/2365a867-6254-4a7c-9718-f325e0bbac5c/904fa10a-747c-46cf-90d1-33d76069dc5d/3d7c722a-11ca-4e65-b53b-d133826eeb8d"
-					(reference "R1")
+					(reference "R6")
 					(unit 1)
 				)
@@
 		(dnp no)
 		(fields_autoplaced yes)
-		(property "Reference" "R4"
+		(property "Reference" "R7"
 			(at 227.33 92.7099 0)
 			(effects
@@
 			(project "PS-Buck"
 				(path "/2365a867-6254-4a7c-9718-f325e0bbac5c/904fa10a-747c-46cf-90d1-33d76069dc5d/3d7c722a-11ca-4e65-b53b-d133826eeb8d"
-					(reference "R4")
-					(unit 1)
-				)
+					(reference "R7")
+					(unit 1)
+				)

Commit message: added debug led
Parts:
- renumbered R6 to R13, R7 to R14
Changed lines of the file:
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@@
 		(dnp no)
 		(fields_autoplaced yes)
-		(property "Reference" "R6"
+		(property "Reference" "R13"
 			(at 227.33 85.0899 0)
 			(effects
@@
 			(project "PS-Buck"
 				(path "/2365a867-6254-4a7c-9718-f325e0bbac5c/904fa10a-747c-46cf-90d1-33d76069dc5d/3d7c722a-11ca-4e65-b53b-d133826eeb8d"
-					(reference "R6")
+					(reference "R13")
 					(unit 1)
 				)
@@
 		(dnp no)
 		(fields_autoplaced yes)
-		(property "Reference" "R7"
+		(property "Reference" "R14"
 			(at 227.33 92.7099 0)
 			(effects
@@
 			(project "PS-Buck"
 				(path "/2365a867-6254-4a7c-9718-f325e0bbac5c/904fa10a-747c-46cf-90d1-33d76069dc5d/3d7c722a-11ca-4e65-b53b-d133826eeb8d"
-					(reference "R7")
+					(reference "R14")
 					(unit 1)
 				)
