File: hardware/Current_Sense.kicad_sch (KiCad schematic)
At the start: 17 parts, among them J4 CAB 500/BPS CAN, J5 LZSR 80-P

Commit message: added calcs, cleaned up, addressed comments
Parts:
- removed J4: CAB 500/BPS CAN, LHRS_Connectors:Molex_Nano-Fit_105309-xx05_1x05_P2.50mm_Vertical, symbol lhrs_connectors:CAN_NANO_01x05
- added C38, C40: 100n, symbol Device:C
- added C39: 1n, symbol Device:C
- added C41: 0.1u, symbol Device:C
- added D17, D18: TVS, Diode_SMD:D_SOD-123F, symbol Device:D_Zener
- added J10: SSA-2-100A, symbol lhrs_connectors:CAN_NANO_01x05
- added J9: SSA-2-100A, LHRS_Connectors:Molex_Nano-Fit_105309-xx05_1x05_P2.50mm_Vertical, symbol lhrs_connectors:CAN_NANO_01x05
- added R35, R36: 100, symbol Device:R
- added R37, R38, R41: 10k, symbol Device:R
- added R40: 20k, symbol Device:R
- added TP16: SHUNT_ADC, symbol Connector:TestPoint
- added TP?: HALL_OCD, symbol Connector:TestPoint
- added TP?: HALL_UREF, symbol Connector:TestPoint
- added TP?: HALL_UOUT, symbol Connector:TestPoint
- added TP?: SHUNT_OUTN, symbol Connector:TestPoint
- added TP?: SHUNT_OUTP, symbol Connector:TestPoint
- added U5: TLV9002QDRQ1, Package_SO:SOIC-8_3.9x4.9mm_P1.27mm, symbol lhrs_misc:TLV9002QDRQ1
- R39: value 0 -> 20k; now fitted
- renumbered C38 to C34, C39 to C35, C40 to C36, C41 to C37, D15 to D13, D16 to D14, D17 to D15, D18 to D16, J5 to J8, R33 to R29, R34 to R30, R35 to R31, R36 to R32, R37 to R33, R38 to R34
Connections:
- net +3V3 is gone; now on net 3v3+: D13.1 (K), D14.1 (K)
- net GND: now also C40.2, C41.2, D18.2 (A), J9.3 (GND), R40.2, U5.4 (V-); no longer R39.1
- net LZSR_OCD: now also TP?.1
- net LZSR_UOUT: now also TP?.1
- net LZSR_UREF: now also TP?.1
- net 3v3+: now reaches R39.2
- net 3v3+: now also C41.1, J9.4 (PWR), U5.8 (V+)
- new net: C39.2, R37.1, R41.2, TP?.1, U5.2 (-)
- new net: C38.1, R35.1, R37.2
- new net: C38.2, R36.1, R38.2
- new net: J9.2 (Out+), R36.2
- new net: J9.1 (Out-), R35.2
- new net: C39.1, R41.1, U5.1, U5.6 (-)
- new net +3v3: D17.1 (K)
- new net SHUNT ADC: D17.2 (A), D18.1 (K), TP16.1, U5.5 (+), U5.7
- new net SHUNT ADC UREF: C40.1, R38.1, R39.1, R40.1, TP?.1, U5.3 (+)
- no-connect marks 0 -> 4
Other:
- removed sheet Shunt Design
- note added: "+30A Uref = 2.5V Uout = 2.734V"
- note added: "+30A Vout+ = 1.8375V Vout- = 1.4625V Vdiff = +0.375V Shunt_ADC = 2.025V"
- note added: "-70A Uref = 2.5V Uout = 1.953V"
- note added: "-70A Vout+ = 1.2125V Vout- = 2.0875V Vdiff = -0.875V Shunt_ADC = 0.775V"
- note added: "0A Uref = 2.5V Uout = 2.5V"
- note added: "0A Vout+ = 1.650V, Vout- = 1.650V Vdiff = 0V Shunt_ADC = 1.650V"
- note added: "Bias to set common mode V = 1.65V"
- note added: "LZSR 80-P Calc"
- note added: "Mating Connector (added for BOM)"
- note added: "Mating connectors: 4 pin female: 1053071204 20-22 AWG female crimps: 1053002200 4-Pin TPA locking: 1053251004"
- note added: "Mating to Board Conn"
- note added: "Nominal Sensitivity (Sn) = 7.813mV/A Reference Voltage (Uref) = 2.5V Uout = Uref + (Sn * Ip) Ip = Uout - Uref/ Sn Ip = Uout - Uref / 7.813mV/A"
- note added: "Offset Error: 3ppm/K = 0.0003%/C = 0.000003 per K or C Offset % = 0.000003 * 50 = 0.00015 (0.015%) Current error = 80A * 0.00015 = +-12mA Offset errorTemp driftV_offset = Vout_FS * TC * Temp change Sensitivity drift = 75ppm/K Gain error = 75 * 10^-6 * 50 = 0.375% Current error = 80A * 0.00375 = +-300mA +-300mA + +-12mA = +-312mA"
- note added: "Resolution = 160A/2^12 = 0.0390A/LSB (39.0mA per step)"
- note added: "Resolution = 200A/2^12 = 0.0488A/LSB (48.8mA per step)"
- note added: "SSA-2-100A SHUNT"
- note added: "Sensitivity: 12.5mV/A Common mode = 1.44V from sensor Op-amp common monde = 1.65V V_diff = I_input * 0.0125V/A Vout+ = 1.65 + V_diff/2 Vout- = 1.65 - V_diff/2 Op-amp gain = 1.0"
- note added: "Shunt Calc"
- note added: "Temp Drift: I_gain_drift = I_measure * TCs * Temp Change 30 ppm/C = 30/1,000,000 = 0.0030%/C Gain error % = 0.000030*50 = 0.0015 = 0.15% Current error @ max = 100A * 0.0015 = +-150mA"
- note added: "Unity Gain Amp"
- note added: "V(bias) = Vcc/2 = 3.3/2 = 1.65V 1.65 = 3.3 * (R40/R40+R39) = 0.5V R(bias) = must maintain gain of 1"
- note removed: "CAB 500 Conn"
- note removed: "I = (Vuout - Vuref) / (7.813mV/A)"
- moved on the sheet: C34, C35, C36, C37, D13, D14, D15, D16, J8, R29, R30, R31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

Commit message: added USB power mux
Parts:
- gave numbers to parts that had none: 5
- renumbered C34 to C35, C35 to C36, C36 to C37, C37 to C38, C38 to C39, C39 to C41, C41 to C42, D13 to D15, D14 to D16, D15 to D17, D16 to D18, D17 to D19, D18 to D20, TP16 to TP20, U5 to U4

Commit message: added STM 32 screenshot
Connections:
- net 3v3+: now also R31.2
- net GND: no longer R31.1
- net LZSR OCD: now also R31.1; no longer R31.2
Other:
- moved on the sheet: R31, R32
Changed lines of the file:
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@@
 	)
 	(junction
-		(at 43.18 85.09)
+		(at 55.88 85.09)
 		(diameter 0)
 		(color 0 0 0 0)
@@
 	(wire
 		(pts
-			(xy 53.34 85.09) (xy 77.47 85.09)
+			(xy 66.04 85.09) (xy 77.47 85.09)
 		)
 		(stroke
@@
 	(wire
 		(pts
-			(xy 43.18 85.09) (xy 45.72 85.09)
+			(xy 55.88 85.09) (xy 58.42 85.09)
 		)
 		(stroke
@@
 	(wire
 		(pts
-			(xy 43.18 92.71) (xy 43.18 93.98)
+			(xy 55.88 83.82) (xy 55.88 85.09)
 		)
 		(stroke
@@
 	(wire
 		(pts
-			(xy 34.29 85.09) (xy 43.18 85.09)
+			(xy 34.29 85.09) (xy 55.88 85.09)
 		)
 		(stroke
@@
 	(hierarchical_label "3v3+"
 		(shape input)
+		(at 55.88 76.2 90)
+		(effects
+			(font
+				(size 1.27 1.27)
+			)
+			(justify left)
+		)
+	)
+	(hierarchical_label "3v3+"
+		(shape input)
 		(at 50.8 52.07 90)
 		(effects
@@
 		(property "Value" "GND"
 			(at 43.18 77.47 0)
+			(hide yes)
 			(show_name no)
 			(do_not_autoplace no)
@@
 	(symbol
 		(lib_id "Device:R")
-		(at 43.18 88.9 180)
+		(at 55.88 80.01 180)
 		(unit 1)
 		(body_style 1)
@@
 		(dnp no)
 		(property "Reference" "R31"
-			(at 37.084 87.63 0)
+			(at 49.784 78.74 0)
 			(show_name no)
 			(do_not_autoplace no)
@@
 		)
 		(property "Value" "20k"
-			(at 37.084 90.17 0)
+			(at 49.784 81.28 0)
 			(show_name no)
 			(do_not_autoplace no)
@@
 		)
 		(property "Footprint" ""
-			(at 44.958 88.9 90)
+			(at 57.658 80.01 90)
 			(hide yes)
 			(show_name no)
@@
 		)
 		(property "Datasheet" ""
-			(at 43.18 88.9 0)
+			(at 55.88 80.01 0)
 			(hide yes)
 			(show_name no)
@@
 		)
 		(property "Description" "Resistor"
-			(at 43.18 88.9 0)
+			(at 55.88 80.01 0)
 			(hide yes)
 			(show_name no)
@@
 	)
 	(symbol
-		(lib_id "power:GND")
-		(at 43.18 93.98 0)
-		(unit 1)
-		(body_style 1)
-		(exclude_from_sim no)
-		(in_bom yes)
-		(on_board yes)
-		(in_pos_files yes)
-		(dnp no)
-		(fields_autoplaced yes)
-		(property "Reference" "#PWR023"
-			(at 43.18 100.33 0)
-			(hide yes)
-			(show_name no)
-			(do_not_autoplace no)
-			(effects
-				(font
-					(size 1.27 1.27)
-				)
-			)
-		)
-		(property "Value" "GND"
-			(at 43.18 99.06 0)
-			(hide yes)
-			(show_name no)
-			(do_not_autoplace no)
-			(effects
-				(font
-					(size 1.27 1.27)
-				)
-			)
-		)
-		(property "Footprint" ""
-			(at 43.18 93.98 0)
-			(hide yes)
-			(show_name no)
-			(do_not_autoplace no)
-			(effects
-				(font
-					(size 1.27 1.27)
-				)
-			)
-		)
-		(property "Datasheet" ""
-			(at 43.18 93.98 0)
-			(hide yes)
-			(show_name no)
-			(do_not_autoplace no)
-			(effects
-				(font
-					(size 1.27 1.27)
-				)
-			)
-		)
-		(property "Description" "Power symbol creates a global label with name \"GND\" , ground"
-			(at 43.18 93.98 0)
-			(hide yes)
-			(show_name no)
-			(do_not_autoplace no)
-			(effects
-				(font
-					(size 1.27 1.27)
-				)
-			)
-		)
-		(pin "1"
-		)
-		(instances
-			(project "PS-HVCarrier"
-				(path "/2365a867-6254-4a7c-9718-f325e0bbac5c/c64f1e33-0c51-411c-bbbf-0af7b620c655"
-					(reference "#PWR023")
-					(unit 1)
-				)
-			)
-		)
-	)
-	(symbol
 		(lib_id "Device:D_Schottky")
 		(at 50.8 29.21 270)
@@
 	(symbol
 		(lib_id "Device:R")
-		(at 49.53 85.09 90)
+		(at 62.23 85.09 90)
 		(unit 1)
 		(body_style 1)
@@
 		(dnp no)
 		(property "Reference" "R32"
-			(at 49.53 78.74 90)
+			(at 62.23 78.74 90)
 			(show_name no)
 			(do_not_autoplace no)
@@
 		)
 		(property "Value" "10k"
-			(at 49.53 81.28 90)
+			(at 62.23 81.28 90)
 			(show_name no)
 			(do_not_autoplace no)
@@
 		)
 		(property "Footprint" ""
-			(at 49.53 86.868 90)
+			(at 62.23 86.868 90)
 			(hide yes)
 			(show_name no)
@@
 		)
 		(property "Datasheet" ""
-			(at 49.53 85.09 0)
+			(at 62.23 85.09 0)
 			(hide yes)
 			(show_name no)
@@
 		)
 		(property "Description" "Resistor"
-			(at 49.53 85.09 0)
+			(at 62.23 85.09 0)
 			(hide yes)
 			(show_name no)

Commit message: fixed ERC warnings
Parts:
- renumbered R33 to R32, R34 to R33, R32 to R34, TP15 to TP16, TP16 to TP17, TP17 to TP18, TP18 to TP19, TP19 to TP20, TP20 to TP21
Connections:
- net 3v3+ is gone; now on net +3v3: C42.1, D15.1 (K), D16.1 (K), J9.4 (PWR), R31.2, R39.2, U4.8 (V+)
Changed lines of the file:
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@@
 		)
 	)
-	(hierarchical_label "3v3+"
-		(shape input)
-		(at 246.38 69.85 90)
+	(hierarchical_label "LZSR UOUT"
+		(shape output)
+		(at 33.02 33.02 180)
 		(effects
 			(font
 				(size 1.27 1.27)
 			)
-			(justify left)
+			(justify right)
 		)
 	)
-	(hierarchical_label "LZSR UOUT"
-		(shape output)
-		(at 33.02 33.02 180)
+	(hierarchical_label "+3v3"
+		(shape input)
+		(at 50.8 52.07 90)
 		(effects
 			(font
 				(size 1.27 1.27)
 			)
-			(justify right)
+			(justify left)
 		)
 	)
-	(hierarchical_label "3v3+"
+	(hierarchical_label "+3v3"
 		(shape input)
 		(at 171.45 69.85 180)
@@
 		)
 	)
-	(hierarchical_label "3v3+"
+	(hierarchical_label "+3v3"
 		(shape input)
-		(at 55.88 76.2 90)
+		(at 50.8 25.4 90)
 		(effects
 			(font
@@
 		)
 	)
-	(hierarchical_label "3v3+"
-		(shape input)
-		(at 50.8 52.07 90)
+	(hierarchical_label "LZSR UREF"
+		(shape output)
+		(at 33.02 60.96 180)
 		(effects
 			(font
 				(size 1.27 1.27)
 			)
-			(justify left)
+			(justify right)
 		)
 	)
-	(hierarchical_label "LZSR UREF"
-		(shape output)
-		(at 33.02 60.96 180)
+	(hierarchical_label "+3v3"
+		(shape input)
+		(at 55.88 76.2 90)
 		(effects
 			(font
 				(size 1.27 1.27)
 			)
-			(justify right)
+			(justify left)
 		)
 	)
-	(hierarchical_label "3v3+"
+	(hierarchical_label "+3v3"
 		(shape input)
-		(at 144.78 60.96 0)
+		(at 246.38 69.85 90)
 		(effects
 			(font
@@
 		)
 	)
-	(hierarchical_label "SHUNT ADC"
-		(shape output)
-		(at 250.19 53.34 0)
+	(hierarchical_label "+3v3"
+		(shape input)
+		(at 144.78 60.96 0)
 		(effects
 			(font
@@
 		)
 	)
-	(hierarchical_label "3v3+"
-		(shape input)
-		(at 50.8 25.4 90)
+	(hierarchical_label "SHUNT ADC"
+		(shape output)
+		(at 250.19 53.34 0)
 		(effects
 			(font
@@
 		(dnp no)
 		(fields_autoplaced yes)
-		(property "Reference" "R34"
+		(property "Reference" "R33"
 			(at 62.23 54.61 90)
 			(show_name no)
@@
 			(project "PS-HVCarrier"
 				(path "/2365a867-6254-4a7c-9718-f325e0bbac5c/c64f1e33-0c51-411c-bbbf-0af7b620c655"
-					(reference "R34")
+					(reference "R33")
 					(unit 1)
 				)
@@
 		(dnp no)
 		(fields_autoplaced yes)
-		(property "Reference" "#PWR025"
+		(property "Reference" "#PWR024"
 			(at 153.67 63.5 0)
 			(hide yes)
@@
 			(project "PS-HVCarrier"
 				(path "/2365a867-6254-4a7c-9718-f325e0bbac5c/c64f1e33-0c51-411c-bbbf-0af7b620c655"
-					(reference "#PWR025")
+					(reference "#PWR024")
 					(unit 1)
 				)
@@
 		(in_pos_files yes)
 		(dnp no)
-		(property "Reference" "TP17"
+		(property "Reference" "TP18"
 			(at 80.01 80.5179 0)
 			(hide yes)
@@
 			(project "PS-HVCarrier"
 				(path "/2365a867-6254-4a7c-9718-f325e0bbac5c/c64f1e33-0c51-411c-bbbf-0af7b620c655"
-					(reference "TP17")
+					(reference "TP18")
 					(unit 1)
 				)
@@
 		(in_pos_files yes)
 		(dnp no)
-		(property "Reference" "TP16"
+		(property "Reference" "TP17"
 			(at 80.01 56.3879 0)
 			(hide yes)
@@
 			(project "PS-HVCarrier"
 				(path "/2365a867-6254-4a7c-9718-f325e0bbac5c/c64f1e33-0c51-411c-bbbf-0af7b620c655"
-					(reference "TP16")
+					(reference "TP17")
 					(unit 1)
 				)
@@
 		(dnp no)
 		(fields_autoplaced yes)
-		(property "Reference" "#PWR027"
+		(property "Reference" "#PWR026"
 			(at 229.87 71.12 0)
 			(hide yes)
@@
 			(project "PS-HVCarrier"
 				(path "/2365a867-6254-4a7c-9718-f325e0bbac5c/c64f1e33-0c51-411c-bbbf-0af7b620c655"
-					(reference "#PWR027")
+					(reference "#PWR026")
 					(unit 1)
 				)
@@
 		(dnp no)
 		(fields_autoplaced yes)
-		(property "Reference" "#PWR026"
+		(property "Reference" "#PWR025"
 			(at 180.34 73.66 0)
 			(hide yes)
@@
 			(project "PS-HVCarrier"
 				(path "/2365a867-6254-4a7c-9718-f325e0bbac5c/c64f1e33-0c51-411c-bbbf-0af7b620c655"
-					(reference "#PWR026")
+					(reference "#PWR025")
 					(unit 1)
 				)
@@
 		(dnp no)
 		(fields_autoplaced yes)
-		(property "Reference" "#PWR024"
+		(property "Reference" "#PWR023"
 			(at 86.36 50.8 0)
 			(hide yes)
@@
 			(project "PS-HVCarrier"
 				(path "/2365a867-6254-4a7c-9718-f325e0bbac5c/c64f1e33-0c51-411c-bbbf-0af7b620c655"
-					(reference "#PWR024")
+					(reference "#PWR023")
 					(unit 1)
 				)
@@
 		(in_pos_files yes)
 		(dnp no)
-		(property "Reference" "TP15"
+		(property "Reference" "TP16"
 			(at 80.01 28.4479 0)
 			(hide yes)
@@
 			(project "PS-HVCarrier"
 				(path "/2365a867-6254-4a7c-9718-f325e0bbac5c/c64f1e33-0c51-411c-bbbf-0af7b620c655"
-					(reference "TP15")
+					(reference "TP16")
 					(unit 1)
 				)
@@
 		(in_pos_files yes)
 		(dnp no)
-		(property "Reference" "TP18"
+		(property "Reference" "TP19"
 			(at 179.07 29.7179 0)
 			(hide yes)
@@
 			(project "PS-HVCarrier"
 				(path "/2365a867-6254-4a7c-9718-f325e0bbac5c/c64f1e33-0c51-411c-bbbf-0af7b620c655"
-					(reference "TP18")
+					(reference "TP19")
 					(unit 1)
 				)
@@
 		(dnp no)
 		(fields_autoplaced yes)
-		(property "Reference" "#PWR028"
+		(property "Reference" "#PWR027"
 			(at 246.38 96.52 0)
 			(hide yes)
@@
 			(project "PS-HVCarrier"
 				(path "/2365a867-6254-4a7c-9718-f325e0bbac5c/c64f1e33-0c51-411c-bbbf-0af7b620c655"
-					(reference "#PWR028")
+					(reference "#PWR027")
 					(unit 1)
 				)
@@
 		(in_pos_files yes)
 		(dnp no)
-		(property "Reference" "TP19"
+		(property "Reference" "TP20"
 			(at 179.07 50.0379 0)
 			(hide yes)
@@
 			(project "PS-HVCarrier"
 				(path "/2365a867-6254-4a7c-9718-f325e0bbac5c/c64f1e33-0c51-411c-bbbf-0af7b620c655"
-					(reference "TP19")
+					(reference "TP20")
 					(unit 1)
 				)
@@
 		(in_pos_files yes)
 		(dnp no)
-		(property "Reference" "R32"
+		(property "Reference" "R34"
 			(at 62.23 78.74 90)
 			(show_name no)
@@
 			(project "PS-HVCarrier"
 				(path "/2365a867-6254-4a7c-9718-f325e0bbac5c/c64f1e33-0c51-411c-bbbf-0af7b620c655"
-					(reference "R32")
+					(reference "R34")
 					(unit 1)
 				)
@@
 		(in_pos_files yes)
 		(dnp no)
-		(property "Reference" "TP20"
+		(property "Reference" "TP21"
 			(at 247.65 48.7679 0)
 			(hide yes)
@@
 			(project "PS-HVCarrier"
 				(path "/2365a867-6254-4a7c-9718-f325e0bbac5c/c64f1e33-0c51-411c-bbbf-0af7b620c655"
-					(reference "TP20")
+					(reference "TP21")
 					(unit 1)
 				)
@@
 		(dnp no)
 		(fields_autoplaced yes)
-		(property "Reference" "R33"
+		(property "Reference" "R32"
 			(at 62.23 26.67 90)
 			(show_name no)
@@
 			(project "PS-HVCarrier"
 				(path "/2365a867-6254-4a7c-9718-f325e0bbac5c/c64f1e33-0c51-411c-bbbf-0af7b620c655"
-					(reference "R33")
+					(reference "R32")
 					(unit 1)
 				)
