File: hardware/Current_Sense.kicad_sch (KiCad schematic)
At the start: 37 parts, among them J10 SSA-2-100A, J11 SSA-2-100A, J9 LZSR 80-P, U8 TLV9002QDRQ1

Commit message: saving
Parts:
- added F?: Fuse_3557_2, LHRS_Power:Fuse-3557-2, symbol lhrs_power:Fuse_3557_2
Connections:
- net +5V: now also F?.1; no longer J9.1 (+UC)
- new net: F?.2, J9.1 (+UC)
Other:
- moved on the sheet: C47, C48
Changed lines of the file:
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@@
 	)
 	(junction
-		(at 93.98 30.48)
+		(at 91.44 30.48)
 		(diameter 0)
 		(color 0 0 0 0)
@@
 	)
 	(junction
-		(at 93.98 40.64)
+		(at 91.44 40.64)
 		(diameter 0)
 		(color 0 0 0 0)
@@
 	)
 	(junction
-		(at 86.36 40.64)
+		(at 83.82 40.64)
 		(diameter 0)
 		(color 0 0 0 0)
@@
 	(wire
 		(pts
-			(xy 86.36 40.64) (xy 86.36 44.45)
+			(xy 83.82 40.64) (xy 83.82 44.45)
 		)
 		(stroke
@@
 	(wire
 		(pts
-			(xy 86.36 30.48) (xy 86.36 40.64)
+			(xy 83.82 30.48) (xy 83.82 40.64)
 		)
 		(stroke
@@
 	(wire
 		(pts
-			(xy 101.6 40.64) (xy 93.98 40.64)
+			(xy 93.98 40.64) (xy 91.44 40.64)
 		)
 		(stroke
@@
 	(wire
 		(pts
-			(xy 93.98 30.48) (xy 93.98 27.94)
+			(xy 91.44 30.48) (xy 91.44 27.94)
 		)
 		(stroke
@@
 	(wire
 		(pts
-			(xy 93.98 30.48) (xy 93.98 40.64)
+			(xy 91.44 30.48) (xy 91.44 40.64)
 		)
 		(stroke
@@
 	(wire
 		(pts
-			(xy 86.36 44.45) (xy 101.6 44.45)
+			(xy 83.82 44.45) (xy 101.6 44.45)
 		)
 		(stroke
@@
 	(hierarchical_label "+5V"
 		(shape input)
-		(at 93.98 27.94 90)
+		(at 91.44 27.94 90)
 		(effects
 			(font
@@
 	(hierarchical_label "GND"
 		(shape input)
-		(at 86.36 44.45 270)
+		(at 83.82 44.45 270)
 		(effects
 			(font
@@
 	)
 	(hierarchical_label "SHUNT ADC UREF"
-		(shape input)
+		(shape output)
 		(at 182.88 58.42 0)
 		(effects
@@
 	(symbol
 		(lib_id "Device:C")
-		(at 90.17 40.64 270)
+		(at 87.63 40.64 270)
 		(unit 1)
 		(body_style 1)
@@
 		(dnp no)
 		(property "Reference" "C48"
-			(at 88.392 35.052 90)
+			(at 85.852 35.052 90)
 			(show_name no)
 			(do_not_autoplace no)
@@
 		)
 		(property "Value" "1u"
-			(at 89.154 37.338 90)
+			(at 86.614 37.338 90)
 			(show_name no)
 			(do_not_autoplace no)
@@
 		)
 		(property "Footprint" "Capacitor_SMD:C_0603_1608Metric_Pad1.08x0.95mm_HandSolder"
-			(at 86.36 41.6052 0)
+			(at 83.82 41.6052 0)
 			(hide yes)
 			(show_name no)
@@
 		)
 		(property "Datasheet" ""
-			(at 90.17 40.64 0)
+			(at 87.63 40.64 0)
 			(hide yes)
 			(show_name no)
@@
 		)
 		(property "Description" "Unpolarized capacitor"
-			(at 90.17 40.64 0)
+			(at 87.63 40.64 0)
 			(hide yes)
 			(show_name no)
@@
 		)
 		(property "LCSC" ""
-			(at 90.17 40.64 90)
+			(at 87.63 40.64 90)
 			(hide yes)
 			(show_name no)
@@
 	(symbol
 		(lib_id "Device:C")
-		(at 90.17 30.48 270)
+		(at 87.63 30.48 270)
 		(unit 1)
 		(body_style 1)
@@
 		(dnp no)
 		(property "Reference" "C47"
-			(at 87.884 24.384 90)
+			(at 85.344 24.384 90)
 			(show_name no)
 			(do_not_autoplace no)
@@
 		)
 		(property "Value" "100n"
-			(at 87.884 26.924 90)
+			(at 85.344 26.924 90)
 			(show_name no)
 			(do_not_autoplace no)
@@
 		)
 		(property "Footprint" "Capacitor_SMD:C_0603_1608Metric_Pad1.08x0.95mm_HandSolder"
-			(at 86.36 31.4452 0)
+			(at 83.82 31.4452 0)
 			(hide yes)
 			(show_name no)
@@
 		)
 		(property "Datasheet" ""
-			(at 90.17 30.48 0)
+			(at 87.63 30.48 0)
 			(hide yes)
 			(show_name no)
@@
 		)
 		(property "Description" "Unpolarized capacitor"
-			(at 90.17 30.48 0)
+			(at 87.63 30.48 0)
 			(hide yes)
 			(show_name no)
@@
 		)
 		(property "LCSC" ""
-			(at 90.17 30.48 90)
+			(at 87.63 30.48 90)
 			(hide yes)
 			(show_name no)
@@
 					(unit 1)
 				)
+			)
+		)
+	)
+	(symbol
+		(lib_id "lhrs_power:Fuse_3557_2")
+		(at 97.79 40.64 90)
+		(unit 1)
+		(body_style 1)
+		(exclude_from_sim no)
+		(in_bom yes)
+		(on_board yes)
+		(in_pos_files yes)
+		(dnp no)
+		(fields_autoplaced yes)
+		(property "Reference" "F?"
+			(at 97.79 34.29 90)
+			(show_name no)
+			(do_not_autoplace no)
+			(effects
+				(font
+					(size 1.27 1.27)
+				)
+			)
+		)
+		(property "Value" "Fuse_3557_2"
+			(at 97.79 36.83 90)
+			(show_name no)
+			(do_not_autoplace no)
+			(effects
+				(font
+					(size 1.27 1.27)
+				)
+			)
+		)
+		(property "Footprint" "LHRS_Power:Fuse-3557-2"
+			(at 97.79 42.418 90)
+			(hide yes)
+			(show_name no)
+			(do_not_autoplace no)
+			(effects
+				(font
+					(size 1.27 1.27)
+				)
+			)
+		)
+		(property "Datasheet" "kicad-embed://3557-2-datasheet.pdf"
+			(at 97.79 40.64 0)
+			(hide yes)
+			(show_name no)
+			(do_not_autoplace no)
+			(effects
+				(font
+					(size 1.27 1.27)
+				)
+			)
+		)
+		(property "Description" "Fuse, low-profile"
+			(at 97.79 40.64 0)
+			(hide yes)
+			(show_name no)
+			(do_not_autoplace no)
+			(effects
+				(font
+					(size 1.27 1.27)
+				)
+			)
+		)
+		(property "P/N" "3557-2"
+			(at 97.79 40.64 0)
+			(hide yes)
+			(show_name no)
+			(do_not_autoplace no)
+			(effects
+				(font
+					(size 1.27 1.27)
+				)
+			)
+		)
+		(property "Mouser P/N" "534-3557-2"
+			(at 97.79 40.64 0)
+			(hide yes)
+			(show_name no)
+			(do_not_autoplace no)
+			(effects
+				(font
+					(size 1.27 1.27)
+				)
+			)
+		)
+		(property "Digikey P/N" "36-3557-2-ND"
+			(at 97.79 40.64 0)
+			(hide yes)
+			(show_name no)
+			(do_not_autoplace no)
+			(effects
+				(font
+					(size 1.27 1.27)
+				)
+			)
+		)
+		(property "LCSC P/N" "C3205238"
+			(at 97.79 40.64 0)
+			(hide yes)
+			(show_name no)
+			(do_not_autoplace no)
+			(effects
+				(font
+					(size 1.27 1.27)
+				)
+			)
+		)
+		(pin "2"
+		)
+		(pin "1"
+		)
+		(instances
+			(project "PS-HVCarrier"
+				(path "/2365a867-6254-4a7c-9718-f325e0bbac5c/c64f1e33-0c51-411c-bbbf-0af7b620c655"
+					(reference "F?")
+					(unit 1)
+				)

Commit message: added outside test points, removed unncessary symbol fields
Parts:
- D17, D18: Mouser Part Number 576-SMF3.3 -> (none)
- F?: Digikey P/N 36-3557-2-ND -> (none); Mouser P/N 534-3557-2 -> (none)
- U8: Digikey P/N 296-TLV9002QDRQ1CT-ND -> (none); JLC P/N C2860922 -> (none); Mouser P/N 595-TLV9002QDRQ1 -> (none)

Commit message: updated kicad sharepoint, added pn
Parts:
- C41: renamed from C45; P/N (none) -> EMK107SD103KA-T
- C42: renamed from C46; P/N (none) -> EMK107SD103KA-T
- C43: renamed from C47; P/N (none) -> MAJCH168BB7104KTEA01
- C44: renamed from C48; P/N (none) -> MLASU168SB5105KTNA01
- C45: renamed from C49; P/N (none) -> MAJCH168BB7104KTEA01
- C46: renamed from C50; P/N (none) -> MAJCH168BB7104KTEA01
- C47: renamed from C51; P/N (none) -> UMK107B7102MAHT
- C48: renamed from C52; P/N (none) -> MLASH168SB7104KTNA01
- R37: renamed from R39; P/N (none) -> CRCW060310K0FKEI
- R38: renamed from R40; P/N (none) -> CRCW060310K0FKEI
- R39: renamed from R41; P/N (none) -> CRCW060310K0FKEI
- R42: renamed from R44; P/N (none) -> CRCW060310K0FKEI
- R43: renamed from R45; P/N (none) -> CRCW060310K0FKEI
- R46: renamed from R48; P/N (none) -> CRCW060310K0FKEI
- gave numbers to parts that had none: 1
- renumbered R36 to R34, R37 to R35, R38 to R36, R42 to R40, R43 to R41, R46 to R44, R47 to R45, TP20 to TP13, TP21 to TP14, TP22 to TP15, TP23 to TP16, TP24 to TP17, TP25 to TP18, U8 to U7
