File: hardware/5VBuck.kicad_sch (KiCad schematic)
At the start: 12 parts, among them U1 LMR51635XDDCR

Commit message: labeled + stm32 cube layout
Parts:
- removed C1: 2.2u, Capacitor_SMD:C_0805_2012Metric_Pad1.18x1.45mm_HandSolder, symbol Device:C_Small
- removed C2: 100n, Capacitor_SMD:C_0603_1608Metric, symbol Device:C_Small
- removed C3, C4: 47u, Capacitor_SMD:C_1210_3225Metric_Pad1.33x2.70mm_HandSolder, symbol Device:C_Small
- removed L1: 10u, LHRS_Passives:SRN8040-101M, symbol Device:L_Small
- removed R1: 53.6k, Resistor_SMD:R_0603_1608Metric, symbol Device:R_Small
- removed R2: 10.2k, Resistor_SMD:R_0603_1608Metric, symbol Device:R_Small
- removed TP?: FB, TestPoint:TestPoint_THTPad_D3.0mm_Drill1.5mm, symbol Connector:TestPoint
- removed TP?: V_in_24V, TestPoint:TestPoint_THTPad_D3.0mm_Drill1.5mm, symbol Connector:TestPoint
- removed TP?: SW, TestPoint:TestPoint_THTPad_D3.0mm_Drill1.5mm, symbol Connector:TestPoint
- removed TP?: CB, TestPoint:TestPoint_THTPad_D3.0mm_Drill1.5mm, symbol Connector:TestPoint
- removed U1: LMR51635XDDCR, LHRS_ICs:DDC0006A-MFG, symbol 2026-04-25_18-34-12:LMR51635XDDCR
- added C13: 2.2u, Capacitor_SMD:C_0805_2012Metric_Pad1.18x1.45mm_HandSolder, symbol Device:C_Small
- added C14: 100n, Capacitor_SMD:C_0603_1608Metric, symbol Device:C_Small
- added C15, C16: 47u, Capacitor_SMD:C_1210_3225Metric_Pad1.33x2.70mm_HandSolder, symbol Device:C_Small
- added L2: 10u, LHRS_Passives:SRN8040-101M, symbol Device:L_Small
- added R8: 53.6k, Resistor_SMD:R_0603_1608Metric, symbol Device:R_Small
- added R9: 10.2k, Resistor_SMD:R_0603_1608Metric, symbol Device:R_Small
- added TP15: V_in_24V, TestPoint:TestPoint_THTPad_D3.0mm_Drill1.5mm, symbol Connector:TestPoint
- added TP16: CB, TestPoint:TestPoint_THTPad_D3.0mm_Drill1.5mm, symbol Connector:TestPoint
- added TP17: FB, TestPoint:TestPoint_THTPad_D3.0mm_Drill1.5mm, symbol Connector:TestPoint
- added TP18: SW, TestPoint:TestPoint_THTPad_D3.0mm_Drill1.5mm, symbol Connector:TestPoint
- added U2: LMR51635XDDCR, LHRS_ICs:DDC0006A-MFG, symbol 2026-04-25_18-34-12:LMR51635XDDCR
Connections:
- net CB: now also C14.1, TP16.1, U2.6 (CB)
- net FB: now also R8.2, R9.1, TP17.1, U2.1 (FB)
- net GND: now also C13.2, C15.2, C16.2, R9.2, U2.4 (GND)
- net SW: now also C14.2, L2.1, TP18.1, U2.5 (SW)
- net V_in_24V: now also C13.1, TP15.1, U2.2 (EN), U2.3 (VIN)
- net V_out_5V: now also C15.1, C16.1, L2.2, R8.1

Commit message: added debug led
Parts:
- renumbered R8 to R15, R9 to R16
Changed lines of the file:
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@@
 		(dnp no)
 		(fields_autoplaced yes)
-		(property "Reference" "R8"
+		(property "Reference" "R15"
 			(at 170.18 41.9099 0)
 			(effects
@@
 			(project "5VBuck"
 				(path "/2365a867-6254-4a7c-9718-f325e0bbac5c/904fa10a-747c-46cf-90d1-33d76069dc5d/cdc38143-6c01-474d-8a8e-ff8bf18b44d0"
-					(reference "R8")
+					(reference "R15")
 					(unit 1)
 				)
@@
 		(dnp no)
 		(fields_autoplaced yes)
-		(property "Reference" "R9"
+		(property "Reference" "R16"
 			(at 170.18 49.5299 0)
 			(effects
@@
 			(project "5VBuck"
 				(path "/2365a867-6254-4a7c-9718-f325e0bbac5c/904fa10a-747c-46cf-90d1-33d76069dc5d/cdc38143-6c01-474d-8a8e-ff8bf18b44d0"
-					(reference "R9")
-					(unit 1)
-				)
+					(reference "R16")
+					(unit 1)
+				)

Commit message: added calcs, cleaned up, addressed comments
Parts:
- renumbered C13 to C30, C14 to C31, C15 to C32, C16 to C33, L2 to L1, R15 to R25, R16 to R26, TP18 to TP10, TP15 to TP7, TP16 to TP8, TP17 to TP9, U2 to U3
Changed lines of the file:
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@@
 		(dnp no)
 		(fields_autoplaced yes)
-		(property "Reference" "C16"
+		(property "Reference" "C33"
 			(at 129.54 49.5362 0)
 			(show_name no)
@@
 			(project "PS-HVCarrier"
 				(path "/2365a867-6254-4a7c-9718-f325e0bbac5c/904fa10a-747c-46cf-90d1-33d76069dc5d/cdc38143-6c01-474d-8a8e-ff8bf18b44d0"
-					(reference "C16")
+					(reference "C33")
 					(unit 1)
 				)
@@
 		(in_pos_files yes)
 		(dnp no)
-		(property "Reference" "TP15"
+		(property "Reference" "TP7"
 			(at 171.45 80.5179 0)
 			(hide yes)
@@
 			(project "PS-HVCarrier"
 				(path "/2365a867-6254-4a7c-9718-f325e0bbac5c/904fa10a-747c-46cf-90d1-33d76069dc5d/cdc38143-6c01-474d-8a8e-ff8bf18b44d0"
-					(reference "TP15")
+					(reference "TP7")
 					(unit 1)
 				)
@@
 		(dnp no)
 		(fields_autoplaced yes)
-		(property "Reference" "C13"
+		(property "Reference" "C30"
 			(at 40.64 45.7262 0)
 			(show_name no)
@@
 			(project "PS-HVCarrier"
 				(path "/2365a867-6254-4a7c-9718-f325e0bbac5c/904fa10a-747c-46cf-90d1-33d76069dc5d/cdc38143-6c01-474d-8a8e-ff8bf18b44d0"
-					(reference "C13")
+					(reference "C30")
 					(unit 1)
 				)
@@
 		(in_pos_files yes)
 		(dnp no)
-		(property "Reference" "L2"
+		(property "Reference" "L1"
 			(at 106.68 48.514 90)
 			(show_name no)
@@
 			(project "PS-HVCarrier"
 				(path "/2365a867-6254-4a7c-9718-f325e0bbac5c/904fa10a-747c-46cf-90d1-33d76069dc5d/cdc38143-6c01-474d-8a8e-ff8bf18b44d0"
-					(reference "L2")
+					(reference "L1")
 					(unit 1)
 				)
@@
 		(dnp no)
 		(fields_autoplaced yes)
-		(property "Reference" "R15"
+		(property "Reference" "R25"
 			(at 170.18 41.9099 0)
 			(show_name no)
@@
 			(project "PS-HVCarrier"
 				(path "/2365a867-6254-4a7c-9718-f325e0bbac5c/904fa10a-747c-46cf-90d1-33d76069dc5d/cdc38143-6c01-474d-8a8e-ff8bf18b44d0"
-					(reference "R15")
+					(reference "R25")
 					(unit 1)
 				)
@@
 		(in_pos_files yes)
 		(dnp no)
-		(property "Reference" "TP18"
+		(property "Reference" "TP10"
 			(at 184.15 93.2179 0)
 			(hide yes)
@@
 			(project "PS-HVCarrier"
 				(path "/2365a867-6254-4a7c-9718-f325e0bbac5c/904fa10a-747c-46cf-90d1-33d76069dc5d/cdc38143-6c01-474d-8a8e-ff8bf18b44d0"
-					(reference "TP18")
+					(reference "TP10")
 					(unit 1)
 				)
@@
 		(in_pos_files yes)
 		(dnp no)
-		(property "Reference" "TP16"
+		(property "Reference" "TP8"
 			(at 171.45 93.2179 0)
 			(hide yes)
@@
 			(project "PS-HVCarrier"
 				(path "/2365a867-6254-4a7c-9718-f325e0bbac5c/904fa10a-747c-46cf-90d1-33d76069dc5d/cdc38143-6c01-474d-8a8e-ff8bf18b44d0"
-					(reference "TP16")
+					(reference "TP8")
 					(unit 1)
 				)
@@
 		(dnp no)
 		(fields_autoplaced yes)
-		(property "Reference" "R16"
+		(property "Reference" "R26"
 			(at 170.18 49.5299 0)
 			(show_name no)
@@
 			(project "PS-HVCarrier"
 				(path "/2365a867-6254-4a7c-9718-f325e0bbac5c/904fa10a-747c-46cf-90d1-33d76069dc5d/cdc38143-6c01-474d-8a8e-ff8bf18b44d0"
-					(reference "R16")
+					(reference "R26")
 					(unit 1)
 				)
@@
 		(dnp no)
 		(fields_autoplaced yes)
-		(property "Reference" "U2"
+		(property "Reference" "U3"
 			(at 73.66 31.75 0)
 			(show_name no)
@@
 			(project "PS-HVCarrier"
 				(path "/2365a867-6254-4a7c-9718-f325e0bbac5c/904fa10a-747c-46cf-90d1-33d76069dc5d/cdc38143-6c01-474d-8a8e-ff8bf18b44d0"
-					(reference "U2")
+					(reference "U3")
 					(unit 1)
 				)
@@
 		(in_pos_files yes)
 		(dnp no)
-		(property "Reference" "#FLG06"
+		(property "Reference" "#FLG02"
 			(at 93.98 45.085 0)
 			(hide yes)
@@
 			(project "PS-HVCarrier"
 				(path "/2365a867-6254-4a7c-9718-f325e0bbac5c/904fa10a-747c-46cf-90d1-33d76069dc5d/cdc38143-6c01-474d-8a8e-ff8bf18b44d0"
-					(reference "#FLG06")
+					(reference "#FLG02")
 					(unit 1)
 				)
@@
 		(dnp no)
 		(fields_autoplaced yes)
-		(property "Reference" "#FLG05"
+		(property "Reference" "#FLG01"
 			(at 93.98 40.005 0)
 			(hide yes)
@@
 			(project "PS-HVCarrier"
 				(path "/2365a867-6254-4a7c-9718-f325e0bbac5c/904fa10a-747c-46cf-90d1-33d76069dc5d/cdc38143-6c01-474d-8a8e-ff8bf18b44d0"
-					(reference "#FLG05")
+					(reference "#FLG01")
 					(unit 1)
 				)
@@
 		(in_pos_files yes)
 		(dnp no)
-		(property "Reference" "C14"
+		(property "Reference" "C31"
 			(at 100.838 40.64 0)
 			(show_name no)
@@
 			(project "PS-HVCarrier"
 				(path "/2365a867-6254-4a7c-9718-f325e0bbac5c/904fa10a-747c-46cf-90d1-33d76069dc5d/cdc38143-6c01-474d-8a8e-ff8bf18b44d0"
-					(reference "C14")
+					(reference "C31")
 					(unit 1)
 				)
@@
 		(dnp no)
 		(fields_autoplaced yes)
-		(property "Reference" "C15"
+		(property "Reference" "C32"
 			(at 118.11 49.5362 0)
 			(show_name no)
@@
 			(project "PS-HVCarrier"
 				(path "/2365a867-6254-4a7c-9718-f325e0bbac5c/904fa10a-747c-46cf-90d1-33d76069dc5d/cdc38143-6c01-474d-8a8e-ff8bf18b44d0"
-					(reference "C15")
+					(reference "C32")
 					(unit 1)
 				)
@@
 		(in_pos_files yes)
 		(dnp no)
-		(property "Reference" "TP17"
+		(property "Reference" "TP9"
 			(at 184.15 80.5179 0)
 			(hide yes)
@@
 			(project "PS-HVCarrier"
 				(path "/2365a867-6254-4a7c-9718-f325e0bbac5c/904fa10a-747c-46cf-90d1-33d76069dc5d/cdc38143-6c01-474d-8a8e-ff8bf18b44d0"
-					(reference "TP17")
-					(unit 1)
-				)
+					(reference "TP9")
+					(unit 1)
+				)

Commit message: fixed ERC warnings
Parts:
- renumbered TP9 to TP10, TP10 to TP11, TP7 to TP8, TP8 to TP9
Changed lines of the file:
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@@
 		(in_pos_files yes)
 		(dnp no)
-		(property "Reference" "TP7"
+		(property "Reference" "TP8"
 			(at 171.45 80.5179 0)
 			(hide yes)
@@
 			(project "PS-HVCarrier"
 				(path "/2365a867-6254-4a7c-9718-f325e0bbac5c/904fa10a-747c-46cf-90d1-33d76069dc5d/cdc38143-6c01-474d-8a8e-ff8bf18b44d0"
-					(reference "TP7")
+					(reference "TP8")
 					(unit 1)
 				)
@@
 		(in_pos_files yes)
 		(dnp no)
-		(property "Reference" "TP10"
+		(property "Reference" "TP11"
 			(at 184.15 93.2179 0)
 			(hide yes)
@@
 			(project "PS-HVCarrier"
 				(path "/2365a867-6254-4a7c-9718-f325e0bbac5c/904fa10a-747c-46cf-90d1-33d76069dc5d/cdc38143-6c01-474d-8a8e-ff8bf18b44d0"
-					(reference "TP10")
+					(reference "TP11")
 					(unit 1)
 				)
@@
 		(in_pos_files yes)
 		(dnp no)
-		(property "Reference" "TP8"
+		(property "Reference" "TP9"
 			(at 171.45 93.2179 0)
 			(hide yes)
@@
 			(project "PS-HVCarrier"
 				(path "/2365a867-6254-4a7c-9718-f325e0bbac5c/904fa10a-747c-46cf-90d1-33d76069dc5d/cdc38143-6c01-474d-8a8e-ff8bf18b44d0"
-					(reference "TP8")
+					(reference "TP9")
 					(unit 1)
 				)
@@
 		(in_pos_files yes)
 		(dnp no)
-		(property "Reference" "TP9"
+		(property "Reference" "TP10"
 			(at 184.15 80.5179 0)
 			(hide yes)
@@
 			(project "PS-HVCarrier"
 				(path "/2365a867-6254-4a7c-9718-f325e0bbac5c/904fa10a-747c-46cf-90d1-33d76069dc5d/cdc38143-6c01-474d-8a8e-ff8bf18b44d0"
-					(reference "TP9")
-					(unit 1)
-				)
+					(reference "TP10")
+					(unit 1)
+				)

Commit message: added HV taps + 48 pin MCU for design consideration
Parts:
- renumbered TP8 to TP14, TP9 to TP15, TP10 to TP16, TP11 to TP17
Changed lines of the file:
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@@
 		(in_pos_files yes)
 		(dnp no)
-		(property "Reference" "TP8"
+		(property "Reference" "TP14"
 			(at 171.45 80.5179 0)
 			(hide yes)
@@
 			(project "PS-HVCarrier"
 				(path "/2365a867-6254-4a7c-9718-f325e0bbac5c/904fa10a-747c-46cf-90d1-33d76069dc5d/cdc38143-6c01-474d-8a8e-ff8bf18b44d0"
-					(reference "TP8")
+					(reference "TP14")
 					(unit 1)
 				)
@@
 		(in_pos_files yes)
 		(dnp no)
-		(property "Reference" "TP11"
+		(property "Reference" "TP17"
 			(at 184.15 93.2179 0)
 			(hide yes)
@@
 			(project "PS-HVCarrier"
 				(path "/2365a867-6254-4a7c-9718-f325e0bbac5c/904fa10a-747c-46cf-90d1-33d76069dc5d/cdc38143-6c01-474d-8a8e-ff8bf18b44d0"
-					(reference "TP11")
+					(reference "TP17")
 					(unit 1)
 				)
@@
 		(in_pos_files yes)
 		(dnp no)
-		(property "Reference" "TP9"
+		(property "Reference" "TP15"
 			(at 171.45 93.2179 0)
 			(hide yes)
@@
 			(project "PS-HVCarrier"
 				(path "/2365a867-6254-4a7c-9718-f325e0bbac5c/904fa10a-747c-46cf-90d1-33d76069dc5d/cdc38143-6c01-474d-8a8e-ff8bf18b44d0"
-					(reference "TP9")
+					(reference "TP15")
 					(unit 1)
 				)
@@
 		(in_pos_files yes)
 		(dnp no)
-		(property "Reference" "TP10"
+		(property "Reference" "TP16"
 			(at 184.15 80.5179 0)
 			(hide yes)
@@
 			(project "PS-HVCarrier"
 				(path "/2365a867-6254-4a7c-9718-f325e0bbac5c/904fa10a-747c-46cf-90d1-33d76069dc5d/cdc38143-6c01-474d-8a8e-ff8bf18b44d0"
-					(reference "TP10")
-					(unit 1)
-				)
+					(reference "TP16")
+					(unit 1)
+				)
