File: hardware/Voltage_Sense.kicad_sch (KiCad schematic)
At the start: 56 parts, among them U5 TLV9002QDRQ1, U6 AMC3311QDWERQ1, U7 AMC3311QDWERQ1

Commit message: added HV taps + 48 pin MCU for design consideration
Parts:
- renumbered C43 to C58, C44 to C59, C45 to C60, C46 to C61, C47 to C62, C48 to C63, C49 to C64, C50 to C65, C51 to C66, C52 to C67, C53 to C68, C54 to C69, C55 to C70, C56 to C71, C57 to C72, C58 to C73, C59 to C74, C61 to C75, C60 to C76, C62 to C77, C63 to C78, D21 to D24, D22 to D25, D23 to D26, D24 to D27, R42 to R50, R43 to R51, R44 to R52, R45 to R53, R46 to R54, R47 to R55, R48 to R56, R49 to R57, R50 to R58, R51 to R59, R52 to R60, R53 to R61, R54 to R62, R55 to R63, R56 to R64, R57 to R65, R58 to R66, R59 to R67, R60 to R68, R61 to R69, TP22 to TP28, TP23 to TP29, TP24 to TP30, TP25 to TP31, TP26 to TP32, TP27 to TP33, TP28 to TP34, TP29 to TP35, U5 to U6, U6 to U7, U7 to U8
Connections:
- net HV GND: now reaches C59.2, C61.2, C62.1, C64.1, C67.1, R59.1, U7.2 (DCDC_HGND), U7.7 (HGND), U7.8 (HGND)
- net Motor GND: now reaches C60.2, C63.1, C65.1, C66.1, C68.1, R60.1, U8.2 (DCDC_HGND), U8.7 (HGND), U8.8 (HGND)
