File: hardware/100PinMCU.kicad_sch (KiCad schematic)
At the start: 33 parts, among them J5 SWD_Header, J6 SWD, SW1 SW_SPDT, U2 STM32G473VETx, Y1 Crystal

Commit message: added HV taps + 48 pin MCU for design consideration
Parts:
- renumbered J5 to J7, J6 to J8

Commit message: added design blocks
Parts:
- renumbered J7 to J6, J8 to J7
Changed lines of the file:
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@@
 		(in_pos_files yes)
 		(dnp no)
-		(property "Reference" "J7"
+		(property "Reference" "J6"
 			(at 225.552 128.524 0)
 			(show_name no)
@@
 			(project "PS-HVCarrier"
 				(path "/2365a867-6254-4a7c-9718-f325e0bbac5c/c5db4e3e-bfb8-40cd-87d6-5e9e9bc2d94c"
-					(reference "J7")
+					(reference "J6")
 					(unit 1)
 				)
@@
 		(in_pos_files yes)
 		(dnp no)
-		(property "Reference" "J8"
+		(property "Reference" "J7"
 			(at 224.536 146.304 0)
 			(show_name no)
@@
 			(project "PS-HVCarrier"
 				(path "/2365a867-6254-4a7c-9718-f325e0bbac5c/c5db4e3e-bfb8-40cd-87d6-5e9e9bc2d94c"
-					(reference "J8")
-					(unit 1)
-				)
+					(reference "J7")
+					(unit 1)
+				)
