File: hardware/48PinMCU.kicad_sch (KiCad schematic)
At the start: 34 parts, among them J10 SWD, J9 SWD_Header, SW2 Reset, SW3 SW_SPDT, U4 STM32G473CETx, Y2 Crystal

Commit message: added design blocks
Parts:
- renumbered J9 to J8, J10 to J9
Changed lines of the file:
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@@
 		(in_pos_files yes)
 		(dnp no)
-		(property "Reference" "J9"
+		(property "Reference" "J8"
 			(at 259.334 135.89 0)
 			(show_name no)
@@
 			(project "PS-HVCarrier"
 				(path "/2365a867-6254-4a7c-9718-f325e0bbac5c/525eebd7-cd9b-471b-950d-358e3ce0c5f6"
-					(reference "J9")
+					(reference "J8")
 					(unit 1)
 				)
@@
 		(in_pos_files yes)
 		(dnp no)
-		(property "Reference" "J10"
+		(property "Reference" "J9"
 			(at 254 151.384 0)
 			(show_name no)
@@
 			(project "PS-HVCarrier"
 				(path "/2365a867-6254-4a7c-9718-f325e0bbac5c/525eebd7-cd9b-471b-950d-358e3ce0c5f6"
-					(reference "J10")
+					(reference "J9")
 					(unit 1)
 				)

Commit message: changed fully to 48 pin MCU
Parts:
- renumbered C34 to C20, C35 to C21, C36 to C22, C37 to C23, C38 to C24, C39 to C25, C40 to C26, C41 to C27, C42 to C28, C43 to C29, C44 to C30, C45 to C31, C46 to C32, C47 to C33, C48 to C34, D13 to D10, D14 to D11, D15 to D12, FB3 to FB1, FB4 to FB2, J8 to J6, J9 to J7, R27 to R19, R28 to R20, R29 to R21, R30 to R22, R31 to R23, R32 to R24, R33 to R25, R34 to R26, SW2 to SW1, SW3 to SW2, U4 to U3, Y2 to Y1
