File: hardware/48PinMCU.kicad_sch (KiCad schematic)
At the start: 34 parts, among them J6 SWD_Header, J7 SWD, SW1 Reset, SW2 SW_SPDT, U7 STM32G473CETx, Y1 Crystal

Commit message: added outside test points, removed unncessary symbol fields
Parts:
- C31: Mouser Part Number 08055D475KAT4A -> (none)
- C32, C33, C34, C35, C36, C37, C38, C39, C40, C41, C42: Mouser Part Number MLASH168SB7104KTNA01 -> (none)
- D8: MANUFACTURER Everlight -> (none)
- D9: Color Blue -> (none); Mouser P/N 771-PESD15VL1BA-T/R -> (none)
- J6: LSCS P/N C17492485 -> (none)
- R27, R32: Mouser Part Number CRCW060310K0FKEI -> (none)
- SW1: Mouser Part Number 612-TL3365AF180QG -> (none)

Commit message: updated kicad sharepoint, added pn
Parts:
- C39: renamed from C43; value 100nF -> 100n; P/N MLASH168SB7104KTNA01 -> MAJCH168BB7104KTEA01
- R28: renamed from R30; P/N FRC0603F22R0TS -> RC0603FR-0722RL
- R29: renamed from R31; P/N FRC0603F22R0TS -> RC0603FR-0722RL
- renumbered C29 to C25, C30 to C26, C31 to C27, C32 to C28, C33 to C29, C34 to C30, C35 to C31, C36 to C32, C37 to C33, C38 to C34, C39 to C35, C40 to C36, C41 to C37, C42 to C38, R26 to R24, R27 to R25, R28 to R26, R29 to R27, R32 to R30, R33 to R31, U7 to U6
Changed lines of the file:
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@@
 		(dnp no)
 		(fields_autoplaced yes)
-		(property "Reference" "C35"
+		(property "Reference" "C31"
 			(at 190.5 57.1499 0)
 			(show_name no)
@@
 			(project "PS-HVCarrier"
 				(path "/2365a867-6254-4a7c-9718-f325e0bbac5c/525eebd7-cd9b-471b-950d-358e3ce0c5f6"
-					(reference "C35")
+					(reference "C31")
 					(unit 1)
 				)
@@
 		(in_pos_files yes)
 		(dnp no)
-		(property "Reference" "R28"
+		(property "Reference" "R26"
 			(at 183.388 154.686 0)
 			(show_name no)
@@
 			(project "PS-HVCarrier"
 				(path "/2365a867-6254-4a7c-9718-f325e0bbac5c/525eebd7-cd9b-471b-950d-358e3ce0c5f6"
-					(reference "R28")
+					(reference "R26")
 					(unit 1)
 				)
@@
 		(in_pos_files yes)
 		(dnp no)
-		(property "Reference" "U7"
+		(property "Reference" "U6"
 			(at 88.392 73.66 0)
 			(hide yes)
@@
 			(project "PS-HVCarrier"
 				(path "/2365a867-6254-4a7c-9718-f325e0bbac5c/525eebd7-cd9b-471b-950d-358e3ce0c5f6"
-					(reference "U7")
+					(reference "U6")
 					(unit 1)
 				)
@@
 		(in_pos_files yes)
 		(dnp no)
-		(property "Reference" "C42"
+		(property "Reference" "C38"
 			(at 246.634 31.75 0)
 			(show_name no)
@@
 			(project "PS-HVCarrier"
 				(path "/2365a867-6254-4a7c-9718-f325e0bbac5c/525eebd7-cd9b-471b-950d-358e3ce0c5f6"
-					(reference "C42")
+					(reference "C38")
 					(unit 1)
 				)
@@
 		(dnp no)
 		(fields_autoplaced yes)
-		(property "Reference" "C37"
+		(property "Reference" "C33"
 			(at 205.105 57.1499 0)
 			(show_name no)
@@
 			(project "PS-HVCarrier"
 				(path "/2365a867-6254-4a7c-9718-f325e0bbac5c/525eebd7-cd9b-471b-950d-358e3ce0c5f6"
-					(reference "C37")
+					(reference "C33")
 					(unit 1)
 				)
@@
 		(dnp no)
 		(fields_autoplaced yes)
-		(property "Reference" "C40"
+		(property "Reference" "C36"
 			(at 223.52 33.0199 0)
 			(show_name no)
@@
 			(project "PS-HVCarrier"
 				(path "/2365a867-6254-4a7c-9718-f325e0bbac5c/525eebd7-cd9b-471b-950d-358e3ce0c5f6"
-					(reference "C40")
+					(reference "C36")
 					(unit 1)
 				)
@@
 		(in_pos_files yes)
 		(dnp no)
-		(property "Reference" "C38"
+		(property "Reference" "C34"
 			(at 210.566 32.766 0)
 			(show_name no)
@@
 			(project "PS-HVCarrier"
 				(path "/2365a867-6254-4a7c-9718-f325e0bbac5c/525eebd7-cd9b-471b-950d-358e3ce0c5f6"
-					(reference "C38")
+					(reference "C34")
 					(unit 1)
 				)
@@
 		(in_pos_files yes)
 		(dnp no)
-		(property "Reference" "C34"
+		(property "Reference" "C30"
 			(at 185.674 33.02 0)
 			(show_name no)
@@
 			(project "PS-HVCarrier"
 				(path "/2365a867-6254-4a7c-9718-f325e0bbac5c/525eebd7-cd9b-471b-950d-358e3ce0c5f6"
-					(reference "C34")
+					(reference "C30")
 					(unit 1)
 				)
@@
 		(dnp no)
 		(fields_autoplaced yes)
-		(property "Reference" "C43"
+		(property "Reference" "C39"
 			(at 258.445 57.785 0)
 			(show_name no)
@@
 			)
 		)
-		(property "Value" "100nF"
+		(property "Value" "100n"
 			(at 258.445 60.325 0)
 			(show_name no)
@@
 			)
 		)
-		(property "P/N" "MLASH168SB7104KTNA01"
+		(property "P/N" "MAJCH168BB7104KTEA01"
 			(at 255.27 58.42 0)
 			(hide yes)
@@
 			(project "PS-HVCarrier"
 				(path "/2365a867-6254-4a7c-9718-f325e0bbac5c/525eebd7-cd9b-471b-950d-358e3ce0c5f6"
-					(reference "C43")
+					(reference "C39")
 					(unit 1)
 				)
@@
 		(in_pos_files yes)
 		(dnp no)
-		(property "Reference" "C36"
+		(property "Reference" "C32"
 			(at 197.358 33.02 0)
 			(show_name no)
@@
 			(project "PS-HVCarrier"
 				(path "/2365a867-6254-4a7c-9718-f325e0bbac5c/525eebd7-cd9b-471b-950d-358e3ce0c5f6"
-					(reference "C36")
+					(reference "C32")
 					(unit 1)
 				)
@@
 		(in_pos_files yes)
 		(dnp no)
-		(property "Reference" "C39"
+		(property "Reference" "C35"
 			(at 217.678 56.388 0)
 			(show_name no)
@@
 			(project "PS-HVCarrier"
 				(path "/2365a867-6254-4a7c-9718-f325e0bbac5c/525eebd7-cd9b-471b-950d-358e3ce0c5f6"
-					(reference "C39")
+					(reference "C35")
 					(unit 1)
 				)
@@
 		(in_pos_files yes)
 		(dnp no)
-		(property "Reference" "R29"
+		(property "Reference" "R27"
 			(at 191.008 154.686 0)
 			(show_name no)
@@
 			(project "PS-HVCarrier"
 				(path "/2365a867-6254-4a7c-9718-f325e0bbac5c/525eebd7-cd9b-471b-950d-358e3ce0c5f6"
-					(reference "R29")
+					(reference "R27")
 					(unit 1)
 				)
@@
 		(in_pos_files yes)
 		(dnp no)
-		(property "Reference" "R33"
+		(property "Reference" "R31"
 			(at 259.588 110.236 0)
 			(show_name no)
@@
 			(project "PS-HVCarrier"
 				(path "/2365a867-6254-4a7c-9718-f325e0bbac5c/525eebd7-cd9b-471b-950d-358e3ce0c5f6"
-					(reference "R33")
+					(reference "R31")
 					(unit 1)
 				)
@@
 		(in_pos_files yes)
 		(dnp no)
-		(property "Reference" "C29"
+		(property "Reference" "C25"
 			(at 34.036 39.624 90)
 			(show_name no)
@@
 			(project "PS-HVCarrier"
 				(path "/2365a867-6254-4a7c-9718-f325e0bbac5c/525eebd7-cd9b-471b-950d-358e3ce0c5f6"
-					(reference "C29")
+					(reference "C25")
 					(unit 1)
 				)
@@
 		(dnp no)
 		(fields_autoplaced yes)
-		(property "Reference" "C32"
+		(property "Reference" "C28"
 			(at 175.26 57.1499 0)
 			(show_name no)
@@
 			(project "PS-HVCarrier"
 				(path "/2365a867-6254-4a7c-9718-f325e0bbac5c/525eebd7-cd9b-471b-950d-358e3ce0c5f6"
-					(reference "C32")
+					(reference "C28")
 					(unit 1)
 				)
@@
 		(dnp no)
 		(fields_autoplaced yes)
-		(property "Reference" "R27"
+		(property "Reference" "R25"
 			(at 180.34 96.5199 0)
 			(show_name no)
@@
 			(project "PS-HVCarrier"
 				(path "/2365a867-6254-4a7c-9718-f325e0bbac5c/525eebd7-cd9b-471b-950d-358e3ce0c5f6"
-					(reference "R27")
+					(reference "R25")
 					(unit 1)
 				)
@@
 		(in_pos_files yes)
 		(dnp no)
-		(property "Reference" "R26"
+		(property "Reference" "R24"
 			(at 175.768 154.686 0)
 			(show_name no)
@@
 			(project "PS-HVCarrier"
 				(path "/2365a867-6254-4a7c-9718-f325e0bbac5c/525eebd7-cd9b-471b-950d-358e3ce0c5f6"
-					(reference "R26")
+					(reference "R24")
 					(unit 1)
 				)
@@
 		(in_pos_files yes)
 		(dnp no)
-		(property "Reference" "R31"
+		(property "Reference" "R29"
 			(at 226.06 149.225 90)
 			(show_name no)
@@
 			)
 		)
-		(property "P/N" "FRC0603F22R0TS"
+		(property "P/N" "RC0603FR-0722RL"
 			(at 226.06 146.05 90)
 			(hide yes)
@@
 			(project "PS-HVCarrier"
 				(path "/2365a867-6254-4a7c-9718-f325e0bbac5c/525eebd7-cd9b-471b-950d-358e3ce0c5f6"
-					(reference "R31")
+					(reference "R29")
 					(unit 1)
 				)
@@
 		(in_pos_files yes)
 		(dnp no)
-		(property "Reference" "C31"
+		(property "Reference" "C27"
 			(at 174.244 33.02 0)
 			(show_name no)
@@
 			(project "PS-HVCarrier"
 				(path "/2365a867-6254-4a7c-9718-f325e0bbac5c/525eebd7-cd9b-471b-950d-358e3ce0c5f6"
-					(reference "C31")
+					(reference "C27")
 					(unit 1)
 				)
@@
 		(in_pos_files yes)
 		(dnp no)
-		(property "Reference" "R32"
+		(property "Reference" "R30"
 			(at 248.285 101.5999 0)
 			(show_name no)
@@
 			(project "PS-HVCarrier"
 				(path "/2365a867-6254-4a7c-9718-f325e0bbac5c/525eebd7-cd9b-471b-950d-358e3ce0c5f6"
-					(reference "R32")
+					(reference "R30")
 					(unit 1)
 				)
@@
 		(dnp no)
 		(fields_autoplaced yes)
-		(property "Reference" "C30"
+		(property "Reference" "C26"
 			(at 34.29 58.928 90)
 			(show_name no)
@@
 			(project "PS-HVCarrier"
 				(path "/2365a867-6254-4a7c-9718-f325e0bbac5c/525eebd7-cd9b-471b-950d-358e3ce0c5f6"
-					(reference "C30")
+					(reference "C26")
 					(unit 1)
 				)
@@
 		(in_pos_files yes)
 		(dnp no)
-		(property "Reference" "C33"
+		(property "Reference" "C29"
 			(at 169.164 106.426 0)
 			(show_name no)
@@
 			(project "PS-HVCarrier"
 				(path "/2365a867-6254-4a7c-9718-f325e0bbac5c/525eebd7-cd9b-471b-950d-358e3ce0c5f6"
-					(reference "C33")
+					(reference "C29")
 					(unit 1)
 				)
@@
 		(dnp no)
 		(fields_autoplaced yes)
-		(property "Reference" "R30"
+		(property "Reference" "R28"
 			(at 226.06 137.795 90)
 			(show_name no)
@@
 			)
 		)
-		(property "P/N" "FRC0603F22R0TS"
+		(property "P/N" "RC0603FR-0722RL"
 			(at 226.06 143.51 90)
 			(hide yes)
@@
 			(project "PS-HVCarrier"
 				(path "/2365a867-6254-4a7c-9718-f325e0bbac5c/525eebd7-cd9b-471b-950d-358e3ce0c5f6"
-					(reference "R30")
+					(reference "R28")
 					(unit 1)
 				)
@@
 		(in_pos_files yes)
 		(dnp no)
-		(property "Reference" "C41"
+		(property "Reference" "C37"
 			(at 233.426 32.004 0)
 			(show_name no)
@@
 			(project "PS-HVCarrier"
 				(path "/2365a867-6254-4a7c-9718-f325e0bbac5c/525eebd7-cd9b-471b-950d-358e3ce0c5f6"
-					(reference "C41")
+					(reference "C37")
 					(unit 1)
 				)
