File: hardware/CAN_Transceiver2.0.kicad_sch (KiCad schematic)
At the start: 9 parts, among them IC1 TCAN3413DR

Commit message: labeled + stm32 cube layout
Parts:
- removed D8: CDSOT23-T24CAN, LHRS_Passives:CDSOT23-T24CAN, symbol CDSOT23-T24CAN:CDSOT23-T24CAN
- removed IC1: TCAN3413DR, LHRS_Passives:TCAN3413DR, symbol TCAN3413DR:TCAN3413DR
- removed R22, R23: 60, Resistor_SMD:R_0603_1608Metric_Pad0.98x0.95mm_HandSolder, symbol Device:R
- added D2: CDSOT23-T24CAN, LHRS_Passives:CDSOT23-T24CAN, symbol CDSOT23-T24CAN:CDSOT23-T24CAN
- added IC2: TCAN3413DR, LHRS_Passives:TCAN3413DR, symbol TCAN3413DR:TCAN3413DR
- added R4, R5: 60, Resistor_SMD:R_0603_1608Metric_Pad0.98x0.95mm_HandSolder, symbol Device:R
Connections:
- net 3.3v: now also IC2.3 (VCC), IC2.5 (SHDNV_IO)
- net CAN_H: now also D2.1 (CAN_H), IC2.7 (CANH), R4.1
- net CAN_L: now also D2.2 (CAN_L), IC2.6 (CANL)
- net CAN_RX: now also IC2.4 (RXD)
- net CAN_TX: now also IC2.1 (TXD)
- net GND: now also D2.3 (GND), IC2.2 (GND), IC2.8 (STB)
- net at C8.2: now also R4.2, R5.1
- net at JP2.1 (A): now also R5.2

Commit message: added debug led
Parts:
- renumbered D2 to D9, R4 to R11, R5 to R12
Changed lines of the file:
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@@
 		(dnp no)
 		(fields_autoplaced yes)
-		(property "Reference" "D2"
+		(property "Reference" "D9"
 			(at 196.85 46.99 0)
 			(effects
@@
 			(project ""
 				(path "/2365a867-6254-4a7c-9718-f325e0bbac5c/7a8f5d40-8cff-476b-a6d6-a001c957bc73"
-					(reference "D2")
+					(reference "D9")
 					(unit 1)
 				)
@@
 		(on_board yes)
 		(dnp no)
-		(property "Reference" "R5"
+		(property "Reference" "R12"
 			(at 201.93 80.01 90)
 			(effects
@@
 			(project "kk36984"
 				(path "/2365a867-6254-4a7c-9718-f325e0bbac5c/7a8f5d40-8cff-476b-a6d6-a001c957bc73"
-					(reference "R5")
+					(reference "R12")
 					(unit 1)
 				)
@@
 		(on_board yes)
 		(dnp no)
-		(property "Reference" "R4"
+		(property "Reference" "R11"
 			(at 176.53 80.01 90)
 			(effects
@@
 			(project ""
 				(path "/2365a867-6254-4a7c-9718-f325e0bbac5c/7a8f5d40-8cff-476b-a6d6-a001c957bc73"
-					(reference "R4")
-					(unit 1)
-				)
+					(reference "R11")
+					(unit 1)
+				)

Commit message: added calcs, cleaned up, addressed comments
Parts:
- renumbered C5 to C26, C6 to C27, C7 to C28, C8 to C29, D9 to D12, IC2 to IC3, R11 to R23, R12 to R24
Changed lines of the file:
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@@
 		(in_pos_files yes)
 		(dnp no)
-		(property "Reference" "C8"
+		(property "Reference" "C29"
 			(at 194.564 88.646 0)
 			(show_name no)
@@
 			(project "PS-HVCarrier"
 				(path "/2365a867-6254-4a7c-9718-f325e0bbac5c/7a8f5d40-8cff-476b-a6d6-a001c957bc73"
-					(reference "C8")
+					(reference "C29")
 					(unit 1)
 				)
@@
 		(dnp no)
 		(fields_autoplaced yes)
-		(property "Reference" "D9"
+		(property "Reference" "D12"
 			(at 196.85 46.99 0)
 			(show_name no)
@@
 			(project "PS-HVCarrier"
 				(path "/2365a867-6254-4a7c-9718-f325e0bbac5c/7a8f5d40-8cff-476b-a6d6-a001c957bc73"
-					(reference "D9")
+					(reference "D12")
 					(unit 1)
 				)
@@
 		(in_pos_files yes)
 		(dnp no)
-		(property "Reference" "R12"
+		(property "Reference" "R24"
 			(at 201.93 80.01 90)
 			(show_name no)
@@
 			(project "PS-HVCarrier"
 				(path "/2365a867-6254-4a7c-9718-f325e0bbac5c/7a8f5d40-8cff-476b-a6d6-a001c957bc73"
-					(reference "R12")
+					(reference "R24")
 					(unit 1)
 				)
@@
 		(in_pos_files yes)
 		(dnp no)
-		(property "Reference" "C7"
+		(property "Reference" "C28"
 			(at 88.138 73.66 0)
 			(show_name no)
@@
 			(project "PS-HVCarrier"
 				(path "/2365a867-6254-4a7c-9718-f325e0bbac5c/7a8f5d40-8cff-476b-a6d6-a001c957bc73"
-					(reference "C7")
+					(reference "C28")
 					(unit 1)
 				)
@@
 		(in_pos_files yes)
 		(dnp no)
-		(property "Reference" "R11"
+		(property "Reference" "R23"
 			(at 176.53 80.01 90)
 			(show_name no)
@@
 			(project "PS-HVCarrier"
 				(path "/2365a867-6254-4a7c-9718-f325e0bbac5c/7a8f5d40-8cff-476b-a6d6-a001c957bc73"
-					(reference "R11")
+					(reference "R23")
 					(unit 1)
 				)
@@
 		(dnp no)
 		(fields_autoplaced yes)
-		(property "Reference" "IC2"
+		(property "Reference" "IC3"
 			(at 128.27 63.5 0)
 			(show_name no)
@@
 			(project "PS-HVCarrier"
 				(path "/2365a867-6254-4a7c-9718-f325e0bbac5c/7a8f5d40-8cff-476b-a6d6-a001c957bc73"
-					(reference "IC2")
+					(reference "IC3")
 					(unit 1)
 				)
@@
 		(in_pos_files yes)
 		(dnp no)
-		(property "Reference" "C6"
+		(property "Reference" "C27"
 			(at 76.2 73.66 0)
 			(show_name no)
@@
 			(project "PS-HVCarrier"
 				(path "/2365a867-6254-4a7c-9718-f325e0bbac5c/7a8f5d40-8cff-476b-a6d6-a001c957bc73"
-					(reference "C6")
+					(reference "C27")
 					(unit 1)
 				)
@@
 		(in_pos_files yes)
 		(dnp no)
-		(property "Reference" "C5"
+		(property "Reference" "C26"
 			(at 65.278 73.66 0)
 			(show_name no)
@@
 			(project "PS-HVCarrier"
 				(path "/2365a867-6254-4a7c-9718-f325e0bbac5c/7a8f5d40-8cff-476b-a6d6-a001c957bc73"
-					(reference "C5")
-					(unit 1)
-				)
+					(reference "C26")
+					(unit 1)
+				)

Commit message: changed fully to 48 pin MCU
Parts:
- renumbered C26 to C12, C27 to C13, C28 to C14, C29 to C15, D12 to D9, R23 to R15, R24 to R16
Changed lines of the file:
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@@
 		(in_pos_files yes)
 		(dnp no)
-		(property "Reference" "C29"
+		(property "Reference" "C15"
 			(at 194.564 88.646 0)
 			(show_name no)
@@
 			(project "PS-HVCarrier"
 				(path "/2365a867-6254-4a7c-9718-f325e0bbac5c/7a8f5d40-8cff-476b-a6d6-a001c957bc73"
-					(reference "C29")
+					(reference "C15")
 					(unit 1)
 				)
@@
 		(dnp no)
 		(fields_autoplaced yes)
-		(property "Reference" "D12"
+		(property "Reference" "D9"
 			(at 196.85 46.99 0)
 			(show_name no)
@@
 			(project "PS-HVCarrier"
 				(path "/2365a867-6254-4a7c-9718-f325e0bbac5c/7a8f5d40-8cff-476b-a6d6-a001c957bc73"
-					(reference "D12")
+					(reference "D9")
 					(unit 1)
 				)
@@
 		(in_pos_files yes)
 		(dnp no)
-		(property "Reference" "R24"
+		(property "Reference" "R16"
 			(at 201.93 80.01 90)
 			(show_name no)
@@
 			(project "PS-HVCarrier"
 				(path "/2365a867-6254-4a7c-9718-f325e0bbac5c/7a8f5d40-8cff-476b-a6d6-a001c957bc73"
-					(reference "R24")
+					(reference "R16")
 					(unit 1)
 				)
@@
 		(in_pos_files yes)
 		(dnp no)
-		(property "Reference" "C28"
+		(property "Reference" "C14"
 			(at 88.138 73.66 0)
 			(show_name no)
@@
 			(project "PS-HVCarrier"
 				(path "/2365a867-6254-4a7c-9718-f325e0bbac5c/7a8f5d40-8cff-476b-a6d6-a001c957bc73"
-					(reference "C28")
+					(reference "C14")
 					(unit 1)
 				)
@@
 		(in_pos_files yes)
 		(dnp no)
-		(property "Reference" "R23"
+		(property "Reference" "R15"
 			(at 176.53 80.01 90)
 			(show_name no)
@@
 			(project "PS-HVCarrier"
 				(path "/2365a867-6254-4a7c-9718-f325e0bbac5c/7a8f5d40-8cff-476b-a6d6-a001c957bc73"
-					(reference "R23")
+					(reference "R15")
 					(unit 1)
 				)
@@
 		(in_pos_files yes)
 		(dnp no)
-		(property "Reference" "C27"
+		(property "Reference" "C13"
 			(at 76.2 73.66 0)
 			(show_name no)
@@
 			(project "PS-HVCarrier"
 				(path "/2365a867-6254-4a7c-9718-f325e0bbac5c/7a8f5d40-8cff-476b-a6d6-a001c957bc73"
-					(reference "C27")
+					(reference "C13")
 					(unit 1)
 				)
@@
 		(in_pos_files yes)
 		(dnp no)
-		(property "Reference" "C26"
+		(property "Reference" "C12"
 			(at 65.278 73.66 0)
 			(show_name no)
@@
 			(project "PS-HVCarrier"
 				(path "/2365a867-6254-4a7c-9718-f325e0bbac5c/7a8f5d40-8cff-476b-a6d6-a001c957bc73"
-					(reference "C26")
-					(unit 1)
-				)
+					(reference "C12")
+					(unit 1)
+				)
