File: hardware/CAN_Transceiver.kicad_sch (KiCad schematic)
At the start: 9 parts, among them IC1 TCAN3413DR

Commit message: labeled + stm32 cube layout
Parts:
- renumbered C5 to C1, C6 to C2, C7 to C3, C8 to C4, D8 to D1, JP2 to JP1, R22 to R2, R23 to R3
Changed lines of the file:
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@@
 		(on_board yes)
 		(dnp no)
-		(property "Reference" "C6"
+		(property "Reference" "C2"
 			(at 76.2 73.66 0)
 			(effects
@@
 			(project ""
 				(path "/2365a867-6254-4a7c-9718-f325e0bbac5c/8e4b18be-f701-4f79-b148-bbeadfa1a129"
-					(reference "C6")
+					(reference "C2")
 					(unit 1)
 				)
@@
 		(on_board yes)
 		(dnp no)
-		(property "Reference" "C8"
+		(property "Reference" "C4"
 			(at 194.564 88.646 0)
 			(effects
@@
 			(project ""
 				(path "/2365a867-6254-4a7c-9718-f325e0bbac5c/8e4b18be-f701-4f79-b148-bbeadfa1a129"
-					(reference "C8")
+					(reference "C4")
 					(unit 1)
 				)
@@
 		(dnp no)
 		(fields_autoplaced yes)
-		(property "Reference" "JP2"
+		(property "Reference" "JP1"
 			(at 215.9 78.74 0)
 			(effects
@@
 			(project ""
 				(path "/2365a867-6254-4a7c-9718-f325e0bbac5c/8e4b18be-f701-4f79-b148-bbeadfa1a129"
-					(reference "JP2")
+					(reference "JP1")
 					(unit 1)
 				)
@@
 		(on_board yes)
 		(dnp no)
-		(property "Reference" "C7"
+		(property "Reference" "C3"
 			(at 88.138 73.66 0)
 			(effects
@@
 			(project ""
 				(path "/2365a867-6254-4a7c-9718-f325e0bbac5c/8e4b18be-f701-4f79-b148-bbeadfa1a129"
-					(reference "C7")
+					(reference "C3")
 					(unit 1)
 				)
@@
 		(on_board yes)
 		(dnp no)
-		(property "Reference" "C5"
+		(property "Reference" "C1"
 			(at 65.278 73.66 0)
 			(effects
@@
 			(project ""
 				(path "/2365a867-6254-4a7c-9718-f325e0bbac5c/8e4b18be-f701-4f79-b148-bbeadfa1a129"
-					(reference "C5")
+					(reference "C1")
 					(unit 1)
 				)
@@
 		(on_board yes)
 		(dnp no)
-		(property "Reference" "R23"
+		(property "Reference" "R3"
 			(at 201.93 80.01 90)
 			(effects
@@
 			(project "kk36984"
 				(path "/2365a867-6254-4a7c-9718-f325e0bbac5c/8e4b18be-f701-4f79-b148-bbeadfa1a129"
-					(reference "R23")
+					(reference "R3")
 					(unit 1)
 				)
@@
 		(dnp no)
 		(fields_autoplaced yes)
-		(property "Reference" "D8"
+		(property "Reference" "D1"
 			(at 196.85 46.99 0)
 			(effects
@@
 			(project ""
 				(path "/2365a867-6254-4a7c-9718-f325e0bbac5c/8e4b18be-f701-4f79-b148-bbeadfa1a129"
-					(reference "D8")
+					(reference "D1")
 					(unit 1)
 				)
@@
 		(on_board yes)
 		(dnp no)
-		(property "Reference" "R22"
+		(property "Reference" "R2"
 			(at 176.53 80.01 90)
 			(effects
@@
 			(project ""
 				(path "/2365a867-6254-4a7c-9718-f325e0bbac5c/8e4b18be-f701-4f79-b148-bbeadfa1a129"
-					(reference "R22")
-					(unit 1)
-				)
+					(reference "R2")
+					(unit 1)
+				)

Commit message: added debug led
Parts:
- renumbered D1 to D8, R3 to R10, R2 to R9
Changed lines of the file:
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@@
 		(on_board yes)
 		(dnp no)
-		(property "Reference" "R3"
+		(property "Reference" "R10"
 			(at 201.93 80.01 90)
 			(effects
@@
 			(project "kk36984"
 				(path "/2365a867-6254-4a7c-9718-f325e0bbac5c/8e4b18be-f701-4f79-b148-bbeadfa1a129"
-					(reference "R3")
+					(reference "R10")
 					(unit 1)
 				)
@@
 		(dnp no)
 		(fields_autoplaced yes)
-		(property "Reference" "D1"
+		(property "Reference" "D8"
 			(at 196.85 46.99 0)
 			(effects
@@
 			(project ""
 				(path "/2365a867-6254-4a7c-9718-f325e0bbac5c/8e4b18be-f701-4f79-b148-bbeadfa1a129"
-					(reference "D1")
+					(reference "D8")
 					(unit 1)
 				)
@@
 		(on_board yes)
 		(dnp no)
-		(property "Reference" "R2"
+		(property "Reference" "R9"
 			(at 176.53 80.01 90)
 			(effects
@@
 			(project ""
 				(path "/2365a867-6254-4a7c-9718-f325e0bbac5c/8e4b18be-f701-4f79-b148-bbeadfa1a129"
-					(reference "R2")
-					(unit 1)
-				)
+					(reference "R9")
+					(unit 1)
+				)

Commit message: added calcs, cleaned up, addressed comments
Parts:
- renumbered C1 to C22, C2 to C23, C3 to C24, C4 to C25, D8 to D11, IC1 to IC2, R9 to R21, R10 to R22
Changed lines of the file:
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@@
 		(in_pos_files yes)
 		(dnp no)
-		(property "Reference" "C2"
+		(property "Reference" "C23"
 			(at 76.2 73.66 0)
 			(show_name no)
@@
 			(project "PS-HVCarrier"
 				(path "/2365a867-6254-4a7c-9718-f325e0bbac5c/8e4b18be-f701-4f79-b148-bbeadfa1a129"
-					(reference "C2")
+					(reference "C23")
 					(unit 1)
 				)
@@
 		(in_pos_files yes)
 		(dnp no)
-		(property "Reference" "C4"
+		(property "Reference" "C25"
 			(at 194.564 88.646 0)
 			(show_name no)
@@
 			(project "PS-HVCarrier"
 				(path "/2365a867-6254-4a7c-9718-f325e0bbac5c/8e4b18be-f701-4f79-b148-bbeadfa1a129"
-					(reference "C4")
+					(reference "C25")
 					(unit 1)
 				)
@@
 		(in_pos_files yes)
 		(dnp no)
-		(property "Reference" "C3"
+		(property "Reference" "C24"
 			(at 88.138 73.66 0)
 			(show_name no)
@@
 			(project "PS-HVCarrier"
 				(path "/2365a867-6254-4a7c-9718-f325e0bbac5c/8e4b18be-f701-4f79-b148-bbeadfa1a129"
-					(reference "C3")
+					(reference "C24")
 					(unit 1)
 				)
@@
 		(in_pos_files yes)
 		(dnp no)
-		(property "Reference" "C1"
+		(property "Reference" "C22"
 			(at 65.278 73.66 0)
 			(show_name no)
@@
 			(project "PS-HVCarrier"
 				(path "/2365a867-6254-4a7c-9718-f325e0bbac5c/8e4b18be-f701-4f79-b148-bbeadfa1a129"
-					(reference "C1")
+					(reference "C22")
 					(unit 1)
 				)
@@
 		(in_pos_files yes)
 		(dnp no)
-		(property "Reference" "R10"
+		(property "Reference" "R22"
 			(at 201.93 80.01 90)
 			(show_name no)
@@
 			(project "PS-HVCarrier"
 				(path "/2365a867-6254-4a7c-9718-f325e0bbac5c/8e4b18be-f701-4f79-b148-bbeadfa1a129"
-					(reference "R10")
+					(reference "R22")
 					(unit 1)
 				)
@@
 		(dnp no)
 		(fields_autoplaced yes)
-		(property "Reference" "D8"
+		(property "Reference" "D11"
 			(at 196.85 46.99 0)
 			(show_name no)
@@
 			(project "PS-HVCarrier"
 				(path "/2365a867-6254-4a7c-9718-f325e0bbac5c/8e4b18be-f701-4f79-b148-bbeadfa1a129"
-					(reference "D8")
+					(reference "D11")
 					(unit 1)
 				)
@@
 		(dnp no)
 		(fields_autoplaced yes)
-		(property "Reference" "IC1"
+		(property "Reference" "IC2"
 			(at 128.27 63.5 0)
 			(show_name no)
@@
 			(project "PS-HVCarrier"
 				(path "/2365a867-6254-4a7c-9718-f325e0bbac5c/8e4b18be-f701-4f79-b148-bbeadfa1a129"
-					(reference "IC1")
+					(reference "IC2")
 					(unit 1)
 				)
@@
 		(in_pos_files yes)
 		(dnp no)
-		(property "Reference" "R9"
+		(property "Reference" "R21"
 			(at 176.53 80.01 90)
 			(show_name no)
@@
 			(project "PS-HVCarrier"
 				(path "/2365a867-6254-4a7c-9718-f325e0bbac5c/8e4b18be-f701-4f79-b148-bbeadfa1a129"
-					(reference "R9")
-					(unit 1)
-				)
+					(reference "R21")
+					(unit 1)
+				)

Commit message: changed fully to 48 pin MCU
Parts:
- renumbered C24 to C10, C25 to C11, C22 to C8, C23 to C9, D11 to D8, R21 to R13, R22 to R14
Changed lines of the file:
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@@
 		(in_pos_files yes)
 		(dnp no)
-		(property "Reference" "C23"
+		(property "Reference" "C9"
 			(at 76.2 73.66 0)
 			(show_name no)
@@
 			(project "PS-HVCarrier"
 				(path "/2365a867-6254-4a7c-9718-f325e0bbac5c/8e4b18be-f701-4f79-b148-bbeadfa1a129"
-					(reference "C23")
+					(reference "C9")
 					(unit 1)
 				)
@@
 		(in_pos_files yes)
 		(dnp no)
-		(property "Reference" "C25"
+		(property "Reference" "C11"
 			(at 194.564 88.646 0)
 			(show_name no)
@@
 			(project "PS-HVCarrier"
 				(path "/2365a867-6254-4a7c-9718-f325e0bbac5c/8e4b18be-f701-4f79-b148-bbeadfa1a129"
-					(reference "C25")
+					(reference "C11")
 					(unit 1)
 				)
@@
 		(in_pos_files yes)
 		(dnp no)
-		(property "Reference" "C24"
+		(property "Reference" "C10"
 			(at 88.138 73.66 0)
 			(show_name no)
@@
 			(project "PS-HVCarrier"
 				(path "/2365a867-6254-4a7c-9718-f325e0bbac5c/8e4b18be-f701-4f79-b148-bbeadfa1a129"
-					(reference "C24")
+					(reference "C10")
 					(unit 1)
 				)
@@
 		(in_pos_files yes)
 		(dnp no)
-		(property "Reference" "C22"
+		(property "Reference" "C8"
 			(at 65.278 73.66 0)
 			(show_name no)
@@
 			(project "PS-HVCarrier"
 				(path "/2365a867-6254-4a7c-9718-f325e0bbac5c/8e4b18be-f701-4f79-b148-bbeadfa1a129"
-					(reference "C22")
+					(reference "C8")
 					(unit 1)
 				)
@@
 		(in_pos_files yes)
 		(dnp no)
-		(property "Reference" "R22"
+		(property "Reference" "R14"
 			(at 201.93 80.01 90)
 			(show_name no)
@@
 			(project "PS-HVCarrier"
 				(path "/2365a867-6254-4a7c-9718-f325e0bbac5c/8e4b18be-f701-4f79-b148-bbeadfa1a129"
-					(reference "R22")
+					(reference "R14")
 					(unit 1)
 				)
@@
 		(dnp no)
 		(fields_autoplaced yes)
-		(property "Reference" "D11"
+		(property "Reference" "D8"
 			(at 196.85 46.99 0)
 			(show_name no)
@@
 			(project "PS-HVCarrier"
 				(path "/2365a867-6254-4a7c-9718-f325e0bbac5c/8e4b18be-f701-4f79-b148-bbeadfa1a129"
-					(reference "D11")
+					(reference "D8")
 					(unit 1)
 				)
@@
 		(in_pos_files yes)
 		(dnp no)
-		(property "Reference" "R21"
+		(property "Reference" "R13"
 			(at 176.53 80.01 90)
 			(show_name no)
@@
 			(project "PS-HVCarrier"
 				(path "/2365a867-6254-4a7c-9718-f325e0bbac5c/8e4b18be-f701-4f79-b148-bbeadfa1a129"
-					(reference "R21")
-					(unit 1)
-				)
+					(reference "R13")
+					(unit 1)
+				)

Commit message: fixed ERC, made it look pretty
Parts:
- removed C11: 0.1u, Capacitor_SMD:C_0603_1608Metric_Pad1.08x0.95mm_HandSolder, symbol ECE319K:C
- removed D8: CDSOT23-T24CAN, LHRS_Passives:CDSOT23-T24CAN, symbol CDSOT23-T24CAN:CDSOT23-T24CAN
- removed IC2: TCAN3413DR, LHRS_Passives:TCAN3413DR, symbol TCAN3413DR:TCAN3413DR
- added C11: 0.1u, Capacitor_SMD:C_0603_1608Metric_Pad1.08x0.95mm_HandSolder, symbol Device:C
- added IC1: TCAN3413DR, LHRS_Passives:TCAN3413DR, symbol lhrs_ics:TCAN3413DR
- added U3: CDSOT23-T24CAN, LHRS_ICs:CDSOT23-T24CAN, symbol lhrs_ics:CDSOT23-T24CAN
Connections:
- net 3.3v: now also IC1.3 (VCC), IC1.5 (SHDNV_IO)
- net CAN_H: now also IC1.7 (CANH), U3.1 (CAN_H)
- net CAN_L: now also IC1.6 (CANL), U3.2 (CAN_L)
- net CAN_RX: now also IC1.4 (RXD)
- net CAN_TX: now also IC1.1 (TXD)
- net GND: now also C11.2, IC1.2 (GND), IC1.8 (STB), U3.3 (GND)
- net at R13.2, R14.1: now also C11.1

Commit message: added outside test points, removed unncessary symbol fields
Parts:
- IC1: Height 1.75 -> (none); Manufacturer_Name Texas Instruments -> (none); Mouser Part Number 595-TCAN3413DR -> (none); Mouser Price/Stock - -> (none)
Changed lines of the file:
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@@
-			)
-		)
-		(property "LCSC" ""
-			(at 189.23 88.9 0)
-			(hide yes)
-			(show_name no)
-			(do_not_autoplace no)
-			(effects
-				(font
-					(size 1.27 1.27)
-				)
 			)
 		)
@@
 		)
 		(property "P/N" "MLASH168SB7104KTNA01"
-			(at 73.66 74.93 0)
-			(hide yes)
-			(show_name no)
-			(do_not_autoplace no)
-			(effects
-				(font
-					(size 1.27 1.27)
-				)
-			)
-		)
-		(property "LCSC" ""
 			(at 73.66 74.93 0)
 			(hide yes)
@@
 			)
 		)
-		(property "LCSC" ""
-			(at 215.9 85.09 0)
-			(hide yes)
-			(show_name no)
-			(do_not_autoplace no)
-			(effects
-				(font
-					(size 1.27 1.27)
-				)
-			)
-		)
 		(pin "1"
 		)
@@
 			)
 		)
-		(property "LCSC" ""
-			(at 85.09 74.93 0)
-			(hide yes)
-			(show_name no)
-			(do_not_autoplace no)
-			(effects
-				(font
-					(size 1.27 1.27)
-				)
-			)
-		)
 		(pin "1"
 		)
@@
 		)
 		(property "P/N" "GRM21BR61H106KE43K"
-			(at 62.23 74.93 0)
-			(hide yes)
-			(show_name no)
-			(do_not_autoplace no)
-			(effects
-				(font
-					(size 1.27 1.27)
-				)
-			)
-		)
-		(property "LCSC" ""
 			(at 62.23 74.93 0)
 			(hide yes)
@@
 			)
 		)
-		(property "Height" "1.75"
-			(at 140.97 466.04 0)
-			(hide yes)
-			(show_name no)
-			(do_not_autoplace no)
-			(effects
-				(font
-					(size 1.27 1.27)
-				)
-				(justify left top)
-			)
-		)
-		(property "Mouser Part Number" "595-TCAN3413DR"
-			(at 140.97 566.04 0)
-			(hide yes)
-			(show_name no)
-			(do_not_autoplace no)
-			(effects
-				(font
-					(size 1.27 1.27)
-				)
-				(justify left top)
-			)
-		)
-		(property "Mouser Price/Stock" "-"
-			(at 140.97 666.04 0)
-			(hide yes)
-			(show_name no)
-			(do_not_autoplace no)
-			(effects
-				(font
-					(size 1.27 1.27)
-				)
-				(justify left top)
-			)
-		)
-		(property "Manufacturer_Name" "Texas Instruments"
-			(at 140.97 766.04 0)
-			(hide yes)
-			(show_name no)
-			(do_not_autoplace no)
-			(effects
-				(font
-					(size 1.27 1.27)
-				)
-				(justify left top)
-			)
-		)
 		(property "P/N" "TCAN3413DR"
 			(at 140.97 866.04 0)
@@
 		)
 		(property "LCSC P/N" "C22433320"
-			(at 111.76 71.12 0)
-			(hide yes)
-			(show_name no)
-			(do_not_autoplace no)
-			(effects
-				(font
-					(size 1.27 1.27)
-				)
-			)
-		)
-		(property "LCSC" ""
 			(at 111.76 71.12 0)
 			(hide yes)
@@
 			)
 		)
-		(property "LCSC" ""
-			(at 201.93 85.09 90)
-			(hide yes)
-			(show_name no)
-			(do_not_autoplace no)
-			(effects
-				(font
-					(size 1.27 1.27)
-				)
-			)
-		)
 		(pin "1"
 		)
@@
 		)
 		(property "P/N" "CRCW060360R4FKEA"
-			(at 176.53 85.09 90)
-			(hide yes)
-			(show_name no)
-			(do_not_autoplace no)
-			(effects
-				(font
-					(size 1.27 1.27)
-				)
-			)
-		)
-		(property "LCSC" ""
 			(at 176.53 85.09 90)
 			(hide yes)
@@
 			(at 194.31 55.88 0)
 			(hide yes)
-			(show_name no)
-			(do_not_autoplace no)
-			(effects
-				(font
-					(size 1.27 1.27)
-				)
-			)
-		)
-		(property "LCSC" ""
-			(at 194.31 55.88 0)
-			(hide yes)
