File: hardware/CAN_Transceiver.kicad_sch (KiCad schematic)
At the start: 9 parts, among them IC1 TCAN3413DR, U3 CDSOT23-T24CAN

Commit message: updated kicad sharepoint, added pn
Parts:
- C11: P/N (none) -> MLASH168SB7104KTNA01
Changed lines of the file:
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@@
+			)
+		)
+		(property "P/N" "MLASH168SB7104KTNA01"
+			(at 189.23 88.9 0)
+			(hide yes)
+			(show_name no)
+			(do_not_autoplace no)
+			(effects
+				(font
+					(size 1.27 1.27)
+				)
 			)
 		)
