File: hardware/AMC3311_OpAmp.kicad_sch (KiCad schematic)
At the start: 16 parts, among them U13 TLV9002QDRQ1

Commit message: saving
Other:
- note added: "+-1% Tolerance Nominal: 1.5M + 20k divider, ratio of 0.013158 140 * 0.013158 = 1.8421 Highest reading: 1,485,000 (min) + 20,200 (max), ratio of 0.013419 140* 0.013419 = 1.8787 (+1.99%) Lowest reading: 1,515,000 (max) + 19,800 (min), ratio of 0.012900 140 * 0.012900 = 1.8060 (-1.96%)"
- note added: "1% Resistor Divider Worst Case"
- note added: "AMC3311 ADC Output Calc"
- note added: "Ratio = V_AMC3311_MAX / V_HV_MAX = 2.0V/140V = 0.014286V/V Op_amp_gain = 1.0 V_Out_Diff = = Vin_HV * Ratio * Op_amp_gain = Vin_HV * 0.014286 * 1 V_ADC = V_Out_Diff * Op_amp_gain"
- note added: "Vin_HV = Motor_ADC = Precharge_ADC 0V = 0V 35V = 0.5V 70V = 1V 105V = 1.5V 140V = 2.0V"
- note added: "Voltage Error @ 140V for 1% tolerance Divider error: +-2% and +-2.8V difference"
Changed lines of the file:
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@@
 	(generator_version "10.0")
 	(paper "A4")
+	(rectangle
+		(start 12.7 155.956)
+		(end 89.535 197.485)
+		(stroke
+			(width 0)
+			(type default)
+		)
+		(fill
+			(type none)
+		)
+	)
+	(rectangle
+		(start 91.567 155.956)
+		(end 174.625 196.85)
+		(stroke
+			(width 0)
+			(type default)
+		)
+		(fill
+			(type none)
+		)
+	)
+	(text "1% Resistor Divider Worst Case"
+		(exclude_from_sim no)
+		(at 107.95 158.115 0)
+		(effects
+			(font
+				(size 1.27 1.27)
+			)
+		)
+	)
+	(text "Voltage Error @ 140V for 1% tolerance\nDivider error: +-2% and +-2.8V difference"
+		(exclude_from_sim no)
+		(at 133.35 184.785 0)
+		(effects
+			(font
+				(size 1.27 1.27)
+			)
+		)
+	)
+	(text "Ratio = V_AMC3311_MAX / V_HV_MAX = 2.0V/140V = 0.014286V/V\n\nOp_amp_gain = 1.0\n\nV_Out_Diff = = Vin_HV * Ratio * Op_amp_gain = Vin_HV * 0.014286 * 1\n\nV_ADC = V_Out_Diff * Op_amp_gain"
+		(exclude_from_sim no)
+		(at 52.07 169.545 0)
+		(effects
+			(font
+				(size 1.27 1.27)
+			)
+		)
+	)
+	(text "AMC3311 ADC Output Calc"
+		(exclude_from_sim no)
+		(at 26.67 158.115 0)
+		(effects
+			(font
+				(size 1.27 1.27)
+			)
+		)
+	)
+	(text "+-1% Tolerance\nNominal: 1.5M + 20k divider, ratio of 0.013158\n140 * 0.013158 = 1.8421\n\nHighest reading: 1,485,000 (min) + 20,200 (max), ratio of 0.013419\n140* 0.013419 = 1.8787 (+1.99%)\n\nLowest reading: 1,515,000 (max) + 19,800 (min), ratio of 0.012900\n140 * 0.012900 = 1.8060 (-1.96%)"
+		(exclude_from_sim no)
+		(at 134.62 170.815 0)
+		(effects
+			(font
+				(size 1.27 1.27)
+			)
+		)
+	)
+	(text "Vin_HV = Motor_ADC = Precharge_ADC\n\n0V = 0V\n35V = 0.5V\n70V = 1V\n105V = 1.5V\n140V = 2.0V"
+		(exclude_from_sim no)
+		(at 52.07 187.325 0)
+		(effects
+			(font
+				(size 1.27 1.27)
+			)
+		)
+	)
 	(junction
 		(at 119.38 66.04)

Commit message: added outside test points, removed unncessary symbol fields
Parts:
- D19, D20, D21, D22: Mouser Part Number 576-SMF3.3 -> (none)
- U13: Digikey P/N 296-TLV9002QDRQ1CT-ND -> (none); JLC P/N C2860922 -> (none); Mouser P/N 595-TLV9002QDRQ1 -> (none)

Commit message: updated kicad sharepoint, added pn
Parts:
- C80: renamed from C84; P/N (none) -> UMK107B7102MAHT
- C81: renamed from C85; P/N (none) -> UMK107B7102MAHT
- C82: renamed from C86; P/N (none) -> MLASH168SB7104KTNA01
- R71: renamed from R73; P/N (none) -> CRCW060310K0FKEI
- R72: renamed from R74; P/N (none) -> CRCW060310K0FKEI
- R73: renamed from R75; P/N (none) -> CRCW060310K0FKEI
- R74: renamed from R76; P/N (none) -> CRCW060310K0FKEI
- R75: renamed from R77; P/N (none) -> CRCW060310K0FKEI
- R76: renamed from R78; P/N (none) -> CRCW060310K0FKEI
- renumbered TP35 to TP34, TP36 to TP35, U13 to U12
