File: hardware/PowerProtection.kicad_sch (KiCad schematic)
At the start: 17 parts, among them U7 LM76202QPWPRQ1

Commit message: labeled + stm32 cube layout
Parts:
- renumbered C20 to C33, C1 to C34, C25 to C35, C2 to C36, C23 to C37, D2 to D6, D10 to D7, R12 to R17, R13 to R18, R15 to R19, R27 to R20, R20 to R21, R30 to R22, R1 to R23, R31 to R24, R23 to R25, U7 to U5
Changed lines of the file:
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@@
 		(dnp no)
 		(fields_autoplaced yes)
-		(property "Reference" "#PWR04"
+		(property "Reference" "#PWR040"
 			(at 146.05 86.36 0)
 			(effects
@@
 			(project "PeripheralSOM"
 				(path "/2365a867-6254-4a7c-9718-f325e0bbac5c/904fa10a-747c-46cf-90d1-33d76069dc5d/429789a2-93db-48e4-a73d-32df605a2afb"
-					(reference "#PWR04")
+					(reference "#PWR040")
 					(unit 1)
 				)
@@
 		(dnp no)
 		(fields_autoplaced yes)
-		(property "Reference" "#PWR024"
+		(property "Reference" "#PWR038"
 			(at 99.06 57.15 0)
 			(effects
@@
 			(project "PeripheralSOM"
 				(path "/2365a867-6254-4a7c-9718-f325e0bbac5c/904fa10a-747c-46cf-90d1-33d76069dc5d/429789a2-93db-48e4-a73d-32df605a2afb"
-					(reference "#PWR024")
+					(reference "#PWR038")
 					(unit 1)
 				)
@@
 		(on_board yes)
 		(dnp yes)
-		(property "Reference" "R31"
+		(property "Reference" "R24"
 			(at 153.67 28.448 90)
 			(effects
@@
 			(project "PeripheralSOM"
 				(path "/2365a867-6254-4a7c-9718-f325e0bbac5c/904fa10a-747c-46cf-90d1-33d76069dc5d/429789a2-93db-48e4-a73d-32df605a2afb"
-					(reference "R31")
+					(reference "R24")
 					(unit 1)
 				)
@@
 		(dnp no)
 		(fields_autoplaced yes)
-		(property "Reference" "D10"
+		(property "Reference" "D7"
 			(at 161.29 35.5599 90)
 			(effects
@@
 			(project ""
 				(path "/2365a867-6254-4a7c-9718-f325e0bbac5c/904fa10a-747c-46cf-90d1-33d76069dc5d/429789a2-93db-48e4-a73d-32df605a2afb"
-					(reference "D10")
+					(reference "D7")
 					(unit 1)
 				)
@@
 		(dnp no)
 		(fields_autoplaced yes)
-		(property "Reference" "#PWR045"
+		(property "Reference" "#PWR037"
 			(at 97.79 30.48 0)
 			(effects
@@
 			(project "BPS-PeripheralSOM"
 				(path "/2365a867-6254-4a7c-9718-f325e0bbac5c/904fa10a-747c-46cf-90d1-33d76069dc5d/429789a2-93db-48e4-a73d-32df605a2afb"
-					(reference "#PWR045")
+					(reference "#PWR037")
 					(unit 1)
 				)
@@
 		(dnp no)
 		(fields_autoplaced yes)
-		(property "Reference" "C25"
+		(property "Reference" "C35"
 			(at 110.49 46.355 0)
 			(effects
@@
 			(project "BPS-PeripheralSOM"
 				(path "/2365a867-6254-4a7c-9718-f325e0bbac5c/904fa10a-747c-46cf-90d1-33d76069dc5d/429789a2-93db-48e4-a73d-32df605a2afb"
-					(reference "C25")
+					(reference "C35")
 					(unit 1)
 				)
@@
 		(dnp no)
 		(fields_autoplaced yes)
-		(property "Reference" "#PWR030"
+		(property "Reference" "#PWR039"
 			(at 120.65 50.8 0)
 			(effects
@@
 			(project "PeripheralSOM"
 				(path "/2365a867-6254-4a7c-9718-f325e0bbac5c/904fa10a-747c-46cf-90d1-33d76069dc5d/429789a2-93db-48e4-a73d-32df605a2afb"
-					(reference "#PWR030")
+					(reference "#PWR039")
 					(unit 1)
 				)
@@
 		(dnp no)
 		(fields_autoplaced yes)
-		(property "Reference" "#PWR022"
+		(property "Reference" "#PWR036"
 			(at 52.07 49.53 0)
 			(effects
@@
 			(project ""
 				(path "/2365a867-6254-4a7c-9718-f325e0bbac5c/904fa10a-747c-46cf-90d1-33d76069dc5d/429789a2-93db-48e4-a73d-32df605a2afb"
-					(reference "#PWR022")
+					(reference "#PWR036")
 					(unit 1)
 				)
@@
 		(on_board yes)
 		(dnp no)
-		(property "Reference" "#FLG02"
+		(property "Reference" "#FLG08"
 			(at 130.81 29.845 0)
 			(effects
@@
 			(project "PeripheralSOM"
 				(path "/2365a867-6254-4a7c-9718-f325e0bbac5c/904fa10a-747c-46cf-90d1-33d76069dc5d/429789a2-93db-48e4-a73d-32df605a2afb"
-					(reference "#FLG02")
+					(reference "#FLG08")
 					(unit 1)
 				)
@@
 		(on_board yes)
 		(dnp no)
-		(property "Reference" "C20"
+		(property "Reference" "C33"
 			(at 32.2072 35.6616 0)
 			(effects
@@
 			(project "BPS-PeripheralSOM"
 				(path "/2365a867-6254-4a7c-9718-f325e0bbac5c/904fa10a-747c-46cf-90d1-33d76069dc5d/429789a2-93db-48e4-a73d-32df605a2afb"
-					(reference "C20")
+					(reference "C33")
 					(unit 1)
 				)
@@
 		(dnp no)
 		(fields_autoplaced yes)
-		(property "Reference" "#PWR05"
+		(property "Reference" "#PWR041"
 			(at 157.48 86.36 0)
 			(effects
@@
 			(project "PeripheralSOM"
 				(path "/2365a867-6254-4a7c-9718-f325e0bbac5c/904fa10a-747c-46cf-90d1-33d76069dc5d/429789a2-93db-48e4-a73d-32df605a2afb"
-					(reference "#PWR05")
+					(reference "#PWR041")
 					(unit 1)
 				)
@@
 		(dnp no)
 		(fields_autoplaced yes)
-		(property "Reference" "R20"
+		(property "Reference" "R21"
 			(at 132.08 91.4399 0)
 			(effects
@@
 			(project "BPS-PeripheralSOM"
 				(path "/2365a867-6254-4a7c-9718-f325e0bbac5c/904fa10a-747c-46cf-90d1-33d76069dc5d/429789a2-93db-48e4-a73d-32df605a2afb"
-					(reference "R20")
+					(reference "R21")
 					(unit 1)
 				)
@@
 		(dnp no)
 		(fields_autoplaced yes)
-		(property "Reference" "R15"
+		(property "Reference" "R19"
 			(at 24.13 121.9199 0)
 			(effects
@@
 			(project "BPS-PeripheralSOM"
 				(path "/2365a867-6254-4a7c-9718-f325e0bbac5c/904fa10a-747c-46cf-90d1-33d76069dc5d/429789a2-93db-48e4-a73d-32df605a2afb"
-					(reference "R15")
+					(reference "R19")
 					(unit 1)
 				)
@@
 		(on_board yes)
 		(dnp no)
-		(property "Reference" "#FLG01"
+		(property "Reference" "#FLG07"
 			(at 29.21 29.845 0)
 			(effects
@@
 			(project "BPS-PeripheralSOM"
 				(path "/2365a867-6254-4a7c-9718-f325e0bbac5c/904fa10a-747c-46cf-90d1-33d76069dc5d/429789a2-93db-48e4-a73d-32df605a2afb"
-					(reference "#FLG01")
+					(reference "#FLG07")
 					(unit 1)
 				)
@@
 		(on_board yes)
 		(dnp no)
-		(property "Reference" "C23"
+		(property "Reference" "C37"
 			(at 133.8072 36.9316 0)
 			(effects
@@
 			(project "BPS-PeripheralSOM"
 				(path "/2365a867-6254-4a7c-9718-f325e0bbac5c/904fa10a-747c-46cf-90d1-33d76069dc5d/429789a2-93db-48e4-a73d-32df605a2afb"
-					(reference "C23")
+					(reference "C37")
 					(unit 1)
 				)
@@
 		(on_board yes)
 		(dnp no)
-		(property "Reference" "R1"
+		(property "Reference" "R23"
 			(at 147.828 87.7316 0)
 			(effects
@@
 			(project "PeripheralSOM"
 				(path "/2365a867-6254-4a7c-9718-f325e0bbac5c/904fa10a-747c-46cf-90d1-33d76069dc5d/429789a2-93db-48e4-a73d-32df605a2afb"
-					(reference "R1")
+					(reference "R23")
 					(unit 1)
 				)
@@
 		(dnp no)
 		(fields_autoplaced yes)
-		(property "Reference" "R23"
+		(property "Reference" "R25"
 			(at 160.02 88.265 0)
 			(effects
@@
 			(project "PeripheralSOM"
 				(path "/2365a867-6254-4a7c-9718-f325e0bbac5c/904fa10a-747c-46cf-90d1-33d76069dc5d/429789a2-93db-48e4-a73d-32df605a2afb"
-					(reference "R23")
+					(reference "R25")
 					(unit 1)
 				)
@@
 		(on_board yes)
 		(dnp no)
-		(property "Reference" "C2"
+		(property "Reference" "C36"
 			(at 123.6472 36.9316 0)
 			(effects
@@
 			(project "PeripheralSOM"
 				(path "/2365a867-6254-4a7c-9718-f325e0bbac5c/904fa10a-747c-46cf-90d1-33d76069dc5d/429789a2-93db-48e4-a73d-32df605a2afb"
-					(reference "C2")
+					(reference "C36")
 					(unit 1)
 				)
@@
 		(on_board yes)
 		(dnp no)
-		(property "Reference" "C1"
+		(property "Reference" "C34"
 			(at 43.6372 35.6616 0)
 			(effects
@@
 			(project "PeripheralSOM"
 				(path "/2365a867-6254-4a7c-9718-f325e0bbac5c/904fa10a-747c-46cf-90d1-33d76069dc5d/429789a2-93db-48e4-a73d-32df605a2afb"
-					(reference "C1")
+					(reference "C34")
 					(unit 1)
 				)
@@
 		(dnp no)
 		(fields_autoplaced yes)
-		(property "Reference" "R27"
+		(property "Reference" "R20"
 			(at 39.37 67.945 0)
 			(effects
@@
 			(project "PeripheralSOM"
 				(path "/2365a867-6254-4a7c-9718-f325e0bbac5c/904fa10a-747c-46cf-90d1-33d76069dc5d/429789a2-93db-48e4-a73d-32df605a2afb"
-					(reference "R27")
+					(reference "R20")
 					(unit 1)
 				)
@@
 		(on_board yes)
 		(dnp no)
-		(property "Reference" "D2"
+		(property "Reference" "D6"
 			(at 54.356 36.068 90)
 			(effects
@@
 			(project "BPS-PeripheralSOM"
 				(path "/2365a867-6254-4a7c-9718-f325e0bbac5c/904fa10a-747c-46cf-90d1-33d76069dc5d/429789a2-93db-48e4-a73d-32df605a2afb"
-					(reference "D2")
+					(reference "D6")
 					(unit 1)
 				)
@@
 		(dnp no)
 		(fields_autoplaced yes)
-		(property "Reference" "R30"
+		(property "Reference" "R22"
 			(at 144.78 35.5599 0)
 			(effects
@@
 			(project ""
 				(path "/2365a867-6254-4a7c-9718-f325e0bbac5c/904fa10a-747c-46cf-90d1-33d76069dc5d/429789a2-93db-48e4-a73d-32df605a2afb"
-					(reference "R30")
+					(reference "R22")
 					(unit 1)
 				)
@@
 		(dnp no)
 		(fields_autoplaced yes)
-		(property "Reference" "U7"
+		(property "Reference" "U5"
 			(at 82.55 24.13 0)
 			(effects
@@
 			(project "BPS-PeripheralSOM"
 				(path "/2365a867-6254-4a7c-9718-f325e0bbac5c/904fa10a-747c-46cf-90d1-33d76069dc5d/429789a2-93db-48e4-a73d-32df605a2afb"
-					(reference "U7")
+					(reference "U5")
 					(unit 1)
 				)
@@
 		(on_board yes)
 		(dnp no)
-		(property "Reference" "#PWR092"
+		(property "Reference" "#PWR042"
 			(at 158.75 49.53 0)
 			(effects
@@
 			(project "PeripheralSOM"
 				(path "/2365a867-6254-4a7c-9718-f325e0bbac5c/904fa10a-747c-46cf-90d1-33d76069dc5d/429789a2-93db-48e4-a73d-32df605a2afb"
-					(reference "#PWR092")
+					(reference "#PWR042")
 					(unit 1)
 				)
@@
 		(dnp no)
 		(fields_autoplaced yes)
-		(property "Reference" "R13"
+		(property "Reference" "R18"
 			(at 24.13 111.7599 0)
 			(effects
@@
 			(project "BPS-PeripheralSOM"
 				(path "/2365a867-6254-4a7c-9718-f325e0bbac5c/904fa10a-747c-46cf-90d1-33d76069dc5d/429789a2-93db-48e4-a73d-32df605a2afb"
-					(reference "R13")
+					(reference "R18")
 					(unit 1)
 				)
@@
 		(on_board yes)
 		(dnp no)
-		(property "Reference" "R12"
+		(property "Reference" "R17"
 			(at 23.368 101.7016 0)
 			(effects
@@
 			(project "BPS-PeripheralSOM"
 				(path "/2365a867-6254-4a7c-9718-f325e0bbac5c/904fa10a-747c-46cf-90d1-33d76069dc5d/429789a2-93db-48e4-a73d-32df605a2afb"
-					(reference "R12")
-					(unit 1)
-				)
+					(reference "R17")
+					(unit 1)
+				)

Commit message: added debug led
Parts:
- renumbered D6 to D13, D7 to D14, R17 to R24, R18 to R25, R19 to R26, R20 to R27, R21 to R28, R22 to R29, R23 to R30, R24 to R31, R25 to R32, U5 to U6
Changed lines of the file:
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@@
 		(dnp no)
 		(fields_autoplaced yes)
-		(property "Reference" "#PWR040"
+		(property "Reference" "#PWR048"
 			(at 146.05 86.36 0)
 			(effects
@@
 			(project "PeripheralSOM"
 				(path "/2365a867-6254-4a7c-9718-f325e0bbac5c/904fa10a-747c-46cf-90d1-33d76069dc5d/429789a2-93db-48e4-a73d-32df605a2afb"
-					(reference "#PWR040")
+					(reference "#PWR048")
 					(unit 1)
 				)
@@
 		(dnp no)
 		(fields_autoplaced yes)
-		(property "Reference" "#PWR038"
+		(property "Reference" "#PWR046"
 			(at 99.06 57.15 0)
 			(effects
@@
 			(project "PeripheralSOM"
 				(path "/2365a867-6254-4a7c-9718-f325e0bbac5c/904fa10a-747c-46cf-90d1-33d76069dc5d/429789a2-93db-48e4-a73d-32df605a2afb"
-					(reference "#PWR038")
+					(reference "#PWR046")
 					(unit 1)
 				)
@@
 		(on_board yes)
 		(dnp yes)
-		(property "Reference" "R24"
+		(property "Reference" "R31"
 			(at 153.67 28.448 90)
 			(effects
@@
 			(project "PeripheralSOM"
 				(path "/2365a867-6254-4a7c-9718-f325e0bbac5c/904fa10a-747c-46cf-90d1-33d76069dc5d/429789a2-93db-48e4-a73d-32df605a2afb"
-					(reference "R24")
+					(reference "R31")
 					(unit 1)
 				)
@@
 		(dnp no)
 		(fields_autoplaced yes)
-		(property "Reference" "D7"
+		(property "Reference" "D14"
 			(at 161.29 35.5599 90)
 			(effects
@@
 			(project ""
 				(path "/2365a867-6254-4a7c-9718-f325e0bbac5c/904fa10a-747c-46cf-90d1-33d76069dc5d/429789a2-93db-48e4-a73d-32df605a2afb"
-					(reference "D7")
+					(reference "D14")
 					(unit 1)
 				)
@@
 		(dnp no)
 		(fields_autoplaced yes)
-		(property "Reference" "#PWR037"
+		(property "Reference" "#PWR045"
 			(at 97.79 30.48 0)
 			(effects
@@
 			(project "BPS-PeripheralSOM"
 				(path "/2365a867-6254-4a7c-9718-f325e0bbac5c/904fa10a-747c-46cf-90d1-33d76069dc5d/429789a2-93db-48e4-a73d-32df605a2afb"
-					(reference "#PWR037")
+					(reference "#PWR045")
 					(unit 1)
 				)
@@
 		(dnp no)
 		(fields_autoplaced yes)
-		(property "Reference" "#PWR039"
+		(property "Reference" "#PWR047"
 			(at 120.65 50.8 0)
 			(effects
@@
 			(project "PeripheralSOM"
 				(path "/2365a867-6254-4a7c-9718-f325e0bbac5c/904fa10a-747c-46cf-90d1-33d76069dc5d/429789a2-93db-48e4-a73d-32df605a2afb"
-					(reference "#PWR039")
+					(reference "#PWR047")
 					(unit 1)
 				)
@@
 		(dnp no)
 		(fields_autoplaced yes)
-		(property "Reference" "#PWR036"
+		(property "Reference" "#PWR044"
 			(at 52.07 49.53 0)
 			(effects
@@
 			(project ""
 				(path "/2365a867-6254-4a7c-9718-f325e0bbac5c/904fa10a-747c-46cf-90d1-33d76069dc5d/429789a2-93db-48e4-a73d-32df605a2afb"
-					(reference "#PWR036")
+					(reference "#PWR044")
 					(unit 1)
 				)
@@
 		(dnp no)
 		(fields_autoplaced yes)
-		(property "Reference" "#PWR041"
+		(property "Reference" "#PWR049"
 			(at 157.48 86.36 0)
 			(effects
@@
 			(project "PeripheralSOM"
 				(path "/2365a867-6254-4a7c-9718-f325e0bbac5c/904fa10a-747c-46cf-90d1-33d76069dc5d/429789a2-93db-48e4-a73d-32df605a2afb"
-					(reference "#PWR041")
+					(reference "#PWR049")
 					(unit 1)
 				)
@@
 		(dnp no)
 		(fields_autoplaced yes)
-		(property "Reference" "R21"
+		(property "Reference" "R28"
 			(at 132.08 91.4399 0)
 			(effects
@@
 			(project "BPS-PeripheralSOM"
 				(path "/2365a867-6254-4a7c-9718-f325e0bbac5c/904fa10a-747c-46cf-90d1-33d76069dc5d/429789a2-93db-48e4-a73d-32df605a2afb"
-					(reference "R21")
+					(reference "R28")
 					(unit 1)
 				)
@@
 		(dnp no)
 		(fields_autoplaced yes)
-		(property "Reference" "R19"
+		(property "Reference" "R26"
 			(at 24.13 121.9199 0)
 			(effects
@@
 			(project "BPS-PeripheralSOM"
 				(path "/2365a867-6254-4a7c-9718-f325e0bbac5c/904fa10a-747c-46cf-90d1-33d76069dc5d/429789a2-93db-48e4-a73d-32df605a2afb"
-					(reference "R19")
+					(reference "R26")
 					(unit 1)
 				)
@@
 		(on_board yes)
 		(dnp no)
-		(property "Reference" "R23"
+		(property "Reference" "R30"
 			(at 147.828 87.7316 0)
 			(effects
@@
 			(project "PeripheralSOM"
 				(path "/2365a867-6254-4a7c-9718-f325e0bbac5c/904fa10a-747c-46cf-90d1-33d76069dc5d/429789a2-93db-48e4-a73d-32df605a2afb"
-					(reference "R23")
+					(reference "R30")
 					(unit 1)
 				)
@@
 		(dnp no)
 		(fields_autoplaced yes)
-		(property "Reference" "R25"
+		(property "Reference" "R32"
 			(at 160.02 88.265 0)
 			(effects
@@
 			(project "PeripheralSOM"
 				(path "/2365a867-6254-4a7c-9718-f325e0bbac5c/904fa10a-747c-46cf-90d1-33d76069dc5d/429789a2-93db-48e4-a73d-32df605a2afb"
-					(reference "R25")
+					(reference "R32")
 					(unit 1)
 				)
@@
 		(dnp no)
 		(fields_autoplaced yes)
-		(property "Reference" "R20"
+		(property "Reference" "R27"
 			(at 39.37 67.945 0)
 			(effects
@@
 			(project "PeripheralSOM"
 				(path "/2365a867-6254-4a7c-9718-f325e0bbac5c/904fa10a-747c-46cf-90d1-33d76069dc5d/429789a2-93db-48e4-a73d-32df605a2afb"
-					(reference "R20")
+					(reference "R27")
 					(unit 1)
 				)
@@
 		(on_board yes)
 		(dnp no)
-		(property "Reference" "D6"
+		(property "Reference" "D13"
 			(at 54.356 36.068 90)
 			(effects
@@
 			(project "BPS-PeripheralSOM"
 				(path "/2365a867-6254-4a7c-9718-f325e0bbac5c/904fa10a-747c-46cf-90d1-33d76069dc5d/429789a2-93db-48e4-a73d-32df605a2afb"
-					(reference "D6")
+					(reference "D13")
 					(unit 1)
 				)
@@
 		(dnp no)
 		(fields_autoplaced yes)
-		(property "Reference" "R22"
+		(property "Reference" "R29"
 			(at 144.78 35.5599 0)
 			(effects
@@
 			(project ""
 				(path "/2365a867-6254-4a7c-9718-f325e0bbac5c/904fa10a-747c-46cf-90d1-33d76069dc5d/429789a2-93db-48e4-a73d-32df605a2afb"
-					(reference "R22")
+					(reference "R29")
 					(unit 1)
 				)
@@
 		(dnp no)
 		(fields_autoplaced yes)
-		(property "Reference" "U5"
+		(property "Reference" "U6"
 			(at 82.55 24.13 0)
 			(effects
@@
 			(project "BPS-PeripheralSOM"
 				(path "/2365a867-6254-4a7c-9718-f325e0bbac5c/904fa10a-747c-46cf-90d1-33d76069dc5d/429789a2-93db-48e4-a73d-32df605a2afb"
-					(reference "U5")
+					(reference "U6")
 					(unit 1)
 				)
@@
 		(on_board yes)
 		(dnp no)
-		(property "Reference" "#PWR042"
+		(property "Reference" "#PWR050"
 			(at 158.75 49.53 0)
 			(effects
@@
 			(project "PeripheralSOM"
 				(path "/2365a867-6254-4a7c-9718-f325e0bbac5c/904fa10a-747c-46cf-90d1-33d76069dc5d/429789a2-93db-48e4-a73d-32df605a2afb"
-					(reference "#PWR042")
+					(reference "#PWR050")
 					(unit 1)
 				)
@@
 		(dnp no)
 		(fields_autoplaced yes)
-		(property "Reference" "R18"
+		(property "Reference" "R25"
 			(at 24.13 111.7599 0)
 			(effects
@@
 			(project "BPS-PeripheralSOM"
 				(path "/2365a867-6254-4a7c-9718-f325e0bbac5c/904fa10a-747c-46cf-90d1-33d76069dc5d/429789a2-93db-48e4-a73d-32df605a2afb"
-					(reference "R18")
+					(reference "R25")
 					(unit 1)
 				)
@@
 		(on_board yes)
 		(dnp no)
-		(property "Reference" "R17"
+		(property "Reference" "R24"
 			(at 23.368 101.7016 0)
 			(effects
@@
 			(project "BPS-PeripheralSOM"
 				(path "/2365a867-6254-4a7c-9718-f325e0bbac5c/904fa10a-747c-46cf-90d1-33d76069dc5d/429789a2-93db-48e4-a73d-32df605a2afb"
-					(reference "R17")
-					(unit 1)
-				)
+					(reference "R24")
+					(unit 1)
+				)

Commit message: addressed 75% of review council 2, cleaned up ERC errors, embedded datasheet and PN
Parts:
- renumbered C34 to C1, C36 to C2, C33 to C20, C37 to C23, C35 to C25, D14 to D10, D13 to D2, R30 to R1, R24 to R12, R25 to R13, R26 to R15, R28 to R20, R32 to R23, R29 to R30, U6 to U7

Commit message: added calcs, cleaned up, addressed comments
Parts:
- removed C20, C23: 10uF, Capacitor_SMD:C_0805_2012Metric_Pad1.18x1.45mm_HandSolder, symbol Device:C
- removed C25: 100nF, Capacitor_SMD:C_0603_1608Metric_Pad1.08x0.95mm_HandSolder, symbol Device:C
- removed D10: TVS, Diode_SMD:D_SOD-123F, symbol Device:D_Zener
- removed D2: TVS, Diode_SMD:D_SOD-323_HandSoldering, symbol Diode:SD12_SOD323
- removed R1, R23, R27: 10k, Resistor_SMD:R_0603_1608Metric_Pad0.98x0.95mm_HandSolder, symbol Device:R
- removed R13: 590, Resistor_SMD:R_0603_1608Metric_Pad0.98x0.95mm_HandSolder, symbol Device:R
- removed R15: 2.1k, Resistor_SMD:R_0603_1608Metric_Pad0.98x0.95mm_HandSolder, symbol Device:R
- removed R20: 402k, Resistor_SMD:R_0603_1608Metric_Pad0.98x0.95mm_HandSolder, symbol Device:R
- removed R30: 24m, Resistor_SMD:R_0603_1608Metric_Pad0.98x0.95mm_HandSolder, symbol Device:R
- removed R31: 100k, Resistor_SMD:R_0603_1608Metric_Pad0.98x0.95mm_HandSolder, symbol Device:R
- removed U7: LM76202QPWPRQ1, LHRS_Power:LM76202QPWPRQ1, symbol lhrs_power:LM76202QPWPRQ1
- added C3: 220n, Capacitor_SMD:C_0603_1608Metric_Pad1.08x0.95mm_HandSolder, symbol Device:C
- added C4: 10n, Capacitor_SMD:C_0603_1608Metric_Pad1.08x0.95mm_HandSolder, symbol ECE319H:C
- added C5: 10u, Capacitor_SMD:C_0805_2012Metric_Pad1.18x1.45mm_HandSolder, symbol Device:C
- added D5: SMBJ30CD, Diode_SMD:D_SMB, symbol Device:D_Zener
- added D6: SMAF4758A, LHRS_Passives:SODFL5026X125N, symbol Device:D_Zener
- added IC1: LM74502DDFR, LHRS_Power:LM74502DDFR, symbol LHRS_ICs:LM74502HDDFR
- added Q1, Q2: PSMN012-100YS, Package_TO_SOT_SMD:LFPAK56, symbol lhrs_power:PSMN012-100YS
- added R10, R11, R7: 10k, Resistor_SMD:R_0603_1608Metric_Pad0.98x0.95mm_HandSolder, symbol Device:R
- added R8: 33, Resistor_SMD:R_0603_1608Metric_Pad0.98x0.95mm_HandSolder, symbol Device:R
- added R9: 221k, Resistor_SMD:R_0603_1608Metric_Pad0.98x0.95mm_HandSolder, symbol Device:R
- C1: value 1uF -> 0.1u; LCSC P/N (none) -> C14663; P/N MLASU168SB5105KTNA01 -> MLASH168SB7104KTNA01
- C2: value 1uF -> 1u; LCSC P/N (none) -> C15849
- R12: value 45.3k -> 137k; LCSC P/N (none) -> C2090646; P/N CRCW060345K3FKEAHP -> CRCW0603137KFKEA
Connections:
- net +24V is gone; now on net GND: C2.1
- net GND: now also C4.2, C5.2, D5.2 (A2), D6.2 (A), IC1.2 (GND), R10.2, R11.2; no longer C2.2
- net 24V_Ext renamed EN/UVLO
- net EN/UVLO: now also IC1.1 (EN/UVLO), R11.1; no longer C1.1
- net UVLO renamed Vin
- net Vin: now also C1.1, D5.1 (A1), Q1.5, R7.2, R9.1
- new net: C2.2, C3.1, D6.1 (K), IC1.5 (VS), R7.1
- new net: C3.2, IC1.4 (VCAP)
- new net: C4.1, R8.1
- new net OV: IC1.7 (OV), R10.1, R9.2
- new net Vout: C5.1, Q2.5
- new net gate: IC1.6 (GATE), Q1.4, Q2.4, R8.2
- new net source: IC1.8 (SRC), Q1.1, Q1.2, Q1.3, Q2.1, Q2.2, Q2.3
- no-connect marks 2 -> 0
Other:
- note added: "1.235 is Enable/UVLO falling threshold on data sheet"
- note added: "4.84ms = 75us + 220nF * 6.5V/300uA 6.5V recommended on datasheet 4.84ms power up delay"
- note added: "Kell Harpole"
- note added: "Overvoltage Protection: 29.03V Vovr = (R2 * Vov)/(R1 + R2) Vov = Vovr * (R1 + R2) / R2 28.875 = 1.25 * (221k + 10k) / 10k"
- note removed: "20.88 ms ramp time"
- note removed: "Current Monitoring"
- note removed: "DNP until validated"
- note removed: "Functional Mode Selection"
- note removed: "ILim(A) = 12/R(k) 1.2A = 12/10kΩ"
- note removed: "OVP set to 27v for buck max voltage of 28v"
- note removed: "Overcurrent Protection"
- note removed: "Pullups"
- note removed: "RTN!=GND Conecting GND to RTN turns off RPP!"
- note removed: "SHDN has weak internal pullup - pulled up to MCU voltage after initial power on"
- note removed: "Set to circuit breaker (latchoff) Use 0 ohm resistor for auto-retry (540ms)"
- note removed: "Typical gain: 78.28 uA/A Vout @ 1.3A = 2.407v R(imon) = 23.7 mΩ"
- note removed: "Under/Overvoltage Protection"

Commit message: fixed ERC, made it look pretty
Parts:
- removed C4: 10n, Capacitor_SMD:C_0603_1608Metric_Pad1.08x0.95mm_HandSolder, symbol ECE319H:C
- removed IC1: LM74502DDFR, LHRS_Power:LM74502DDFR, symbol LHRS_ICs:LM74502HDDFR
- added C4: 10n, Capacitor_SMD:C_0603_1608Metric_Pad1.08x0.95mm_HandSolder, symbol Device:C
- added U1: LM74502DDFR, LHRS_Power:LM74502DDFR, symbol lhrs_power:LM74502DDFR
Connections:
- net EN/UVLO: now also U1.1 (EN/UVLO)
- net GND: now also C4.2, U1.2 (GND)
- net OV: now also U1.7 (OV)
- net gate: now also U1.6 (GATE)
- net source: now also U1.8 (SRC)
- net at C2.2, C3.1, D6.1 (K)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: now also U1.5 (VS)
- net at C3.2: now also U1.4 (VCAP)
- net at R8.1: now also C4.1

Commit message: added outside test points, removed unncessary symbol fields
Parts:
- C3, C4: Mouser Part Number 963-MSASU168SB7224KT -> (none)
- D6: Mouser Part Number 833-SMAF4758A-TP -> (none)
- R7: Mouser Part Number 71-CRCW060310K0FKEI -> (none)
- R8: Mouser Part Number 594-MCT06030C2003FP5 -> (none)
- U1: Manufacturer_Name Texas Instruments -> (none); Manufacturer_Part_Number LM74502DDFR -> (none); Mouser Part Number 595-LM74502DDFR -> (none); Mouser Price/Stock https://www.mouser.co.uk/ProductDetail/Texas-Instruments/LM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 -> (none)

Commit message: updated kicad sharepoint, added pn
Parts:
- C4: P/N MSASU168SB7224KTNB25 -> EMK107SD103KA-T
- R10, R11, R7: P/N CRCW060310K0FKEI -> CRCW060310K0FKEI
Changed lines of the file:
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@@
 			)
 		)
-		(property "P/N" "MSASU168SB7224KTNB25"
+		(property "P/N" "EMK107SD103KA-T"
 			(at 60.96 63.5 0)
 			(hide yes)
@@
 			)
 		)
-		(property "P/N" "CRCW060310K0FKEI"
+		(property "P/N" "CRCW060310K0FKEI "
 			(at 43.18 62.23 0)
 			(hide yes)
@@
 			)
 		)
-		(property "P/N" "CRCW060310K0FKEI"
+		(property "P/N" "CRCW060310K0FKEI "
 			(at 128.27 77.47 0)
 			(hide yes)
@@
 			)
 		)
-		(property "P/N" "CRCW060310K0FKEI"
+		(property "P/N" "CRCW060310K0FKEI "
 			(at 116.84 87.63 0)
 			(hide yes)
