File: hardware/Power.kicad_sch (KiCad schematic)
At the start: 12 parts, among them J8 USB_C_Receptacle_USB2.0_16P

Commit message: updated kicad sharepoint, added pn
Parts:
- C40: renamed from C44; P/N TMK212BBJ106MGHT -> GRM21BR61H106KE43K
- R32: renamed from R34; P/N (none) -> CRCW06035K10FKEC
- R33: renamed from R35; P/N (none) -> CRCW06035K10FKEC
- renumbered TP17 to TP10, TP18 to TP11, TP19 to TP12, TP14 to TP7, TP15 to TP8, TP16 to TP9
Other:
- removed sheet 5VBuck
- added sheet 12VBuck (12VBuck.kicad_sch)
Changed lines of the file:
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@@
 	(wire
 		(pts
-			(xy 184.15 49.53) (xy 193.04 49.53)
+			(xy 176.53 48.26) (xy 185.42 48.26)
 		)
 		(stroke
@@
 	(wire
 		(pts
-			(xy 115.57 48.26) (xy 124.46 48.26)
+			(xy 115.57 48.26) (xy 130.81 48.26)
 		)
 		(stroke
@@
 	(wire
 		(pts
-			(xy 157.48 57.15) (xy 157.48 54.61)
+			(xy 161.29 64.77) (xy 161.29 62.23)
 		)
 		(stroke
@@
 	)
 	(label "Buck_5V"
-		(at 193.04 49.53 180)
+		(at 185.42 48.26 180)
 		(effects
 			(font
@@
 	(hierarchical_label "GND"
 		(shape input)
-		(at 157.48 57.15 270)
+		(at 161.29 64.77 270)
 		(effects
 			(font
@@
 		(in_pos_files yes)
 		(dnp no)
-		(property "Reference" "TP18"
+		(property "Reference" "TP11"
 			(at 92.456 22.098 0)
 			(hide yes)
@@
 			(project "PS-HVCarrier"
 				(path "/2365a867-6254-4a7c-9718-f325e0bbac5c/904fa10a-747c-46cf-90d1-33d76069dc5d"
-					(reference "TP18")
+					(reference "TP11")
 					(unit 1)
 				)
@@
 		(in_pos_files yes)
 		(dnp no)
-		(property "Reference" "TP17"
+		(property "Reference" "TP10"
 			(at 84.836 22.098 0)
 			(hide yes)
@@
 			(project "PS-HVCarrier"
 				(path "/2365a867-6254-4a7c-9718-f325e0bbac5c/904fa10a-747c-46cf-90d1-33d76069dc5d"
-					(reference "TP17")
+					(reference "TP10")
 					(unit 1)
 				)
@@
 		(in_pos_files yes)
 		(dnp no)
-		(property "Reference" "R34"
+		(property "Reference" "R32"
 			(at 78.486 109.22 90)
 			(show_name no)
@@
 		)
 		(property "LCSC P/N" "C23186"
+			(at 82.55 109.22 90)
+			(hide yes)
+			(show_name no)
+			(do_not_autoplace no)
+			(effects
+				(font
+					(size 1.27 1.27)
+				)
+			)
+		)
+		(property "P/N" "CRCW06035K10FKEC "
 			(at 82.55 109.22 90)
 			(hide yes)
@@
 			(project "PS-HVCarrier"
 				(path "/2365a867-6254-4a7c-9718-f325e0bbac5c/904fa10a-747c-46cf-90d1-33d76069dc5d"
-					(reference "R34")
+					(reference "R32")
 					(unit 1)
 				)
@@
 		(in_pos_files yes)
 		(dnp no)
-		(property "Reference" "R35"
+		(property "Reference" "R33"
 			(at 86.106 109.22 90)
 			(show_name no)
@@
 		)
 		(property "LCSC P/N" "C23186"
+			(at 90.17 109.22 90)
+			(hide yes)
+			(show_name no)
+			(do_not_autoplace no)
+			(effects
+				(font
+					(size 1.27 1.27)
+				)
+			)
+		)
+		(property "P/N" "CRCW06035K10FKEC "
 			(at 90.17 109.22 90)
 			(hide yes)
@@
 			(project "PS-HVCarrier"
 				(path "/2365a867-6254-4a7c-9718-f325e0bbac5c/904fa10a-747c-46cf-90d1-33d76069dc5d"
-					(reference "R35")
+					(reference "R33")
 					(unit 1)
 				)
@@
 		(in_pos_files yes)
 		(dnp no)
-		(property "Reference" "TP15"
+		(property "Reference" "TP8"
 			(at 70.358 21.844 0)
 			(hide yes)
@@
 			(project "PS-HVCarrier"
 				(path "/2365a867-6254-4a7c-9718-f325e0bbac5c/904fa10a-747c-46cf-90d1-33d76069dc5d"
-					(reference "TP15")
+					(reference "TP8")
 					(unit 1)
 				)
@@
 		(in_pos_files yes)
 		(dnp no)
-		(property "Reference" "TP19"
+		(property "Reference" "TP12"
 			(at 120.65 123.6979 0)
 			(hide yes)
@@
 			(project "PS-HVCarrier"
 				(path "/2365a867-6254-4a7c-9718-f325e0bbac5c/904fa10a-747c-46cf-90d1-33d76069dc5d"
-					(reference "TP19")
+					(reference "TP12")
 					(unit 1)
 				)
@@
 		(in_pos_files yes)
 		(dnp no)
-		(property "Reference" "TP14"
+		(property "Reference" "TP7"
 			(at 73.1521 86.36 0)
 			(hide yes)
@@
 			(project "PS-HVCarrier"
 				(path "/2365a867-6254-4a7c-9718-f325e0bbac5c/904fa10a-747c-46cf-90d1-33d76069dc5d"
-					(reference "TP14")
+					(reference "TP7")
 					(unit 1)
 				)
@@
 		(in_pos_files yes)
 		(dnp no)
-		(property "Reference" "TP16"
+		(property "Reference" "TP9"
 			(at 77.216 22.098 0)
 			(hide yes)
@@
 			(project "PS-HVCarrier"
 				(path "/2365a867-6254-4a7c-9718-f325e0bbac5c/904fa10a-747c-46cf-90d1-33d76069dc5d"
-					(reference "TP16")
+					(reference "TP9")
 					(unit 1)
 				)
@@
 		(dnp no)
 		(fields_autoplaced yes)
-		(property "Reference" "#FLG04"
+		(property "Reference" "#FLG02"
 			(at 71.755 91.44 0)
 			(hide yes)
@@
 			(project "PS-HVCarrier"
 				(path "/2365a867-6254-4a7c-9718-f325e0bbac5c/904fa10a-747c-46cf-90d1-33d76069dc5d"
-					(reference "#FLG04")
+					(reference "#FLG02")
 					(unit 1)
 				)
@@
 		(in_pos_files yes)
 		(dnp no)
-		(property "Reference" "C44"
+		(property "Reference" "C40"
 			(at 64.3128 98.9584 0)
 			(show_name no)
@@
 			)
 		)
-		(property "P/N" "TMK212BBJ106MGHT"
+		(property "P/N" "GRM21BR61H106KE43K"
 			(at 67.31 97.79 0)
 			(hide yes)
@@
 			(project "PS-HVCarrier"
 				(path "/2365a867-6254-4a7c-9718-f325e0bbac5c/904fa10a-747c-46cf-90d1-33d76069dc5d"
-					(reference "C44")
+					(reference "C40")
 					(unit 1)
 				)
@@
 	)
 	(sheet
+		(at 130.81 36.83)
+		(size 45.72 25.4)
+		(exclude_from_sim no)
+		(in_bom yes)
+		(on_board yes)
+		(dnp no)
+		(fields_autoplaced yes)
+		(stroke
+			(width 0.1524)
+			(type solid)
+		)
+		(fill
+			(color 0 0 0 0)
+		)
+		(property "Sheetname" "12VBuck"
+			(at 130.81 36.1184 0)
+			(show_name no)
+			(do_not_autoplace no)
+			(effects
+				(font
+					(size 1.27 1.27)
+				)
+				(justify left bottom)
+			)
+		)
+		(property "Sheetfile" "12VBuck.kicad_sch"
+			(at 130.81 62.3066 0)
+			(show_name no)
+			(do_not_autoplace no)
+			(effects
+				(font
+					(size 1.27 1.27)
+				)
+				(justify left top)
+			)
+		)
+		(pin "GND" bidirectional
+			(at 161.29 62.23 270)
+			(effects
+				(font
+					(size 1.27 1.27)
+				)
+				(justify left)
+			)
+		)
+		(pin "V_in_12V" input
+			(at 130.81 48.26 180)
+			(effects
+				(font
+					(size 1.27 1.27)
+				)
+				(justify left)
+			)
+		)
+		(pin "V_out_5V" output
+			(at 176.53 48.26 0)
+			(effects
+				(font
+					(size 1.27 1.27)
+				)
+				(justify right)
+			)
+		)
+		(instances
+			(project "PS-HVCarrier"
+				(path "/2365a867-6254-4a7c-9718-f325e0bbac5c/904fa10a-747c-46cf-90d1-33d76069dc5d"
+					(page "18")
+				)
+			)
+		)
+	)
+	(sheet
 		(at 36.83 33.02)
 		(size 72.39 30.48)
@@
 				)
 			)
-		)
-	)
-	(sheet
-		(at 124.46 31.75)
-		(size 59.69 22.86)
-		(exclude_from_sim no)
-		(in_bom yes)
-		(on_board yes)
-		(dnp no)
-		(fields_autoplaced yes)
-		(stroke
-			(width 0.1524)
-			(type solid)
-		)
-		(fill
-			(color 0 0 0 0)
-		)
-		(property "Sheetname" "5VBuck"
-			(at 124.46 31.0384 0)
-			(show_name no)
-			(do_not_autoplace no)
-			(effects
-				(font
-					(size 1.27 1.27)
-				)
-				(justify left bottom)
-			)
-		)
-		(property "Sheetfile" "5VBuck.kicad_sch"
-			(at 124.46 54.5596 0)
-			(show_name no)
-			(do_not_autoplace no)
-			(effects
-				(font
-					(size 1.27 1.27)
-				)
-				(justify left top)
-			)
-		)
-		(pin "GND" input
-			(at 157.48 54.61 270)
-			(effects
-				(font
-					(size 1.27 1.27)
-				)
-				(justify left)
-			)
-		)
-		(pin "V_in_24V" input
-			(at 124.46 48.26 180)
-			(effects
-				(font
-					(size 1.27 1.27)
-				)
-				(justify left)
-			)
-		)
-		(pin "V_out_5V" output
-			(at 184.15 49.53 0)
-			(effects
-				(font
-					(size 1.27 1.27)
-				)
-				(justify right)
-			)
-		)
-		(instances
-			(project "PS-HVCarrier"
-				(path "/2365a867-6254-4a7c-9718-f325e0bbac5c/904fa10a-747c-46cf-90d1-33d76069dc5d"
-					(page "7")
-				)
-			)

Commit message: updated PN
Changed lines of the file:
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@@
 		)
 	)
-	(hierarchical_label "+24V_Ext"
+	(hierarchical_label "+12V_Ext"
 		(shape input)
 		(at 31.75 48.26 180)
@@
 		)
 	)
-	(hierarchical_label "+24V"
+	(hierarchical_label "+12V"
 		(shape output)
 		(at 115.57 44.45 90)
