File: hardware/HV_Carrier/KiCAD-Sharepoint/LHRS_Design_Blocks.kicad_blocks/PowerProtection.kicad_block/PowerProtection.kicad_sch (KiCad schematic)
At the start: 16 parts, among them IC1 LM74502DDFR, Q1 PSMN012-100YS, Q2 PSMN012-100YS

Commit message: updatred PP
Parts:
- removed D1: SMAF4758A, LHRS_Passives:SODFL5026X125N, symbol Device:D_Zener
- removed D2: SMBJ30CD, Diode_SMD:D_SMB, symbol Device:D_Zener
- removed R6: 137k, Resistor_SMD:R_0603_1608Metric_Pad0.98x0.95mm_HandSolder, symbol Device:R
- removed R7: 10k, Resistor_SMD:R_0603_1608Metric_Pad0.98x0.95mm_HandSolder, symbol Device:R
- added C6, C7: 0.1u, Capacitor_SMD:C_0603_1608Metric_Pad1.08x0.95mm_HandSolder, symbol Device:C
- added D1: SMAF4758A, LHRS_Passives:SODFL5026X125N, symbol lhrs_power:SMAF4758A
- added D2: SMBJ15CA, Diode_SMD:D_SMB, symbol lhrs_power:SMBJ15CA
- added R6: 15.8k, Resistor_SMD:R_0603_1608Metric_Pad0.98x0.95mm_HandSolder, symbol Device:R_US
- added R7: 100k, Resistor_SMD:R_0603_1608Metric_Pad0.98x0.95mm_HandSolder, symbol Device:R_US
- IC1: symbol LHRS_ICs:LM74502HDDFR -> lhrs_power:LM74502HDDFR
- R1, R3: symbol Device:R -> Device:R_US
- R4: value 221k -> 100k; symbol Device:R -> Device:R_US
- R5: value 10k -> 7.32k; symbol Device:R -> Device:R_US
Connections:
- net EN/UVLO: now also C6.2, R6.2, R7.2
- net GND: now also C6.1, C7.1, D1.2 (A), D2.1 (A1), R6.1
- net OV: now also C7.2
- net Vin: now also D2.2 (A2), R7.1
- net at C2.2, C3.1, IC1.5 (VS)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: now also D1.1 (K)
Other:
- note added: "Output of Python Calulations for Resistor Values"
- note removed: "1.235 is Enable/UVLO falling threshold on data sheet"
- note removed: "Overvoltage Protection: 29.03V Vovr = (R2 * Vov)/(R1 + R2) Vov = Vovr * (R1 + R2) / R2 28.875 = 1.25 * (221k + 10k) / 10k"
- moved on the sheet: C2, Q2
