File: hardware/HV_Carrier/48PinMCU.kicad_sch (KiCad schematic)
At the start: 34 parts, among them J6 SWD_Header, J7 SWD, SW1 Reset, SW2 SW_SPDT, U6 STM32G473CETx, Y1 Crystal

Commit message: update dPN for a bunch of stuff
Parts:
- C30: renamed from C27; value 10uF -> 10u; footprint Capacitor_SMD:C_0805_2012Metric -> Capacitor_SMD:C_0805_2012Metric_Pad1.18x1.45mm_HandSolder
- C42: renamed from C39; P/N MAJCH168BB7104KTEA01 -> MLASH168SB7104KTNA01
- R27: renamed from R25; P/N CRCW060310K0FKEI -> CRCW060310K0FKEI
- R32: renamed from R30; P/N CRCW060310K0FKEI -> CRCW060310K0FKEI
- renumbered C25 to C28, C26 to C29, C28 to C31, C29 to C32, C30 to C33, C31 to C34, C32 to C35, C33 to C36, C34 to C37, C35 to C38, C36 to C39, C37 to C40, C38 to C41, D8 to D10, D9 to D11, D10 to D12, J6 to J7, J7 to J8, R24 to R26, R26 to R28, R27 to R29, R28 to R30, R29 to R31, R31 to R33, U6 to U5
