File: hardware/HV_Carrier/CAN_Transceiver.kicad_sch (KiCad schematic)
At the start: 9 parts, among them IC1 TCAN3413DR, U3 CDSOT23-T24CAN

Commit message: update dPN for a bunch of stuff
Parts:
- renumbered C8 to C10, C9 to C11, C10 to C12, C11 to C13, IC1 to IC2, U3 to U2
Changed lines of the file:
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@@
 		(dnp no)
 		(fields_autoplaced yes)
-		(property "Reference" "C11"
+		(property "Reference" "C13"
 			(at 193.04 87.6299 0)
 			(show_name no)
@@
 			(project "PS-HVCarrier"
 				(path "/2365a867-6254-4a7c-9718-f325e0bbac5c/891507c0-eb7b-4bd7-b7e8-bba1d4bfa654"
-					(reference "C11")
+					(reference "C13")
 					(unit 1)
 				)
 				(path "/2365a867-6254-4a7c-9718-f325e0bbac5c/8e4b18be-f701-4f79-b148-bbeadfa1a129"
-					(reference "C15")
+					(reference "C17")
 					(unit 1)
 				)
@@
 		(in_pos_files yes)
 		(dnp no)
-		(property "Reference" "C9"
+		(property "Reference" "C11"
 			(at 76.2 73.66 0)
 			(show_name no)
@@
 			(project "PS-HVCarrier"
 				(path "/2365a867-6254-4a7c-9718-f325e0bbac5c/891507c0-eb7b-4bd7-b7e8-bba1d4bfa654"
-					(reference "C9")
+					(reference "C11")
 					(unit 1)
 				)
 				(path "/2365a867-6254-4a7c-9718-f325e0bbac5c/8e4b18be-f701-4f79-b148-bbeadfa1a129"
-					(reference "C13")
+					(reference "C15")
 					(unit 1)
 				)
@@
 		(in_pos_files yes)
 		(dnp no)
-		(property "Reference" "C10"
+		(property "Reference" "C12"
 			(at 88.138 73.66 0)
 			(show_name no)
@@
 			(project "PS-HVCarrier"
 				(path "/2365a867-6254-4a7c-9718-f325e0bbac5c/891507c0-eb7b-4bd7-b7e8-bba1d4bfa654"
-					(reference "C10")
+					(reference "C12")
 					(unit 1)
 				)
 				(path "/2365a867-6254-4a7c-9718-f325e0bbac5c/8e4b18be-f701-4f79-b148-bbeadfa1a129"
-					(reference "C14")
+					(reference "C16")
 					(unit 1)
 				)
@@
 		(in_pos_files yes)
 		(dnp no)
-		(property "Reference" "C8"
+		(property "Reference" "C10"
 			(at 65.278 73.66 0)
 			(show_name no)
@@
 			(project "PS-HVCarrier"
 				(path "/2365a867-6254-4a7c-9718-f325e0bbac5c/891507c0-eb7b-4bd7-b7e8-bba1d4bfa654"
-					(reference "C8")
+					(reference "C10")
 					(unit 1)
 				)
 				(path "/2365a867-6254-4a7c-9718-f325e0bbac5c/8e4b18be-f701-4f79-b148-bbeadfa1a129"
-					(reference "C12")
+					(reference "C14")
 					(unit 1)
 				)
@@
 		(dnp no)
 		(fields_autoplaced yes)
-		(property "Reference" "IC1"
+		(property "Reference" "IC2"
 			(at 128.27 63.5 0)
 			(show_name no)
@@
 			(project "PS-HVCarrier"
 				(path "/2365a867-6254-4a7c-9718-f325e0bbac5c/891507c0-eb7b-4bd7-b7e8-bba1d4bfa654"
-					(reference "IC1")
+					(reference "IC2")
 					(unit 1)
 				)
 				(path "/2365a867-6254-4a7c-9718-f325e0bbac5c/8e4b18be-f701-4f79-b148-bbeadfa1a129"
-					(reference "IC2")
+					(reference "IC3")
 					(unit 1)
 				)
@@
 		(dnp no)
 		(fields_autoplaced yes)
-		(property "Reference" "U3"
+		(property "Reference" "U2"
 			(at 194.31 48.26 0)
 			(show_name no)
@@
 			(project "PS-HVCarrier"
 				(path "/2365a867-6254-4a7c-9718-f325e0bbac5c/891507c0-eb7b-4bd7-b7e8-bba1d4bfa654"
+					(reference "U2")
+					(unit 1)
+				)
+				(path "/2365a867-6254-4a7c-9718-f325e0bbac5c/8e4b18be-f701-4f79-b148-bbeadfa1a129"
 					(reference "U3")
 					(unit 1)
 				)
-				(path "/2365a867-6254-4a7c-9718-f325e0bbac5c/8e4b18be-f701-4f79-b148-bbeadfa1a129"
-					(reference "U4")
-					(unit 1)
-				)
