File: hardware/HV_Carrier/LDO.kicad_sch (KiCad schematic)
At the start: 5 parts, among them U2 MCP1826S

Commit message: update dPN for a bunch of stuff
Parts:
- renumbered C6 to C8, C7 to C9, U2 to U1
Changed lines of the file:
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@@
 		(dnp no)
 		(fields_autoplaced yes)
-		(property "Reference" "C7"
+		(property "Reference" "C9"
 			(at 168.275 68.5735 0)
 			(show_name no)
@@
 			(project "PS-HVCarrier"
 				(path "/2365a867-6254-4a7c-9718-f325e0bbac5c/904fa10a-747c-46cf-90d1-33d76069dc5d/d9c02800-502d-4b66-a933-6a0fcb4cc3ad"
-					(reference "C7")
+					(reference "C9")
 					(unit 1)
 				)
@@
 		(dnp no)
 		(fields_autoplaced yes)
-		(property "Reference" "U2"
+		(property "Reference" "U1"
 			(at 152.4 56.515 0)
 			(show_name no)
@@
 			(project "PS-HVCarrier"
 				(path "/2365a867-6254-4a7c-9718-f325e0bbac5c/904fa10a-747c-46cf-90d1-33d76069dc5d/d9c02800-502d-4b66-a933-6a0fcb4cc3ad"
-					(reference "U2")
+					(reference "U1")
 					(unit 1)
 				)
@@
 		(dnp no)
 		(fields_autoplaced yes)
-		(property "Reference" "C6"
+		(property "Reference" "C8"
 			(at 142.875 68.5735 0)
 			(show_name no)
@@
 			(project "PS-HVCarrier"
 				(path "/2365a867-6254-4a7c-9718-f325e0bbac5c/904fa10a-747c-46cf-90d1-33d76069dc5d/d9c02800-502d-4b66-a933-6a0fcb4cc3ad"
-					(reference "C6")
-					(unit 1)
-				)
+					(reference "C8")
+					(unit 1)
+				)
