File: hardware/HV_Carrier/PowerProtection.kicad_sch (KiCad schematic)
At the start: 16 parts, among them Q1 PSMN012-100YS, Q2 PSMN012-100YS, U1 LM74502DDFR

Commit message: updatred PP
Parts:
- removed C4: 10n, Capacitor_SMD:C_0603_1608Metric_Pad1.08x0.95mm_HandSolder, symbol Device:C
- removed D5: SMBJ30CD, Diode_SMD:D_SMB, symbol Device:D_Zener
- removed D6: SMAF4758A, LHRS_Passives:SODFL5026X125N, symbol Device:D_Zener
- removed R11: 10k, Resistor_SMD:R_0603_1608Metric_Pad0.98x0.95mm_HandSolder, symbol Device:R
- removed R12: 137k, Resistor_SMD:R_0603_1608Metric_Pad0.98x0.95mm_HandSolder, symbol Device:R
- removed U1: LM74502DDFR, LHRS_Power:LM74502DDFR, symbol lhrs_power:LM74502DDFR
- added C4: 10n, Capacitor_SMD:C_0603_1608Metric_Pad1.08x0.95mm_HandSolder, symbol ECE319H:C
- added C6, C7: 0.1u, Capacitor_SMD:C_0603_1608Metric_Pad1.08x0.95mm_HandSolder, symbol Device:C
- added D1: SMAF4758A, LHRS_Passives:SODFL5026X125N, symbol lhrs_power:SMAF4758A
- added D2: SMBJ15CA, Diode_SMD:D_SMB, symbol lhrs_power:SMBJ15CA
- added IC1: LM74502DDFR, LHRS_Power:LM74502DDFR, symbol lhrs_power:LM74502HDDFR
- added R6: 15.8k, Resistor_SMD:R_0603_1608Metric_Pad0.98x0.95mm_HandSolder, symbol Device:R_US
- added R7: 100k, Resistor_SMD:R_0603_1608Metric_Pad0.98x0.95mm_HandSolder, symbol Device:R_US
- C3: Mouser Part Number (none) -> 963-MSASU168SB7224KT
- R1: renamed from R7; symbol Device:R -> Device:R_US; Mouser Part Number (none) -> 71-CRCW060310K0FKEI; P/N CRCW060310K0FKEI -> CRCW060310K0FKEI
- R3: renamed from R8; symbol Device:R -> Device:R_US; Mouser Part Number (none) -> 594-MCT06030C2003FP5
- R4: renamed from R9; value 221k -> 100k; symbol Device:R -> Device:R_US
- R5: renamed from R10; value 10k -> 7.32k; symbol Device:R -> Device:R_US; P/N CRCW060310K0FKEI -> CRCW060310K0FKEI
Connections:
- net EN/UVLO: now also C6.2, IC1.1 (EN/UVLO), R6.2, R7.2
- net GND: now also C4.2, C6.1, C7.1, D1.2 (A), D2.1 (A1), IC1.2 (GND), R6.1
- net OV: now also C7.2, IC1.7 (OV)
- net Vin: now also D2.2 (A2), R7.1
- net gate: now also IC1.6 (GATE)
- net source: now also IC1.8 (SRC)
- net at C2.2, C3.1, R1.1: now also D1.1 (K), IC1.5 (VS)
- net at C3.2: now also IC1.4 (VCAP)
- net at R3.1: now also C4.1
Other:
- note added: "Output of Python Calulations for Resistor Values"
- note removed: "1.235 is Enable/UVLO falling threshold on data sheet"
- note removed: "Overvoltage Protection: 29.03V Vovr = (R2 * Vov)/(R1 + R2) Vov = Vovr * (R1 + R2) / R2 28.875 = 1.25 * (221k + 10k) / 10k"
- moved on the sheet: C2, Q2

Commit message: update dPN for a bunch of stuff
Parts:
- removed C4: 10n, Capacitor_SMD:C_0603_1608Metric_Pad1.08x0.95mm_HandSolder, symbol ECE319H:C
- added C4: 10n, Capacitor_SMD:C_0603_1608Metric_Pad1.08x0.95mm_HandSolder, symbol Device:C
- C3: Mouser Part Number 963-MSASU168SB7224KT -> (none)
- C6: renamed from C7; P/N (none) -> MLASH168SB7104KTNA01
- C7: renamed from C6; P/N (none) -> MLASH168SB7104KTNA01
- IC1: Height 1.1 -> (none); Manufacturer_Name Texas Instruments -> (none); Manufacturer_Part_Number LM74502DDFR -> (none); Mouser Part Number 595-LM74502DDFR -> (none); Mouser Price/Stock https://www.mouser.co.uk/ProductDetail/Texas-Instruments/LM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 -> (none)
- R10: renamed from R5; LCSC P/N C25804 -> C843967; P/N CRCW060310K0FKEI -> CRCW06037K32FKEA
- R11: renamed from R7; LCSC P/N C25804 -> C844916; P/N CRCW060310K0FKEI -> CRCW0603100KFKED
- R7: renamed from R1; Mouser Part Number 71-CRCW060310K0FKEI -> (none)
- R8: renamed from R3; Mouser Part Number 594-MCT06030C2003FP5 -> (none)
- R9: renamed from R4; LCSC P/N C2090661 -> C844916; P/N CRCW0603221KFKEA -> CRCW0603100KFKED
- renumbered D2 to D5, D1 to D6, R6 to R12
Connections:
- net GND: now also C4.2
- net at R8.1: now also C4.1
