File: hardware/HV_Carrier/12VBuck.kicad_sch (KiCad schematic)
At the start: 12 parts, among them U14 LMR51635XDDCR

Commit message: update dPN for a bunch of stuff
Parts:
- C88: renamed from C86; P/N MSASL168SB5475KTNA01 -> 08055D475KAT4A
- C89: renamed from C87; P/N MAJCH168BB7104KTEA01 -> MLASH168SB7104KTNA01
- C90: renamed from C88; P/N MAJCH168BB7104KTEA01 -> MLASH168SB7104KTNA01
- C91: renamed from C89; P/N ZRB18AC80E476ME01L -> C1210C476M9RAC
- renumbered TP38 to TP35, TP39 to TP36, TP40 to TP37, TP41 to TP38, U14 to U13
Changed lines of the file:
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@@
 		(dnp no)
 		(fields_autoplaced yes)
-		(property "Reference" "C86"
+		(property "Reference" "C88"
 			(at 96.52 85.0962 0)
 			(show_name no)
@@
 			)
 		)
-		(property "P/N" "MSASL168SB5475KTNA01"
+		(property "P/N" "08055D475KAT4A"
 			(at 93.98 86.36 0)
 			(hide yes)
@@
 			(project "PS-HVCarrier"
 				(path "/2365a867-6254-4a7c-9718-f325e0bbac5c/904fa10a-747c-46cf-90d1-33d76069dc5d/3d5e6349-9b57-4f3d-adb1-46bcc69fbb65"
-					(reference "C86")
+					(reference "C88")
 					(unit 1)
 				)
@@
 		(in_pos_files yes)
 		(dnp no)
-		(property "Reference" "TP38"
+		(property "Reference" "TP35"
 			(at 229.87 123.6979 0)
 			(hide yes)
@@
 			(project "PS-HVCarrier"
 				(path "/2365a867-6254-4a7c-9718-f325e0bbac5c/904fa10a-747c-46cf-90d1-33d76069dc5d/3d5e6349-9b57-4f3d-adb1-46bcc69fbb65"
-					(reference "TP38")
+					(reference "TP35")
 					(unit 1)
 				)
@@
 		(dnp no)
 		(fields_autoplaced yes)
-		(property "Reference" "U14"
+		(property "Reference" "U13"
 			(at 129.54 71.12 0)
 			(show_name no)
@@
 			(project "PS-HVCarrier"
 				(path "/2365a867-6254-4a7c-9718-f325e0bbac5c/904fa10a-747c-46cf-90d1-33d76069dc5d/3d5e6349-9b57-4f3d-adb1-46bcc69fbb65"
-					(reference "U14")
+					(reference "U13")
 					(unit 1)
 				)
@@
 		(in_pos_files yes)
 		(dnp no)
-		(property "Reference" "TP40"
+		(property "Reference" "TP37"
 			(at 242.57 123.6979 0)
 			(hide yes)
@@
 			(project "PS-HVCarrier"
 				(path "/2365a867-6254-4a7c-9718-f325e0bbac5c/904fa10a-747c-46cf-90d1-33d76069dc5d/3d5e6349-9b57-4f3d-adb1-46bcc69fbb65"
-					(reference "TP40")
+					(reference "TP37")
 					(unit 1)
 				)
@@
 		(in_pos_files yes)
 		(dnp no)
-		(property "Reference" "TP39"
+		(property "Reference" "TP36"
 			(at 229.87 136.3979 0)
 			(hide yes)
@@
 			(project "PS-HVCarrier"
 				(path "/2365a867-6254-4a7c-9718-f325e0bbac5c/904fa10a-747c-46cf-90d1-33d76069dc5d/3d5e6349-9b57-4f3d-adb1-46bcc69fbb65"
-					(reference "TP39")
+					(reference "TP36")
 					(unit 1)
 				)
@@
 		(in_pos_files yes)
 		(dnp no)
-		(property "Reference" "TP41"
+		(property "Reference" "TP38"
 			(at 242.57 136.3979 0)
 			(hide yes)
@@
 			(project "PS-HVCarrier"
 				(path "/2365a867-6254-4a7c-9718-f325e0bbac5c/904fa10a-747c-46cf-90d1-33d76069dc5d/3d5e6349-9b57-4f3d-adb1-46bcc69fbb65"
-					(reference "TP41")
+					(reference "TP38")
 					(unit 1)
 				)
@@
 		(dnp no)
 		(fields_autoplaced yes)
-		(property "Reference" "C89"
+		(property "Reference" "C91"
 			(at 184.15 88.9062 0)
 			(show_name no)
@@
 			)
 		)
-		(property "P/N" "ZRB18AC80E476ME01L"
+		(property "P/N" "C1210C476M9RAC"
 			(at 181.61 90.17 0)
 			(hide yes)
@@
 			(project "PS-HVCarrier"
 				(path "/2365a867-6254-4a7c-9718-f325e0bbac5c/904fa10a-747c-46cf-90d1-33d76069dc5d/3d5e6349-9b57-4f3d-adb1-46bcc69fbb65"
-					(reference "C89")
+					(reference "C91")
 					(unit 1)
 				)
@@
 		(in_pos_files yes)
 		(dnp no)
-		(property "Reference" "C88"
+		(property "Reference" "C90"
 			(at 156.718 80.01 0)
 			(show_name no)
@@
 			)
 		)
-		(property "P/N" "MAJCH168BB7104KTEA01"
+		(property "P/N" "MLASH168SB7104KTNA01"
 			(at 153.67 83.82 0)
 			(hide yes)
@@
 			(project "PS-HVCarrier"
 				(path "/2365a867-6254-4a7c-9718-f325e0bbac5c/904fa10a-747c-46cf-90d1-33d76069dc5d/3d5e6349-9b57-4f3d-adb1-46bcc69fbb65"
-					(reference "C88")
+					(reference "C90")
 					(unit 1)
 				)
@@
 		(dnp no)
 		(fields_autoplaced yes)
-		(property "Reference" "C87"
+		(property "Reference" "C89"
 			(at 105.41 87.6362 0)
 			(show_name no)
@@
 			)
 		)
-		(property "P/N" "MAJCH168BB7104KTEA01"
+		(property "P/N" "MLASH168SB7104KTNA01"
 			(at 102.87 88.9 0)
 			(hide yes)
@@
 			(project "PS-HVCarrier"
 				(path "/2365a867-6254-4a7c-9718-f325e0bbac5c/904fa10a-747c-46cf-90d1-33d76069dc5d/3d5e6349-9b57-4f3d-adb1-46bcc69fbb65"
-					(reference "C87")
-					(unit 1)
-				)
+					(reference "C89")
+					(unit 1)
+				)

Commit message: added scrut breakout conn
Parts:
- renumbered R83 to R85, R84 to R86, TP35 to TP38, TP36 to TP39, TP37 to TP40, TP38 to TP41
Changed lines of the file:
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@@
 		(in_pos_files yes)
 		(dnp no)
-		(property "Reference" "TP35"
+		(property "Reference" "TP38"
 			(at 229.87 123.6979 0)
 			(hide yes)
@@
 			(project "PS-HVCarrier"
 				(path "/2365a867-6254-4a7c-9718-f325e0bbac5c/904fa10a-747c-46cf-90d1-33d76069dc5d/3d5e6349-9b57-4f3d-adb1-46bcc69fbb65"
-					(reference "TP35")
+					(reference "TP38")
 					(unit 1)
 				)
@@
 		(in_pos_files yes)
 		(dnp no)
-		(property "Reference" "TP37"
+		(property "Reference" "TP40"
 			(at 242.57 123.6979 0)
 			(hide yes)
@@
 			(project "PS-HVCarrier"
 				(path "/2365a867-6254-4a7c-9718-f325e0bbac5c/904fa10a-747c-46cf-90d1-33d76069dc5d/3d5e6349-9b57-4f3d-adb1-46bcc69fbb65"
-					(reference "TP37")
+					(reference "TP40")
 					(unit 1)
 				)
@@
 		(in_pos_files yes)
 		(dnp no)
-		(property "Reference" "TP36"
+		(property "Reference" "TP39"
 			(at 229.87 136.3979 0)
 			(hide yes)
@@
 			(project "PS-HVCarrier"
 				(path "/2365a867-6254-4a7c-9718-f325e0bbac5c/904fa10a-747c-46cf-90d1-33d76069dc5d/3d5e6349-9b57-4f3d-adb1-46bcc69fbb65"
-					(reference "TP36")
+					(reference "TP39")
 					(unit 1)
 				)
@@
 		(in_pos_files yes)
 		(dnp no)
-		(property "Reference" "TP38"
+		(property "Reference" "TP41"
 			(at 242.57 136.3979 0)
 			(hide yes)
@@
 			(project "PS-HVCarrier"
 				(path "/2365a867-6254-4a7c-9718-f325e0bbac5c/904fa10a-747c-46cf-90d1-33d76069dc5d/3d5e6349-9b57-4f3d-adb1-46bcc69fbb65"
-					(reference "TP38")
+					(reference "TP41")
 					(unit 1)
 				)
@@
 		(dnp no)
 		(fields_autoplaced yes)
-		(property "Reference" "R83"
+		(property "Reference" "R85"
 			(at 227.33 85.0899 0)
 			(show_name no)
@@
 			(project "PS-HVCarrier"
 				(path "/2365a867-6254-4a7c-9718-f325e0bbac5c/904fa10a-747c-46cf-90d1-33d76069dc5d/3d5e6349-9b57-4f3d-adb1-46bcc69fbb65"
-					(reference "R83")
+					(reference "R85")
 					(unit 1)
 				)
@@
 		(dnp no)
 		(fields_autoplaced yes)
-		(property "Reference" "R84"
+		(property "Reference" "R86"
 			(at 227.33 92.7099 0)
 			(show_name no)
@@
 			(project "PS-HVCarrier"
 				(path "/2365a867-6254-4a7c-9718-f325e0bbac5c/904fa10a-747c-46cf-90d1-33d76069dc5d/3d5e6349-9b57-4f3d-adb1-46bcc69fbb65"
-					(reference "R84")
-					(unit 1)
-				)
+					(reference "R86")
+					(unit 1)
+				)
