File: hardware/HV_Carrier/AMC3311_OpAmp.kicad_sch (KiCad schematic)
At the start: 16 parts, among them U12 TLV9002QDRQ1

Commit message: update dPN for a bunch of stuff
Parts:
- C82: renamed from C80; P/N UMK107B7102MAHT -> MLASU063SB7102KFNA01
- C83: renamed from C81; P/N UMK107B7102MAHT -> MLASU063SB7102KFNA01
- R71, R72, R73, R74, R75, R76: P/N CRCW060310K0FKEI -> CRCW060310K0FKEI
- renumbered C82 to C84, TP34 to TP31, TP35 to TP32, U12 to U11
Changed lines of the file:
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@@
 		(in_pos_files yes)
 		(dnp no)
-		(property "Reference" "TP35"
+		(property "Reference" "TP32"
 			(at 121.92 61.4679 0)
 			(hide yes)
@@
 			(project "PS-HVCarrier"
 				(path "/2365a867-6254-4a7c-9718-f325e0bbac5c/83ab5b0b-4732-42c0-82fe-e74f4113c82a/9068f688-485f-416c-9cd2-e445ef73f243"
-					(reference "TP35")
-					(unit 1)
-				)
-				(path "/2365a867-6254-4a7c-9718-f325e0bbac5c/83ab5b0b-4732-42c0-82fe-e74f4113c82a/a79c140a-76cc-4bbb-b1f3-7013b136bd70"
-					(reference "TP37")
+					(reference "TP32")
+					(unit 1)
+				)
+				(path "/2365a867-6254-4a7c-9718-f325e0bbac5c/83ab5b0b-4732-42c0-82fe-e74f4113c82a/a79c140a-76cc-4bbb-b1f3-7013b136bd70"
+					(reference "TP34")
 					(unit 1)
 				)
@@
 			)
 		)
-		(property "P/N" "CRCW060310K0FKEI "
+		(property "P/N" "CRCW060310K0FKEI"
 			(at 86.36 113.03 90)
 			(hide yes)
@@
 			)
 		)
-		(property "P/N" "CRCW060310K0FKEI "
+		(property "P/N" "CRCW060310K0FKEI"
 			(at 67.31 105.41 90)
 			(hide yes)
@@
 		(in_pos_files yes)
 		(dnp no)
-		(property "Reference" "C82"
+		(property "Reference" "C84"
 			(at 165.354 85.09 0)
 			(show_name no)
@@
 			(project "PS-HVCarrier"
 				(path "/2365a867-6254-4a7c-9718-f325e0bbac5c/83ab5b0b-4732-42c0-82fe-e74f4113c82a/9068f688-485f-416c-9cd2-e445ef73f243"
-					(reference "C82")
-					(unit 1)
-				)
-				(path "/2365a867-6254-4a7c-9718-f325e0bbac5c/83ab5b0b-4732-42c0-82fe-e74f4113c82a/a79c140a-76cc-4bbb-b1f3-7013b136bd70"
-					(reference "C85")
+					(reference "C84")
+					(unit 1)
+				)
+				(path "/2365a867-6254-4a7c-9718-f325e0bbac5c/83ab5b0b-4732-42c0-82fe-e74f4113c82a/a79c140a-76cc-4bbb-b1f3-7013b136bd70"
+					(reference "C87")
 					(unit 1)
 				)
@@
 		(in_pos_files yes)
 		(dnp no)
-		(property "Reference" "C80"
+		(property "Reference" "C82"
 			(at 85.09 87.122 90)
 			(show_name no)
@@
 			)
 		)
-		(property "P/N" "UMK107B7102MAHT"
+		(property "P/N" "MLASU063SB7102KFNA01"
 			(at 85.09 81.28 90)
 			(hide yes)
@@
 			(project "PS-HVCarrier"
 				(path "/2365a867-6254-4a7c-9718-f325e0bbac5c/83ab5b0b-4732-42c0-82fe-e74f4113c82a/9068f688-485f-416c-9cd2-e445ef73f243"
-					(reference "C80")
-					(unit 1)
-				)
-				(path "/2365a867-6254-4a7c-9718-f325e0bbac5c/83ab5b0b-4732-42c0-82fe-e74f4113c82a/a79c140a-76cc-4bbb-b1f3-7013b136bd70"
-					(reference "C83")
+					(reference "C82")
+					(unit 1)
+				)
+				(path "/2365a867-6254-4a7c-9718-f325e0bbac5c/83ab5b0b-4732-42c0-82fe-e74f4113c82a/a79c140a-76cc-4bbb-b1f3-7013b136bd70"
+					(reference "C85")
 					(unit 1)
 				)
@@
 		(dnp no)
 		(fields_autoplaced yes)
-		(property "Reference" "U12"
+		(property "Reference" "U11"
 			(at 181.61 86.3599 0)
 			(show_name no)
@@
 			(project "PS-HVCarrier"
 				(path "/2365a867-6254-4a7c-9718-f325e0bbac5c/83ab5b0b-4732-42c0-82fe-e74f4113c82a/9068f688-485f-416c-9cd2-e445ef73f243"
+					(reference "U11")
+					(unit 3)
+				)
+				(path "/2365a867-6254-4a7c-9718-f325e0bbac5c/83ab5b0b-4732-42c0-82fe-e74f4113c82a/a79c140a-76cc-4bbb-b1f3-7013b136bd70"
 					(reference "U12")
-					(unit 3)
-				)
-				(path "/2365a867-6254-4a7c-9718-f325e0bbac5c/83ab5b0b-4732-42c0-82fe-e74f4113c82a/a79c140a-76cc-4bbb-b1f3-7013b136bd70"
-					(reference "U13")
 					(unit 3)
 				)
@@
 			)
 		)
-		(property "P/N" "CRCW060310K0FKEI "
+		(property "P/N" "CRCW060310K0FKEI"
 			(at 67.31 100.33 90)
 			(hide yes)
@@
 		(dnp no)
 		(fields_autoplaced yes)
-		(property "Reference" "U12"
+		(property "Reference" "U11"
 			(at 83.82 55.88 0)
 			(show_name no)
@@
 			(project "PS-HVCarrier"
 				(path "/2365a867-6254-4a7c-9718-f325e0bbac5c/83ab5b0b-4732-42c0-82fe-e74f4113c82a/9068f688-485f-416c-9cd2-e445ef73f243"
+					(reference "U11")
+					(unit 1)
+				)
+				(path "/2365a867-6254-4a7c-9718-f325e0bbac5c/83ab5b0b-4732-42c0-82fe-e74f4113c82a/a79c140a-76cc-4bbb-b1f3-7013b136bd70"
 					(reference "U12")
-					(unit 1)
-				)
-				(path "/2365a867-6254-4a7c-9718-f325e0bbac5c/83ab5b0b-4732-42c0-82fe-e74f4113c82a/a79c140a-76cc-4bbb-b1f3-7013b136bd70"
-					(reference "U13")
 					(unit 1)
 				)
@@
 		(in_pos_files yes)
 		(dnp no)
-		(property "Reference" "C81"
+		(property "Reference" "C83"
 			(at 86.36 126.492 90)
 			(show_name no)
@@
 			)
 		)
-		(property "P/N" "UMK107B7102MAHT"
+		(property "P/N" "MLASU063SB7102KFNA01"
 			(at 86.36 120.65 90)
 			(hide yes)
@@
 			(project "PS-HVCarrier"
 				(path "/2365a867-6254-4a7c-9718-f325e0bbac5c/83ab5b0b-4732-42c0-82fe-e74f4113c82a/9068f688-485f-416c-9cd2-e445ef73f243"
-					(reference "C81")
-					(unit 1)
-				)
-				(path "/2365a867-6254-4a7c-9718-f325e0bbac5c/83ab5b0b-4732-42c0-82fe-e74f4113c82a/a79c140a-76cc-4bbb-b1f3-7013b136bd70"
-					(reference "C84")
+					(reference "C83")
+					(unit 1)
+				)
+				(path "/2365a867-6254-4a7c-9718-f325e0bbac5c/83ab5b0b-4732-42c0-82fe-e74f4113c82a/a79c140a-76cc-4bbb-b1f3-7013b136bd70"
+					(reference "C86")
 					(unit 1)
 				)
@@
 			)
 		)
-		(property "P/N" "CRCW060310K0FKEI "
+		(property "P/N" "CRCW060310K0FKEI"
 			(at 66.04 63.5 90)
 			(hide yes)
@@
 			)
 		)
-		(property "P/N" "CRCW060310K0FKEI "
+		(property "P/N" "CRCW060310K0FKEI"
 			(at 85.09 73.66 90)
 			(hide yes)
@@
 			)
 		)
-		(property "P/N" "CRCW060310K0FKEI "
+		(property "P/N" "CRCW060310K0FKEI"
 			(at 66.04 68.58 90)
 			(hide yes)
@@
 		(in_pos_files yes)
 		(dnp no)
-		(property "Reference" "TP34"
+		(property "Reference" "TP31"
 			(at 116.84 98.2979 0)
 			(hide yes)
@@
 			(project "PS-HVCarrier"
 				(path "/2365a867-6254-4a7c-9718-f325e0bbac5c/83ab5b0b-4732-42c0-82fe-e74f4113c82a/9068f688-485f-416c-9cd2-e445ef73f243"
-					(reference "TP34")
-					(unit 1)
-				)
-				(path "/2365a867-6254-4a7c-9718-f325e0bbac5c/83ab5b0b-4732-42c0-82fe-e74f4113c82a/a79c140a-76cc-4bbb-b1f3-7013b136bd70"
-					(reference "TP36")
+					(reference "TP31")
+					(unit 1)
+				)
+				(path "/2365a867-6254-4a7c-9718-f325e0bbac5c/83ab5b0b-4732-42c0-82fe-e74f4113c82a/a79c140a-76cc-4bbb-b1f3-7013b136bd70"
+					(reference "TP33")
 					(unit 1)
 				)
@@
 		(dnp no)
 		(fields_autoplaced yes)
-		(property "Reference" "U12"
+		(property "Reference" "U11"
 			(at 85.09 92.71 0)
 			(show_name no)
@@
 			(project "PS-HVCarrier"
 				(path "/2365a867-6254-4a7c-9718-f325e0bbac5c/83ab5b0b-4732-42c0-82fe-e74f4113c82a/9068f688-485f-416c-9cd2-e445ef73f243"
+					(reference "U11")
+					(unit 2)
+				)
+				(path "/2365a867-6254-4a7c-9718-f325e0bbac5c/83ab5b0b-4732-42c0-82fe-e74f4113c82a/a79c140a-76cc-4bbb-b1f3-7013b136bd70"
 					(reference "U12")
 					(unit 2)
 				)
-				(path "/2365a867-6254-4a7c-9718-f325e0bbac5c/83ab5b0b-4732-42c0-82fe-e74f4113c82a/a79c140a-76cc-4bbb-b1f3-7013b136bd70"
-					(reference "U13")
-					(unit 2)
-				)

Commit message: added scrut breakout conn
Parts:
- renumbered R71 to R73, R72 to R74, R73 to R75, R74 to R76, R75 to R77, R76 to R78, TP31 to TP34, TP32 to TP35
Changed lines of the file:
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@@
 		(in_pos_files yes)
 		(dnp no)
-		(property "Reference" "TP32"
+		(property "Reference" "TP35"
 			(at 121.92 61.4679 0)
 			(hide yes)
@@
 			(project "PS-HVCarrier"
 				(path "/2365a867-6254-4a7c-9718-f325e0bbac5c/83ab5b0b-4732-42c0-82fe-e74f4113c82a/9068f688-485f-416c-9cd2-e445ef73f243"
-					(reference "TP32")
-					(unit 1)
-				)
-				(path "/2365a867-6254-4a7c-9718-f325e0bbac5c/83ab5b0b-4732-42c0-82fe-e74f4113c82a/a79c140a-76cc-4bbb-b1f3-7013b136bd70"
-					(reference "TP34")
+					(reference "TP35")
+					(unit 1)
+				)
+				(path "/2365a867-6254-4a7c-9718-f325e0bbac5c/83ab5b0b-4732-42c0-82fe-e74f4113c82a/a79c140a-76cc-4bbb-b1f3-7013b136bd70"
+					(reference "TP37")
 					(unit 1)
 				)
@@
 		(in_pos_files yes)
 		(dnp no)
-		(property "Reference" "R76"
+		(property "Reference" "R78"
 			(at 86.36 113.03 90)
 			(show_name no)
@@
 			(project "PS-HVCarrier"
 				(path "/2365a867-6254-4a7c-9718-f325e0bbac5c/83ab5b0b-4732-42c0-82fe-e74f4113c82a/9068f688-485f-416c-9cd2-e445ef73f243"
-					(reference "R76")
-					(unit 1)
-				)
-				(path "/2365a867-6254-4a7c-9718-f325e0bbac5c/83ab5b0b-4732-42c0-82fe-e74f4113c82a/a79c140a-76cc-4bbb-b1f3-7013b136bd70"
-					(reference "R82")
+					(reference "R78")
+					(unit 1)
+				)
+				(path "/2365a867-6254-4a7c-9718-f325e0bbac5c/83ab5b0b-4732-42c0-82fe-e74f4113c82a/a79c140a-76cc-4bbb-b1f3-7013b136bd70"
+					(reference "R84")
 					(unit 1)
 				)
@@
 		(in_pos_files yes)
 		(dnp no)
-		(property "Reference" "R74"
+		(property "Reference" "R76"
 			(at 67.31 105.41 90)
 			(show_name no)
@@
 			(project "PS-HVCarrier"
 				(path "/2365a867-6254-4a7c-9718-f325e0bbac5c/83ab5b0b-4732-42c0-82fe-e74f4113c82a/9068f688-485f-416c-9cd2-e445ef73f243"
-					(reference "R74")
-					(unit 1)
-				)
-				(path "/2365a867-6254-4a7c-9718-f325e0bbac5c/83ab5b0b-4732-42c0-82fe-e74f4113c82a/a79c140a-76cc-4bbb-b1f3-7013b136bd70"
-					(reference "R80")
+					(reference "R76")
+					(unit 1)
+				)
+				(path "/2365a867-6254-4a7c-9718-f325e0bbac5c/83ab5b0b-4732-42c0-82fe-e74f4113c82a/a79c140a-76cc-4bbb-b1f3-7013b136bd70"
+					(reference "R82")
 					(unit 1)
 				)
@@
 		(in_pos_files yes)
 		(dnp no)
-		(property "Reference" "R73"
+		(property "Reference" "R75"
 			(at 67.31 100.33 90)
 			(show_name no)
@@
 			(project "PS-HVCarrier"
 				(path "/2365a867-6254-4a7c-9718-f325e0bbac5c/83ab5b0b-4732-42c0-82fe-e74f4113c82a/9068f688-485f-416c-9cd2-e445ef73f243"
-					(reference "R73")
-					(unit 1)
-				)
-				(path "/2365a867-6254-4a7c-9718-f325e0bbac5c/83ab5b0b-4732-42c0-82fe-e74f4113c82a/a79c140a-76cc-4bbb-b1f3-7013b136bd70"
-					(reference "R79")
+					(reference "R75")
+					(unit 1)
+				)
+				(path "/2365a867-6254-4a7c-9718-f325e0bbac5c/83ab5b0b-4732-42c0-82fe-e74f4113c82a/a79c140a-76cc-4bbb-b1f3-7013b136bd70"
+					(reference "R81")
 					(unit 1)
 				)
@@
 		(in_pos_files yes)
 		(dnp no)
-		(property "Reference" "R71"
+		(property "Reference" "R73"
 			(at 66.04 63.5 90)
 			(show_name no)
@@
 			(project "PS-HVCarrier"
 				(path "/2365a867-6254-4a7c-9718-f325e0bbac5c/83ab5b0b-4732-42c0-82fe-e74f4113c82a/9068f688-485f-416c-9cd2-e445ef73f243"
-					(reference "R71")
-					(unit 1)
-				)
-				(path "/2365a867-6254-4a7c-9718-f325e0bbac5c/83ab5b0b-4732-42c0-82fe-e74f4113c82a/a79c140a-76cc-4bbb-b1f3-7013b136bd70"
-					(reference "R77")
+					(reference "R73")
+					(unit 1)
+				)
+				(path "/2365a867-6254-4a7c-9718-f325e0bbac5c/83ab5b0b-4732-42c0-82fe-e74f4113c82a/a79c140a-76cc-4bbb-b1f3-7013b136bd70"
+					(reference "R79")
 					(unit 1)
 				)
@@
 		(in_pos_files yes)
 		(dnp no)
-		(property "Reference" "R75"
+		(property "Reference" "R77"
 			(at 85.09 73.66 90)
 			(show_name no)
@@
 			(project "PS-HVCarrier"
 				(path "/2365a867-6254-4a7c-9718-f325e0bbac5c/83ab5b0b-4732-42c0-82fe-e74f4113c82a/9068f688-485f-416c-9cd2-e445ef73f243"
-					(reference "R75")
-					(unit 1)
-				)
-				(path "/2365a867-6254-4a7c-9718-f325e0bbac5c/83ab5b0b-4732-42c0-82fe-e74f4113c82a/a79c140a-76cc-4bbb-b1f3-7013b136bd70"
-					(reference "R81")
+					(reference "R77")
+					(unit 1)
+				)
+				(path "/2365a867-6254-4a7c-9718-f325e0bbac5c/83ab5b0b-4732-42c0-82fe-e74f4113c82a/a79c140a-76cc-4bbb-b1f3-7013b136bd70"
+					(reference "R83")
 					(unit 1)
 				)
@@
 		(in_pos_files yes)
 		(dnp no)
-		(property "Reference" "R72"
+		(property "Reference" "R74"
 			(at 66.04 68.58 90)
 			(show_name no)
@@
 			(project "PS-HVCarrier"
 				(path "/2365a867-6254-4a7c-9718-f325e0bbac5c/83ab5b0b-4732-42c0-82fe-e74f4113c82a/9068f688-485f-416c-9cd2-e445ef73f243"
-					(reference "R72")
-					(unit 1)
-				)
-				(path "/2365a867-6254-4a7c-9718-f325e0bbac5c/83ab5b0b-4732-42c0-82fe-e74f4113c82a/a79c140a-76cc-4bbb-b1f3-7013b136bd70"
-					(reference "R78")
+					(reference "R74")
+					(unit 1)
+				)
+				(path "/2365a867-6254-4a7c-9718-f325e0bbac5c/83ab5b0b-4732-42c0-82fe-e74f4113c82a/a79c140a-76cc-4bbb-b1f3-7013b136bd70"
+					(reference "R80")
 					(unit 1)
 				)
@@
 		(in_pos_files yes)
 		(dnp no)
-		(property "Reference" "TP31"
+		(property "Reference" "TP34"
 			(at 116.84 98.2979 0)
 			(hide yes)
@@
 			(project "PS-HVCarrier"
 				(path "/2365a867-6254-4a7c-9718-f325e0bbac5c/83ab5b0b-4732-42c0-82fe-e74f4113c82a/9068f688-485f-416c-9cd2-e445ef73f243"
-					(reference "TP31")
-					(unit 1)
-				)
-				(path "/2365a867-6254-4a7c-9718-f325e0bbac5c/83ab5b0b-4732-42c0-82fe-e74f4113c82a/a79c140a-76cc-4bbb-b1f3-7013b136bd70"
-					(reference "TP33")
-					(unit 1)
-				)
+					(reference "TP34")
+					(unit 1)
+				)
+				(path "/2365a867-6254-4a7c-9718-f325e0bbac5c/83ab5b0b-4732-42c0-82fe-e74f4113c82a/a79c140a-76cc-4bbb-b1f3-7013b136bd70"
+					(reference "TP36")
+					(unit 1)
+				)
