File: hardware/HV_Carrier/AMC3311_Sense.kicad_sch (KiCad schematic)
At the start: 17 parts, among them U5 AMC3311QDWERQ1

Commit message: update dPN for a bunch of stuff
Parts:
- C19: renamed from C17; P/N UMK107B7102MAHT -> MLASU063SB7102KFNA01
- C20: renamed from C18; P/N MAJCH168BB7104KTEA01 -> MLASH168SB7104KTNA01
- C21: renamed from C19; P/N MAJCH168BB7104KTEA01 -> MLASH168SB7104KTNA01
- C22: renamed from C20; P/N UMK107B7102MAHT -> MLASU063SB7102KFNA01
- C23: renamed from C21; P/N MAJCH168BB7104KTEA01 -> MLASH168SB7104KTNA01
- C24: renamed from C22; P/N UMK107B7102MAHT -> MLASU063SB7102KFNA01
- C26: renamed from C24; P/N EMK107SD103KA-T -> MSASH168SB5103KTNA01
- renumbered C16 to C18, C23 to C25, U5 to U4
