File: hardware/HV_Carrier/Current_Sense.kicad_sch (KiCad schematic)
At the start: 38 parts, among them J10 SSA-2-100A, J11 SSA-2-100A, J9 LZSR 80-P, U7 TLV9002QDRQ1

Commit message: update dPN for a bunch of stuff
Parts:
- C43: renamed from C41; P/N MAJCH168BB7104KTEA01 -> MLASH168SB7104KTNA01
- C45: renamed from C43; P/N EMK107SD103KA-T -> MSASH168SB5103KTNA01
- C46: renamed from C44; P/N EMK107SD103KA-T -> MSASH168SB5103KTNA01
- C47: renamed from C45; P/N MAJCH168BB7104KTEA01 -> MLASH168SB7104KTNA01
- C48: renamed from C46; P/N MAJCH168BB7104KTEA01 -> MLASH168SB7104KTNA01
- C49: renamed from C47; P/N UMK107B7102MAHT -> MLASU063SB7102KFNA01
- R34, R35, R36, R42, R43, R46: P/N CRCW060310K0FKEI -> CRCW060310K0FKEI
- renumbered C42 to C44, C48 to C50, TP13 to TP10, TP14 to TP11, TP15 to TP12, TP16 to TP13, TP17 to TP14, TP18 to TP15, U7 to U6
Changed lines of the file:
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@@
 			)
 		)
-		(property "P/N" "CRCW060310K0FKEI "
+		(property "P/N" "CRCW060310K0FKEI"
 			(at 77.47 60.96 90)
 			(hide yes)
@@
 			)
 		)
-		(property "P/N" "CRCW060310K0FKEI "
+		(property "P/N" "CRCW060310K0FKEI"
 			(at 171.45 46.99 90)
 			(hide yes)
@@
 		(in_pos_files yes)
 		(dnp no)
-		(property "Reference" "C48"
+		(property "Reference" "C50"
 			(at 233.934 78.74 0)
 			(show_name no)
@@
 			(project "PS-HVCarrier"
 				(path "/2365a867-6254-4a7c-9718-f325e0bbac5c/c64f1e33-0c51-411c-bbbf-0af7b620c655"
-					(reference "C48")
+					(reference "C50")
 					(unit 1)
 				)
@@
 		(in_pos_files yes)
 		(dnp no)
-		(property "Reference" "C42"
+		(property "Reference" "C44"
 			(at 53.848 35.052 90)
 			(show_name no)
@@
 			(project "PS-HVCarrier"
 				(path "/2365a867-6254-4a7c-9718-f325e0bbac5c/c64f1e33-0c51-411c-bbbf-0af7b620c655"
-					(reference "C42")
+					(reference "C44")
 					(unit 1)
 				)
@@
 		(in_pos_files yes)
 		(dnp no)
-		(property "Reference" "C41"
+		(property "Reference" "C43"
 			(at 54.356 24.384 90)
 			(show_name no)
@@
 			)
 		)
-		(property "P/N" "MAJCH168BB7104KTEA01"
+		(property "P/N" "MLASH168SB7104KTNA01"
 			(at 52.07 30.48 90)
 			(hide yes)
@@
 			(project "PS-HVCarrier"
 				(path "/2365a867-6254-4a7c-9718-f325e0bbac5c/c64f1e33-0c51-411c-bbbf-0af7b620c655"
-					(reference "C41")
+					(reference "C43")
 					(unit 1)
 				)
@@
 		(in_pos_files yes)
 		(dnp no)
-		(property "Reference" "TP15"
+		(property "Reference" "TP12"
 			(at 59.69 80.5179 0)
 			(hide yes)
@@
 			(project "PS-HVCarrier"
 				(path "/2365a867-6254-4a7c-9718-f325e0bbac5c/c64f1e33-0c51-411c-bbbf-0af7b620c655"
-					(reference "TP15")
+					(reference "TP12")
 					(unit 1)
 				)
@@
 		(in_pos_files yes)
 		(dnp no)
-		(property "Reference" "U7"
+		(property "Reference" "U6"
 			(at 193.802 44.196 0)
 			(show_name no)
@@
 			(project "PS-HVCarrier"
 				(path "/2365a867-6254-4a7c-9718-f325e0bbac5c/c64f1e33-0c51-411c-bbbf-0af7b620c655"
-					(reference "U7")
+					(reference "U6")
 					(unit 1)
 				)
@@
 		(in_pos_files yes)
 		(dnp no)
-		(property "Reference" "C43"
+		(property "Reference" "C45"
 			(at 101.854 35.306 0)
 			(show_name no)
@@
 			)
 		)
-		(property "P/N" "EMK107SD103KA-T"
+		(property "P/N" "MSASH168SB5103KTNA01"
 			(at 104.14 36.83 0)
 			(hide yes)
@@
 			(project "PS-HVCarrier"
 				(path "/2365a867-6254-4a7c-9718-f325e0bbac5c/c64f1e33-0c51-411c-bbbf-0af7b620c655"
-					(reference "C43")
+					(reference "C45")
 					(unit 1)
 				)
@@
 		(in_pos_files yes)
 		(dnp no)
-		(property "Reference" "TP14"
+		(property "Reference" "TP11"
 			(at 59.69 56.3879 0)
 			(hide yes)
@@
 			(project "PS-HVCarrier"
 				(path "/2365a867-6254-4a7c-9718-f325e0bbac5c/c64f1e33-0c51-411c-bbbf-0af7b620c655"
-					(reference "TP14")
+					(reference "TP11")
 					(unit 1)
 				)
@@
 		(in_pos_files yes)
 		(dnp no)
-		(property "Reference" "C47"
+		(property "Reference" "C49"
 			(at 189.23 28.956 90)
 			(show_name no)
@@
 			)
 		)
-		(property "P/N" "UMK107B7102MAHT"
+		(property "P/N" "MLASU063SB7102KFNA01"
 			(at 189.23 34.29 90)
 			(hide yes)
@@
 			(project "PS-HVCarrier"
 				(path "/2365a867-6254-4a7c-9718-f325e0bbac5c/c64f1e33-0c51-411c-bbbf-0af7b620c655"
-					(reference "C47")
+					(reference "C49")
 					(unit 1)
 				)
@@
 			)
 		)
-		(property "P/N" "CRCW060310K0FKEI "
+		(property "P/N" "CRCW060310K0FKEI"
 			(at 171.45 54.61 90)
 			(hide yes)
@@
 		(in_pos_files yes)
 		(dnp no)
-		(property "Reference" "C46"
+		(property "Reference" "C48"
 			(at 180.34 60.198 0)
 			(show_name no)
@@
 			)
 		)
-		(property "P/N" "MAJCH168BB7104KTEA01"
+		(property "P/N" "MLASH168SB7104KTNA01"
 			(at 176.53 62.23 0)
 			(hide yes)
@@
 			(project "PS-HVCarrier"
 				(path "/2365a867-6254-4a7c-9718-f325e0bbac5c/c64f1e33-0c51-411c-bbbf-0af7b620c655"
-					(reference "C46")
+					(reference "C48")
 					(unit 1)
 				)
@@
 		(dnp no)
 		(fields_autoplaced yes)
-		(property "Reference" "U7"
+		(property "Reference" "U6"
 			(at 214.63 43.18 0)
 			(show_name no)
@@
 			(project "PS-HVCarrier"
 				(path "/2365a867-6254-4a7c-9718-f325e0bbac5c/c64f1e33-0c51-411c-bbbf-0af7b620c655"
-					(reference "U7")
+					(reference "U6")
 					(unit 2)
 				)
@@
 		(in_pos_files yes)
 		(dnp no)
-		(property "Reference" "TP13"
+		(property "Reference" "TP10"
 			(at 59.69 28.4479 0)
 			(hide yes)
@@
 			(project "PS-HVCarrier"
 				(path "/2365a867-6254-4a7c-9718-f325e0bbac5c/c64f1e33-0c51-411c-bbbf-0af7b620c655"
-					(reference "TP13")
+					(reference "TP10")
 					(unit 1)
 				)
@@
 		(in_pos_files yes)
 		(dnp no)
-		(property "Reference" "TP16"
+		(property "Reference" "TP13"
 			(at 179.07 29.7179 0)
 			(hide yes)
@@
 			(project "PS-HVCarrier"
 				(path "/2365a867-6254-4a7c-9718-f325e0bbac5c/c64f1e33-0c51-411c-bbbf-0af7b620c655"
-					(reference "TP16")
+					(reference "TP13")
 					(unit 1)
 				)
@@
 		(in_pos_files yes)
 		(dnp no)
-		(property "Reference" "TP17"
+		(property "Reference" "TP14"
 			(at 179.07 50.0379 0)
 			(hide yes)
@@
 			(project "PS-HVCarrier"
 				(path "/2365a867-6254-4a7c-9718-f325e0bbac5c/c64f1e33-0c51-411c-bbbf-0af7b620c655"
-					(reference "TP17")
+					(reference "TP14")
 					(unit 1)
 				)
@@
 			)
 		)
-		(property "P/N" "CRCW060310K0FKEI "
+		(property "P/N" "CRCW060310K0FKEI"
 			(at 189.23 40.64 90)
 			(hide yes)
@@
 		(in_pos_files yes)
 		(dnp no)
-		(property "Reference" "C45"
+		(property "Reference" "C47"
 			(at 162.052 49.53 0)
 			(show_name no)
@@
 			)
 		)
-		(property "P/N" "MAJCH168BB7104KTEA01"
+		(property "P/N" "MLASH168SB7104KTNA01"
 			(at 165.1 50.8 0)
 			(hide yes)
@@
 			(project "PS-HVCarrier"
 				(path "/2365a867-6254-4a7c-9718-f325e0bbac5c/c64f1e33-0c51-411c-bbbf-0af7b620c655"
-					(reference "C45")
+					(reference "C47")
 					(unit 1)
 				)
@@
 		(in_pos_files yes)
 		(dnp no)
-		(property "Reference" "C44"
+		(property "Reference" "C46"
 			(at 101.854 63.246 0)
 			(show_name no)
@@
 			)
 		)
-		(property "P/N" "EMK107SD103KA-T"
+		(property "P/N" "MSASH168SB5103KTNA01"
 			(at 104.14 64.77 0)
 			(hide yes)
@@
 			(project "PS-HVCarrier"
 				(path "/2365a867-6254-4a7c-9718-f325e0bbac5c/c64f1e33-0c51-411c-bbbf-0af7b620c655"
-					(reference "C44")
+					(reference "C46")
 					(unit 1)
 				)
@@
 		(in_pos_files yes)
 		(dnp no)
-		(property "Reference" "U7"
+		(property "Reference" "U6"
 			(at 247.65 79.248 0)
 			(show_name no)
@@
 			(project "PS-HVCarrier"
 				(path "/2365a867-6254-4a7c-9718-f325e0bbac5c/c64f1e33-0c51-411c-bbbf-0af7b620c655"
-					(reference "U7")
+					(reference "U6")
 					(unit 3)
 				)
@@
 			)
 		)
-		(property "P/N" "CRCW060310K0FKEI "
+		(property "P/N" "CRCW060310K0FKEI"
 			(at 77.47 85.09 90)
 			(hide yes)
@@
 		(in_pos_files yes)
 		(dnp no)
-		(property "Reference" "TP18"
+		(property "Reference" "TP15"
 			(at 247.65 48.7679 0)
 			(hide yes)
@@
 			(project "PS-HVCarrier"
 				(path "/2365a867-6254-4a7c-9718-f325e0bbac5c/c64f1e33-0c51-411c-bbbf-0af7b620c655"
-					(reference "TP18")
+					(reference "TP15")
 					(unit 1)
 				)
@@
 			)
 		)
-		(property "P/N" "CRCW060310K0FKEI "
+		(property "P/N" "CRCW060310K0FKEI"
 			(at 77.47 33.02 90)
 			(hide yes)

Commit message: added scrut breakout conn
Parts:
- added J12: Discharge Vin, symbol Connector_Generic:Conn_01x02
- added J13: Charge Vin, symbol Connector_Generic:Conn_01x02
- added R47: 90k, symbol Device:R
- added R48: 10k, symbol Device:R
- added S1: OS102011MS2QN1, OS102011MS2QN1:OS102011MA1QN1, symbol OS102011MS2QN1:OS102011MS2QN1
- added TP15: Scurt Vin+, TestPoint:TestPoint_THTPad_D3.0mm_Drill1.5mm, symbol Connector:TestPoint
- added TP16: Scurt Vout, TestPoint:TestPoint_THTPad_D3.0mm_Drill1.5mm, symbol Connector:TestPoint
- added TP17: Scurt Vin-, TestPoint:TestPoint_THTPad_D3.0mm_Drill1.5mm, symbol Connector:TestPoint
- TP18: renamed from TP15; value SHUNT_ADC -> SHUNT_Vout
Connections:
- net SHUNT ADC: now also S1.2; no longer D17.2 (A), D18.1 (K), TP18.1, U6.5 (+), U6.7
- net SHUNT ADC UREF: now also U6.5 (+)
- net SHUNT Vout: now reaches C49.1, R46.1, U6.1
- net SHUNT Vout: now also D17.2 (A), D18.1 (K), TP18.1, S1.3; no longer U6.6 (-)
- new net Scrut Vout: R47.2, R48.1, S1.1, TP16.1
- new net Vin+: J12.1 (Pin_1), J13.2 (Pin_2), R47.1, TP15.1
- new net Vin-: J12.2 (Pin_2), J13.1 (Pin_1), R48.2, TP17.1, U6.6 (-), U6.7
Other:
- note added: "Charge: Vin+ = Vin- − V_bench = 1.65V − V_bench Scurt_Vout = 1.65V − 0.1 × V_bench For -40A: 0.1 × V_bench = 0.5V V_bench = 5V"
- note added: "Current Scrut"
- note added: "Discharge: Vin+ = Vin- + V_bench = 1.65V + V_bench Scurt_Vout = Vin- + (Vin+ − Vin-) × R2/(R1+R2) = 1.65V + V_bench × (1k/10k) = 1.65V + 0.1 × V_bench For 70A: 0.1 × V_bench = 0.875V V_bench = 8.75V"
- note added: "Leave Default at POS.2 to short 2 and 3 POS 2. to read Shunt Vout POS 1. to read Scrut Vout"
- note added: "Unity Gain to Prevent Vin- Tapping into a live node"
- note removed: "Unity Gain Amp"
- moved on the sheet: C50, D17, D18, U6B, U6C
