File: hardware/HV_Carrier/Current_Sense.kicad_sch (KiCad schematic)
At the start: 46 parts, among them J10 SSA-2-100A, J11 SSA-2-100A, J12 Discharge Vin, J13 Charge Vin, J9 LZSR 80-P, U6 TLV9002QDRQ1

Commit message: reduced random fields
Parts:
- J12, J13: footprint (none) -> LHRS_Connectors:Molex_Nano-Fit_105309-xx02_1x02_P2.50mm_Vertical
- R47, R48: footprint (none) -> Resistor_SMD:R_0603_1608Metric_Pad0.98x0.95mm_HandSolder
Changed lines of the file:
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@@
 			)
 		)
-		(property "Footprint" ""
+		(property "Footprint" "LHRS_Connectors:Molex_Nano-Fit_105309-xx02_1x02_P2.50mm_Vertical"
 			(at 186.69 116.84 0)
 			(hide yes)
@@
 			)
 		)
-		(property "Footprint" ""
+		(property "Footprint" "Resistor_SMD:R_0603_1608Metric_Pad0.98x0.95mm_HandSolder"
 			(at 221.742 128.27 90)
 			(hide yes)
@@
 			)
 		)
-		(property "Footprint" ""
+		(property "Footprint" "LHRS_Connectors:Molex_Nano-Fit_105309-xx02_1x02_P2.50mm_Vertical"
 			(at 186.69 130.81 0)
 			(hide yes)
@@
 			)
 		)
-		(property "Footprint" ""
+		(property "Footprint" "Resistor_SMD:R_0603_1608Metric_Pad0.98x0.95mm_HandSolder"
 			(at 221.742 114.3 90)
 			(hide yes)
