File: hardware/HV_Carrier/Power_Mux.kicad_sch (KiCad schematic)
At the start: 8 parts, among them U11 TPS2117DRLR

Commit message: update dPN for a bunch of stuff
Parts:
- R70: P/N CRCW060310K0FKEI -> CRCW060310K0FKEI
- U10: renamed from U11; MANUFACTURER Texas Instruments -> (none); MAXIMUM_PACKAGE_HEIGHT 0.6mm -> (none); PARTREV A -> (none); STANDARD IPC-7351B -> (none)
- renumbered C76 to C78, C77 to C79, C78 to C80, C79 to C81
Changed lines of the file:
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@@
 		(in_pos_files yes)
 		(dnp no)
-		(property "Reference" "C79"
+		(property "Reference" "C81"
 			(at 91.8972 57.2516 0)
 			(show_name no)
@@
 			(project "PS-HVCarrier"
 				(path "/2365a867-6254-4a7c-9718-f325e0bbac5c/904fa10a-747c-46cf-90d1-33d76069dc5d/b66ae0b0-03e3-4dd0-8364-435fb922b758"
-					(reference "C79")
+					(reference "C81")
 					(unit 1)
 				)
@@
 			)
 		)
-		(property "P/N" "CRCW060310K0FKEI "
+		(property "P/N" "CRCW060310K0FKEI"
 			(at 76.2 68.58 90)
 			(hide yes)
@@
 		(in_pos_files yes)
 		(dnp no)
-		(property "Reference" "C76"
+		(property "Reference" "C78"
 			(at 24.5872 44.5516 0)
 			(show_name no)
@@
 			(project "PS-HVCarrier"
 				(path "/2365a867-6254-4a7c-9718-f325e0bbac5c/904fa10a-747c-46cf-90d1-33d76069dc5d/b66ae0b0-03e3-4dd0-8364-435fb922b758"
-					(reference "C76")
+					(reference "C78")
 					(unit 1)
 				)
@@
 		(dnp no)
 		(fields_autoplaced yes)
-		(property "Reference" "U11"
+		(property "Reference" "U10"
 			(at 60.96 44.45 0)
 			(show_name no)
@@
 					(size 1.27 1.27)
 				)
-			)
-		)
-		(property "PARTREV" "A"
-			(at 60.96 62.23 0)
-			(hide yes)
-			(show_name no)
-			(do_not_autoplace no)
-			(effects
-				(font
-					(size 1.27 1.27)
-				)
-				(justify bottom)
-			)
-		)
-		(property "STANDARD" "IPC-7351B"
-			(at 60.96 62.23 0)
-			(hide yes)
-			(show_name no)
-			(do_not_autoplace no)
-			(effects
-				(font
-					(size 1.27 1.27)
-				)
-				(justify bottom)
-			)
-		)
-		(property "MAXIMUM_PACKAGE_HEIGHT" "0.6mm"
-			(at 60.96 62.23 0)
-			(hide yes)
-			(show_name no)
-			(do_not_autoplace no)
-			(effects
-				(font
-					(size 1.27 1.27)
-				)
-				(justify bottom)
-			)
-		)
-		(property "MANUFACTURER" "Texas Instruments"
-			(at 60.96 62.23 0)
-			(hide yes)
-			(show_name no)
-			(do_not_autoplace no)
-			(effects
-				(font
-					(size 1.27 1.27)
-				)
-				(justify bottom)
 			)
 		)
@@
 			(project "PS-HVCarrier"
 				(path "/2365a867-6254-4a7c-9718-f325e0bbac5c/904fa10a-747c-46cf-90d1-33d76069dc5d/b66ae0b0-03e3-4dd0-8364-435fb922b758"
-					(reference "U11")
+					(reference "U10")
 					(unit 1)
 				)
@@
 		(in_pos_files yes)
 		(dnp no)
-		(property "Reference" "C78"
+		(property "Reference" "C80"
 			(at 43.6372 67.4116 0)
 			(show_name no)
@@
 			(project "PS-HVCarrier"
 				(path "/2365a867-6254-4a7c-9718-f325e0bbac5c/904fa10a-747c-46cf-90d1-33d76069dc5d/b66ae0b0-03e3-4dd0-8364-435fb922b758"
-					(reference "C78")
+					(reference "C80")
 					(unit 1)
 				)
@@
 		(in_pos_files yes)
 		(dnp no)
-		(property "Reference" "C77"
+		(property "Reference" "C79"
 			(at 38.5572 44.5516 0)
 			(show_name no)
@@
 			(project "PS-HVCarrier"
 				(path "/2365a867-6254-4a7c-9718-f325e0bbac5c/904fa10a-747c-46cf-90d1-33d76069dc5d/b66ae0b0-03e3-4dd0-8364-435fb922b758"
-					(reference "C77")
-					(unit 1)
-				)
+					(reference "C79")
+					(unit 1)
+				)

Commit message: added scrut breakout conn
Parts:
- renumbered R68 to R70, R69 to R71, R70 to R72
Changed lines of the file:
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@@
 		(in_pos_files yes)
 		(dnp no)
-		(property "Reference" "R70"
+		(property "Reference" "R72"
 			(at 78.994 67.564 0)
 			(show_name no)
@@
 			(project "PS-HVCarrier"
 				(path "/2365a867-6254-4a7c-9718-f325e0bbac5c/904fa10a-747c-46cf-90d1-33d76069dc5d/b66ae0b0-03e3-4dd0-8364-435fb922b758"
-					(reference "R70")
+					(reference "R72")
 					(unit 1)
 				)
@@
 		(in_pos_files yes)
 		(dnp no)
-		(property "Reference" "R68"
+		(property "Reference" "R70"
 			(at 35.052 59.944 0)
 			(show_name no)
@@
 			(project "PS-HVCarrier"
 				(path "/2365a867-6254-4a7c-9718-f325e0bbac5c/904fa10a-747c-46cf-90d1-33d76069dc5d/b66ae0b0-03e3-4dd0-8364-435fb922b758"
-					(reference "R68")
+					(reference "R70")
 					(unit 1)
 				)
@@
 		(in_pos_files yes)
 		(dnp no)
-		(property "Reference" "R69"
+		(property "Reference" "R71"
 			(at 35.052 67.564 0)
 			(show_name no)
@@
 			(project "PS-HVCarrier"
 				(path "/2365a867-6254-4a7c-9718-f325e0bbac5c/904fa10a-747c-46cf-90d1-33d76069dc5d/b66ae0b0-03e3-4dd0-8364-435fb922b758"
-					(reference "R69")
-					(unit 1)
-				)
+					(reference "R71")
+					(unit 1)
+				)
