File: hardware/HV_Carrier/Voltage_Sense.kicad_sch (KiCad schematic)
At the start: 15 parts

Commit message: update dPN for a bunch of stuff
Parts:
- renumbered TP19 to TP16, TP20 to TP17, TP21 to TP18, TP22 to TP19, TP23 to TP20, TP24 to TP21, TP25 to TP22, TP26 to TP23, TP27 to TP24, TP28 to TP25, TP29 to TP26, TP30 to TP27, TP31 to TP28, TP32 to TP29, TP33 to TP30
Changed lines of the file:
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@@
 		(in_pos_files yes)
 		(dnp no)
-		(property "Reference" "TP20"
+		(property "Reference" "TP17"
 			(at 31.75 100.8379 0)
 			(hide yes)
@@
 			(project "PS-HVCarrier"
 				(path "/2365a867-6254-4a7c-9718-f325e0bbac5c/83ab5b0b-4732-42c0-82fe-e74f4113c82a"
-					(reference "TP20")
+					(reference "TP17")
 					(unit 1)
 				)
@@
 		(in_pos_files yes)
 		(dnp no)
-		(property "Reference" "TP32"
+		(property "Reference" "TP29"
 			(at 151.13 51.3079 0)
 			(hide yes)
@@
 			(project "PS-HVCarrier"
 				(path "/2365a867-6254-4a7c-9718-f325e0bbac5c/83ab5b0b-4732-42c0-82fe-e74f4113c82a"
-					(reference "TP32")
+					(reference "TP29")
 					(unit 1)
 				)
@@
 		(in_pos_files yes)
 		(dnp no)
-		(property "Reference" "TP24"
+		(property "Reference" "TP21"
 			(at 72.39 102.1079 0)
 			(hide yes)
@@
 			(project "PS-HVCarrier"
 				(path "/2365a867-6254-4a7c-9718-f325e0bbac5c/83ab5b0b-4732-42c0-82fe-e74f4113c82a"
-					(reference "TP24")
+					(reference "TP21")
 					(unit 1)
 				)
@@
 		(in_pos_files yes)
 		(dnp no)
-		(property "Reference" "TP23"
+		(property "Reference" "TP20"
 			(at 72.39 97.0279 0)
 			(hide yes)
@@
 			(project "PS-HVCarrier"
 				(path "/2365a867-6254-4a7c-9718-f325e0bbac5c/83ab5b0b-4732-42c0-82fe-e74f4113c82a"
-					(reference "TP23")
+					(reference "TP20")
 					(unit 1)
 				)
@@
 		(in_pos_files yes)
 		(dnp no)
-		(property "Reference" "TP31"
+		(property "Reference" "TP28"
 			(at 148.59 102.1079 0)
 			(hide yes)
@@
 			(project "PS-HVCarrier"
 				(path "/2365a867-6254-4a7c-9718-f325e0bbac5c/83ab5b0b-4732-42c0-82fe-e74f4113c82a"
-					(reference "TP31")
+					(reference "TP28")
 					(unit 1)
 				)
@@
 		(in_pos_files yes)
 		(dnp no)
-		(property "Reference" "TP33"
+		(property "Reference" "TP30"
 			(at 151.13 91.9479 0)
 			(hide yes)
@@
 			(project "PS-HVCarrier"
 				(path "/2365a867-6254-4a7c-9718-f325e0bbac5c/83ab5b0b-4732-42c0-82fe-e74f4113c82a"
-					(reference "TP33")
+					(reference "TP30")
 					(unit 1)
 				)
@@
 		(in_pos_files yes)
 		(dnp no)
-		(property "Reference" "TP26"
+		(property "Reference" "TP23"
 			(at 74.93 91.9479 0)
 			(hide yes)
@@
 			(project "PS-HVCarrier"
 				(path "/2365a867-6254-4a7c-9718-f325e0bbac5c/83ab5b0b-4732-42c0-82fe-e74f4113c82a"
-					(reference "TP26")
+					(reference "TP23")
 					(unit 1)
 				)
@@
 		(in_pos_files yes)
 		(dnp no)
-		(property "Reference" "TP29"
+		(property "Reference" "TP26"
 			(at 148.59 61.4679 0)
 			(hide yes)
@@
 			(project "PS-HVCarrier"
 				(path "/2365a867-6254-4a7c-9718-f325e0bbac5c/83ab5b0b-4732-42c0-82fe-e74f4113c82a"
-					(reference "TP29")
+					(reference "TP26")
 					(unit 1)
 				)
@@
 		(in_pos_files yes)
 		(dnp no)
-		(property "Reference" "TP19"
+		(property "Reference" "TP16"
 			(at 31.75 60.1979 0)
 			(hide yes)
@@
 			(project "PS-HVCarrier"
 				(path "/2365a867-6254-4a7c-9718-f325e0bbac5c/83ab5b0b-4732-42c0-82fe-e74f4113c82a"
-					(reference "TP19")
+					(reference "TP16")
 					(unit 1)
 				)
@@
 		(in_pos_files yes)
 		(dnp no)
-		(property "Reference" "TP27"
+		(property "Reference" "TP24"
 			(at 107.95 60.1979 0)
 			(hide yes)
@@
 			(project "PS-HVCarrier"
 				(path "/2365a867-6254-4a7c-9718-f325e0bbac5c/83ab5b0b-4732-42c0-82fe-e74f4113c82a"
-					(reference "TP27")
+					(reference "TP24")
 					(unit 1)
 				)
@@
 		(in_pos_files yes)
 		(dnp no)
-		(property "Reference" "TP21"
+		(property "Reference" "TP18"
 			(at 72.39 56.3879 0)
 			(hide yes)
@@
 			(project "PS-HVCarrier"
 				(path "/2365a867-6254-4a7c-9718-f325e0bbac5c/83ab5b0b-4732-42c0-82fe-e74f4113c82a"
-					(reference "TP21")
+					(reference "TP18")
 					(unit 1)
 				)
@@
 		(in_pos_files yes)
 		(dnp no)
-		(property "Reference" "TP22"
+		(property "Reference" "TP19"
 			(at 72.39 61.4679 0)
 			(hide yes)
@@
 			(project "PS-HVCarrier"
 				(path "/2365a867-6254-4a7c-9718-f325e0bbac5c/83ab5b0b-4732-42c0-82fe-e74f4113c82a"
-					(reference "TP22")
+					(reference "TP19")
 					(unit 1)
 				)
@@
 		(in_pos_files yes)
 		(dnp no)
-		(property "Reference" "TP28"
+		(property "Reference" "TP25"
 			(at 148.59 56.3879 0)
 			(hide yes)
@@
 			(project "PS-HVCarrier"
 				(path "/2365a867-6254-4a7c-9718-f325e0bbac5c/83ab5b0b-4732-42c0-82fe-e74f4113c82a"
-					(reference "TP28")
+					(reference "TP25")
 					(unit 1)
 				)
@@
 		(in_pos_files yes)
 		(dnp no)
-		(property "Reference" "TP25"
+		(property "Reference" "TP22"
 			(at 74.93 51.3079 0)
 			(hide yes)
@@
 			(project "PS-HVCarrier"
 				(path "/2365a867-6254-4a7c-9718-f325e0bbac5c/83ab5b0b-4732-42c0-82fe-e74f4113c82a"
-					(reference "TP25")
+					(reference "TP22")
 					(unit 1)
 				)
@@
 		(in_pos_files yes)
 		(dnp no)
-		(property "Reference" "TP30"
+		(property "Reference" "TP27"
 			(at 148.59 97.0279 0)
 			(hide yes)
@@
 			(project "PS-HVCarrier"
 				(path "/2365a867-6254-4a7c-9718-f325e0bbac5c/83ab5b0b-4732-42c0-82fe-e74f4113c82a"
-					(reference "TP30")
-					(unit 1)
-				)
+					(reference "TP27")
+					(unit 1)
+				)

Commit message: added scrut breakout conn
Parts:
- renumbered TP16 to TP19, TP17 to TP20, TP18 to TP21, TP19 to TP22, TP20 to TP23, TP21 to TP24, TP22 to TP25, TP23 to TP26, TP24 to TP27, TP25 to TP28, TP26 to TP29, TP27 to TP30, TP28 to TP31, TP29 to TP32, TP30 to TP33
Changed lines of the file:
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@@
 		(in_pos_files yes)
 		(dnp no)
-		(property "Reference" "TP17"
+		(property "Reference" "TP20"
 			(at 31.75 100.8379 0)
 			(hide yes)
@@
 			(project "PS-HVCarrier"
 				(path "/2365a867-6254-4a7c-9718-f325e0bbac5c/83ab5b0b-4732-42c0-82fe-e74f4113c82a"
-					(reference "TP17")
+					(reference "TP20")
 					(unit 1)
 				)
@@
 		(in_pos_files yes)
 		(dnp no)
-		(property "Reference" "TP29"
+		(property "Reference" "TP32"
 			(at 151.13 51.3079 0)
 			(hide yes)
@@
 			(project "PS-HVCarrier"
 				(path "/2365a867-6254-4a7c-9718-f325e0bbac5c/83ab5b0b-4732-42c0-82fe-e74f4113c82a"
-					(reference "TP29")
+					(reference "TP32")
 					(unit 1)
 				)
@@
 		(in_pos_files yes)
 		(dnp no)
-		(property "Reference" "TP21"
+		(property "Reference" "TP24"
 			(at 72.39 102.1079 0)
 			(hide yes)
@@
 			(project "PS-HVCarrier"
 				(path "/2365a867-6254-4a7c-9718-f325e0bbac5c/83ab5b0b-4732-42c0-82fe-e74f4113c82a"
-					(reference "TP21")
+					(reference "TP24")
 					(unit 1)
 				)
@@
 		(in_pos_files yes)
 		(dnp no)
-		(property "Reference" "TP20"
+		(property "Reference" "TP23"
 			(at 72.39 97.0279 0)
 			(hide yes)
@@
 			(project "PS-HVCarrier"
 				(path "/2365a867-6254-4a7c-9718-f325e0bbac5c/83ab5b0b-4732-42c0-82fe-e74f4113c82a"
-					(reference "TP20")
+					(reference "TP23")
 					(unit 1)
 				)
@@
 		(in_pos_files yes)
 		(dnp no)
-		(property "Reference" "TP28"
+		(property "Reference" "TP31"
 			(at 148.59 102.1079 0)
 			(hide yes)
@@
 			(project "PS-HVCarrier"
 				(path "/2365a867-6254-4a7c-9718-f325e0bbac5c/83ab5b0b-4732-42c0-82fe-e74f4113c82a"
-					(reference "TP28")
+					(reference "TP31")
 					(unit 1)
 				)
@@
 		(in_pos_files yes)
 		(dnp no)
-		(property "Reference" "TP30"
+		(property "Reference" "TP33"
 			(at 151.13 91.9479 0)
 			(hide yes)
@@
 			(project "PS-HVCarrier"
 				(path "/2365a867-6254-4a7c-9718-f325e0bbac5c/83ab5b0b-4732-42c0-82fe-e74f4113c82a"
-					(reference "TP30")
+					(reference "TP33")
 					(unit 1)
 				)
@@
 		(in_pos_files yes)
 		(dnp no)
-		(property "Reference" "TP23"
+		(property "Reference" "TP26"
 			(at 74.93 91.9479 0)
 			(hide yes)
@@
 			(project "PS-HVCarrier"
 				(path "/2365a867-6254-4a7c-9718-f325e0bbac5c/83ab5b0b-4732-42c0-82fe-e74f4113c82a"
-					(reference "TP23")
+					(reference "TP26")
 					(unit 1)
 				)
@@
 		(in_pos_files yes)
 		(dnp no)
-		(property "Reference" "TP26"
+		(property "Reference" "TP29"
 			(at 148.59 61.4679 0)
 			(hide yes)
@@
 			(project "PS-HVCarrier"
 				(path "/2365a867-6254-4a7c-9718-f325e0bbac5c/83ab5b0b-4732-42c0-82fe-e74f4113c82a"
-					(reference "TP26")
+					(reference "TP29")
 					(unit 1)
 				)
@@
 		(in_pos_files yes)
 		(dnp no)
-		(property "Reference" "TP16"
+		(property "Reference" "TP19"
 			(at 31.75 60.1979 0)
 			(hide yes)
@@
 			(project "PS-HVCarrier"
 				(path "/2365a867-6254-4a7c-9718-f325e0bbac5c/83ab5b0b-4732-42c0-82fe-e74f4113c82a"
-					(reference "TP16")
+					(reference "TP19")
 					(unit 1)
 				)
@@
 		(in_pos_files yes)
 		(dnp no)
-		(property "Reference" "TP24"
+		(property "Reference" "TP27"
 			(at 107.95 60.1979 0)
 			(hide yes)
@@
 			(project "PS-HVCarrier"
 				(path "/2365a867-6254-4a7c-9718-f325e0bbac5c/83ab5b0b-4732-42c0-82fe-e74f4113c82a"
-					(reference "TP24")
+					(reference "TP27")
 					(unit 1)
 				)
@@
 		(in_pos_files yes)
 		(dnp no)
-		(property "Reference" "TP18"
+		(property "Reference" "TP21"
 			(at 72.39 56.3879 0)
 			(hide yes)
@@
 			(project "PS-HVCarrier"
 				(path "/2365a867-6254-4a7c-9718-f325e0bbac5c/83ab5b0b-4732-42c0-82fe-e74f4113c82a"
-					(reference "TP18")
+					(reference "TP21")
 					(unit 1)
 				)
@@
 		(in_pos_files yes)
 		(dnp no)
-		(property "Reference" "TP19"
+		(property "Reference" "TP22"
 			(at 72.39 61.4679 0)
 			(hide yes)
@@
 			(project "PS-HVCarrier"
 				(path "/2365a867-6254-4a7c-9718-f325e0bbac5c/83ab5b0b-4732-42c0-82fe-e74f4113c82a"
-					(reference "TP19")
+					(reference "TP22")
 					(unit 1)
 				)
@@
 		(in_pos_files yes)
 		(dnp no)
-		(property "Reference" "TP25"
+		(property "Reference" "TP28"
 			(at 148.59 56.3879 0)
 			(hide yes)
@@
 			(project "PS-HVCarrier"
 				(path "/2365a867-6254-4a7c-9718-f325e0bbac5c/83ab5b0b-4732-42c0-82fe-e74f4113c82a"
-					(reference "TP25")
+					(reference "TP28")
 					(unit 1)
 				)
@@
 		(in_pos_files yes)
 		(dnp no)
-		(property "Reference" "TP22"
+		(property "Reference" "TP25"
 			(at 74.93 51.3079 0)
 			(hide yes)
@@
 			(project "PS-HVCarrier"
 				(path "/2365a867-6254-4a7c-9718-f325e0bbac5c/83ab5b0b-4732-42c0-82fe-e74f4113c82a"
-					(reference "TP22")
+					(reference "TP25")
 					(unit 1)
 				)
@@
 		(in_pos_files yes)
 		(dnp no)
-		(property "Reference" "TP27"
+		(property "Reference" "TP30"
 			(at 148.59 97.0279 0)
 			(hide yes)
@@
 			(project "PS-HVCarrier"
 				(path "/2365a867-6254-4a7c-9718-f325e0bbac5c/83ab5b0b-4732-42c0-82fe-e74f4113c82a"
-					(reference "TP27")
-					(unit 1)
-				)
+					(reference "TP30")
+					(unit 1)
+				)
